File: psram.kicad_sch (KiCad schematic)
At the start: 3 parts, among them U6 ESP-PSRAM32

Commit message: 1.01 WIP
Parts:
- C21: renamed from C17; LCSC (none) -> C1711
- JP2: renamed from JP1; AliExpress (none) -> https://www.aliexpress.com/item/1005006454399822.html
- renumbered U6 to U4
Other:
- moved on the sheet: JP2
Changed lines of the file:
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@@
 	(title_block
 		(title "${NAME}")
-		(date "2025-04-30")
+		(date "2025-04-24")
 		(rev "${VERSION}")
 		(company "Mikhail Matveev")
-		(comment 1 "https://github.com/rh1tech/echo")
+		(comment 1 "https://github.com/xtremespb/frank")
 	)
 	(junction
@@
 	(wire
 		(pts
+			(xy 91.44 67.31) (xy 91.44 63.5)
+		)
+		(stroke
+			(width 0)
+			(type default)
+		)
+	)
+	(wire
+		(pts
+			(xy 91.44 67.31) (xy 92.71 67.31)
+		)
+		(stroke
+			(width 0)
+			(type default)
+		)
+	)
+	(wire
+		(pts
 			(xy 46.99 45.72) (xy 46.99 49.53)
 		)
@@
 	(wire
 		(pts
-			(xy 100.33 63.5) (xy 110.49 63.5)
-		)
-		(stroke
-			(width 0)
-			(type default)
-		)
-	)
-	(wire
-		(pts
-			(xy 80.01 63.5) (xy 92.71 63.5)
+			(xy 102.87 67.31) (xy 102.87 63.5)
+		)
+		(stroke
+			(width 0)
+			(type default)
+		)
+	)
+	(wire
+		(pts
+			(xy 102.87 63.5) (xy 110.49 63.5)
+		)
+		(stroke
+			(width 0)
+			(type default)
+		)
+	)
+	(wire
+		(pts
+			(xy 100.33 67.31) (xy 102.87 67.31)
+		)
+		(stroke
+			(width 0)
+			(type default)
+		)
+	)
+	(wire
+		(pts
+			(xy 91.44 63.5) (xy 80.01 63.5)
 		)
 		(stroke
@@
 		(on_board yes)
 		(dnp no)
-		(property "Reference" "#PWR058"
+		(property "Reference" "#PWR051"
 			(at 67.31 77.47 0)
 			(effects
@@
 		(instances
 			(project "frank2"
-				(path "/8c0b3d8b-46d3-4173-ab1e-a61765f77d61/611d88ca-5abf-4eb3-b43a-16174ce65c80"
-					(reference "#PWR058")
+				(path "/8c0b3d8b-46d3-4173-ab1e-a61765f77d61/7211ee19-9793-42f3-8e73-45a2f784dfc8/e4f32ba4-68a3-410a-adde-c38fbc94b887"
+					(reference "#PWR051")
 					(unit 1)
 				)
@@
 		(dnp no)
 		(fields_autoplaced yes)
-		(property "Reference" "#PWR056"
+		(property "Reference" "#PWR049"
 			(at 77.47 49.53 0)
 			(effects
@@
 		(instances
 			(project ""
-				(path "/8c0b3d8b-46d3-4173-ab1e-a61765f77d61/611d88ca-5abf-4eb3-b43a-16174ce65c80"
-					(reference "#PWR056")
+				(path "/8c0b3d8b-46d3-4173-ab1e-a61765f77d61/7211ee19-9793-42f3-8e73-45a2f784dfc8/e4f32ba4-68a3-410a-adde-c38fbc94b887"
+					(reference "#PWR049")
 					(unit 1)
 				)
@@
 		(dnp no)
 		(fields_autoplaced yes)
-		(property "Reference" "U6"
+		(property "Reference" "U4"
 			(at 60.96 57.1499 0)
 			(effects
@@
 		(instances
 			(project "frank2"
-				(path "/8c0b3d8b-46d3-4173-ab1e-a61765f77d61/611d88ca-5abf-4eb3-b43a-16174ce65c80"
-					(reference "U6")
+				(path "/8c0b3d8b-46d3-4173-ab1e-a61765f77d61/7211ee19-9793-42f3-8e73-45a2f784dfc8/e4f32ba4-68a3-410a-adde-c38fbc94b887"
+					(reference "U4")
 					(unit 1)
 				)
@@
 		(on_board yes)
 		(dnp no)
-		(property "Reference" "C17"
+		(property "Reference" "C21"
 			(at 49.911 52.1716 0)
 			(effects
@@
 			)
 		)
+		(property "LCSC" "C1711"
+			(at 46.99 53.34 0)
+			(effects
+				(font
+					(size 1.27 1.27)
+				)
+			)
+		)
 		(pin "1"
 		)
@@
 		(instances
 			(project "frank2"
-				(path "/8c0b3d8b-46d3-4173-ab1e-a61765f77d61/611d88ca-5abf-4eb3-b43a-16174ce65c80"
-					(reference "C17")
+				(path "/8c0b3d8b-46d3-4173-ab1e-a61765f77d61/7211ee19-9793-42f3-8e73-45a2f784dfc8/e4f32ba4-68a3-410a-adde-c38fbc94b887"
+					(reference "C21")
 					(unit 1)
 				)
@@
 	(symbol
 		(lib_id "Jumper:SolderJumper_2_Open")
-		(at 96.52 63.5 0)
+		(at 96.52 67.31 0)
 		(unit 1)
 		(exclude_from_sim no)
@@
 		(on_board yes)
 		(dnp no)
-		(property "Reference" "JP1"
-			(at 96.52 66.04 0)
+		(property "Reference" "JP2"
+			(at 96.52 69.85 0)
 			(effects
 				(font
@@
 		)
 		(property "Value" "Jumper (Solder)"
-			(at 97.028 66.04 0)
+			(at 97.028 69.85 0)
 			(effects
 				(font
@@
 		)
 		(property "Footprint" "FRANK:Jumper (solder)"
-			(at 96.52 63.5 0)
+			(at 96.52 67.31 0)
 			(effects
 				(font
@@
 		)
 		(property "Datasheet" "~"
-			(at 96.52 63.5 0)
+			(at 96.52 67.31 0)
 			(effects
 				(font
@@
 		)
 		(property "Description" "Solder Jumper, 2-pole, open"
-			(at 96.52 63.5 0)
-			(effects
-				(font
-					(size 1.27 1.27)
-				)
-				(hide yes)
-			)
-		)
-		(property "AliExpress" ""
-			(at 96.52 63.5 0)
+			(at 96.52 67.31 0)
+			(effects
+				(font
+					(size 1.27 1.27)
+				)
+				(hide yes)
+			)
+		)
+		(property "AliExpress" "https://www.aliexpress.com/item/1005006454399822.html"
+			(at 96.52 67.31 0)
 			(effects
 				(font
@@
 		(instances
 			(project "frank2"
-				(path "/8c0b3d8b-46d3-4173-ab1e-a61765f77d61/611d88ca-5abf-4eb3-b43a-16174ce65c80"
-					(reference "JP1")
+				(path "/8c0b3d8b-46d3-4173-ab1e-a61765f77d61/7211ee19-9793-42f3-8e73-45a2f784dfc8/e4f32ba4-68a3-410a-adde-c38fbc94b887"
+					(reference "JP2")
 					(unit 1)
 				)
@@
 		(on_board yes)
 		(dnp no)
-		(property "Reference" "#PWR057"
+		(property "Reference" "#PWR050"
 			(at 46.99 67.31 0)
 			(effects
@@
 		(instances
 			(project "frank2"
-				(path "/8c0b3d8b-46d3-4173-ab1e-a61765f77d61/611d88ca-5abf-4eb3-b43a-16174ce65c80"
-					(reference "#PWR057")
+				(path "/8c0b3d8b-46d3-4173-ab1e-a61765f77d61/7211ee19-9793-42f3-8e73-45a2f784dfc8/e4f32ba4-68a3-410a-adde-c38fbc94b887"
+					(reference "#PWR050")
 					(unit 1)
 				)
