File: usbstack.kicad_sch (KiCad schematic)
At the start: 7 parts, among them J8 SS-52100-004

Commit message: Work-in-progress
Parts:
- C15: renamed from C14; LCSC C1713 -> (none)
- C16: renamed from C15; LCSC C1713 -> (none)
- R31: renamed from R25; LCSC C352241 -> (none)
- R32: renamed from R26; LCSC C352241 -> (none)
- R33: renamed from R27; LCSC C352241 -> (none)
- R34: renamed from R28; LCSC C352241 -> (none)
- renumbered J8 to J9
Changed lines of the file:
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@@
 	(title_block
 		(title "${NAME}")
-		(date "2025-04-29")
+		(date "2025-04-30")
 		(rev "${VERSION}")
 		(company "Mikhail Matveev")
@@
 		(dnp no)
 		(fields_autoplaced yes)
-		(property "Reference" "J8"
+		(property "Reference" "J9"
 			(at 121.92 68.58 0)
 			(effects
@@
 			(project "turbofrank"
 				(path "/8c0b3d8b-46d3-4173-ab1e-a61765f77d61/c9a29eca-a7d2-4be5-b06e-7fab67c7ffa0"
-					(reference "J8")
+					(reference "J9")
 					(unit 1)
 				)
@@
 		(on_board yes)
 		(dnp no)
-		(property "Reference" "C14"
+		(property "Reference" "C15"
 			(at 168.021 82.6516 0)
 			(effects
@@
 			)
 		)
-		(property "LCSC" "C1713"
+		(property "LCSC" ""
 			(at 165.1 83.82 0)
 			(effects
@@
 			(project "turbofrank"
 				(path "/8c0b3d8b-46d3-4173-ab1e-a61765f77d61/c9a29eca-a7d2-4be5-b06e-7fab67c7ffa0"
-					(reference "C14")
+					(reference "C15")
 					(unit 1)
 				)
@@
 		(on_board yes)
 		(dnp no)
-		(property "Reference" "R27"
+		(property "Reference" "R33"
 			(at 145.542 104.14 90)
 			(effects
@@
 			)
 		)
-		(property "LCSC" "C352241"
+		(property "LCSC" ""
 			(at 143.51 104.14 0)
 			(effects
@@
 			(project "turbofrank"
 				(path "/8c0b3d8b-46d3-4173-ab1e-a61765f77d61/c9a29eca-a7d2-4be5-b06e-7fab67c7ffa0"
-					(reference "R27")
+					(reference "R33")
 					(unit 1)
 				)
@@
 		(on_board yes)
 		(dnp no)
-		(property "Reference" "C15"
+		(property "Reference" "C16"
 			(at 179.451 82.6516 0)
 			(effects
@@
 			)
 		)
-		(property "LCSC" "C1713"
+		(property "LCSC" ""
 			(at 176.53 83.82 0)
 			(effects
@@
 			(project "turbofrank"
 				(path "/8c0b3d8b-46d3-4173-ab1e-a61765f77d61/c9a29eca-a7d2-4be5-b06e-7fab67c7ffa0"
-					(reference "C15")
+					(reference "C16")
 					(unit 1)
 				)
@@
 		(on_board yes)
 		(dnp no)
-		(property "Reference" "#PWR041"
+		(property "Reference" "#PWR051"
 			(at 135.89 78.74 0)
 			(effects
@@
 			(project "turbofrank"
 				(path "/8c0b3d8b-46d3-4173-ab1e-a61765f77d61/c9a29eca-a7d2-4be5-b06e-7fab67c7ffa0"
-					(reference "#PWR041")
+					(reference "#PWR051")
 					(unit 1)
 				)
@@
 		(on_board yes)
 		(dnp no)
-		(property "Reference" "#PWR043"
+		(property "Reference" "#PWR053"
 			(at 165.1 95.25 0)
 			(effects
@@
 			(project "turbofrank"
 				(path "/8c0b3d8b-46d3-4173-ab1e-a61765f77d61/c9a29eca-a7d2-4be5-b06e-7fab67c7ffa0"
-					(reference "#PWR043")
+					(reference "#PWR053")
 					(unit 1)
 				)
@@
 		(on_board yes)
 		(dnp no)
-		(property "Reference" "R26"
+		(property "Reference" "R32"
 			(at 154.432 102.87 90)
 			(effects
@@
 			)
 		)
-		(property "LCSC" "C352241"
+		(property "LCSC" ""
 			(at 152.4 102.87 0)
 			(effects
@@
 			(project "turbofrank"
 				(path "/8c0b3d8b-46d3-4173-ab1e-a61765f77d61/c9a29eca-a7d2-4be5-b06e-7fab67c7ffa0"
-					(reference "R26")
+					(reference "R32")
 					(unit 1)
 				)
@@
 		(on_board yes)
 		(dnp no)
-		(property "Reference" "#PWR044"
+		(property "Reference" "#PWR054"
 			(at 176.53 95.25 0)
 			(effects
@@
 			(project "turbofrank"
 				(path "/8c0b3d8b-46d3-4173-ab1e-a61765f77d61/c9a29eca-a7d2-4be5-b06e-7fab67c7ffa0"
-					(reference "#PWR044")
+					(reference "#PWR054")
 					(unit 1)
 				)
@@
 		(on_board yes)
 		(dnp no)
-		(property "Reference" "R25"
+		(property "Reference" "R31"
 			(at 141.732 97.79 90)
 			(effects
@@
 			)
 		)
-		(property "LCSC" "C352241"
+		(property "LCSC" ""
 			(at 139.7 97.79 0)
 			(effects
@@
 			(project "turbofrank"
 				(path "/8c0b3d8b-46d3-4173-ab1e-a61765f77d61/c9a29eca-a7d2-4be5-b06e-7fab67c7ffa0"
-					(reference "R25")
+					(reference "R31")
 					(unit 1)
 				)
@@
 		(on_board yes)
 		(dnp no)
-		(property "Reference" "#PWR042"
+		(property "Reference" "#PWR052"
 			(at 142.24 78.74 0)
 			(effects
@@
 			(project "turbofrank"
 				(path "/8c0b3d8b-46d3-4173-ab1e-a61765f77d61/c9a29eca-a7d2-4be5-b06e-7fab67c7ffa0"
-					(reference "#PWR042")
+					(reference "#PWR052")
 					(unit 1)
 				)
@@
 		(dnp no)
 		(fields_autoplaced yes)
-		(property "Reference" "#PWR045"
+		(property "Reference" "#PWR055"
 			(at 121.92 111.76 0)
 			(effects
@@
 			(project "turbofrank"
 				(path "/8c0b3d8b-46d3-4173-ab1e-a61765f77d61/c9a29eca-a7d2-4be5-b06e-7fab67c7ffa0"
-					(reference "#PWR045")
+					(reference "#PWR055")
 					(unit 1)
 				)
@@
 		(on_board yes)
 		(dnp no)
-		(property "Reference" "R28"
+		(property "Reference" "R34"
 			(at 158.242 109.22 90)
 			(effects
@@
 			)
 		)
-		(property "LCSC" "C352241"
+		(property "LCSC" ""
 			(at 156.21 109.22 0)
 			(effects
@@
 			(project "turbofrank"
 				(path "/8c0b3d8b-46d3-4173-ab1e-a61765f77d61/c9a29eca-a7d2-4be5-b06e-7fab67c7ffa0"
-					(reference "R28")
+					(reference "R34")
 					(unit 1)
 				)

Commit message: 1.01 WIP
Parts:
- renumbered J9 to J8, R31 to R35, R32 to R36, R33 to R37, R34 to R38
Changed lines of the file:
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@@
 		(dnp no)
 		(fields_autoplaced yes)
-		(property "Reference" "J9"
+		(property "Reference" "J8"
 			(at 121.92 68.58 0)
 			(effects
@@
 			(project "turbofrank"
 				(path "/8c0b3d8b-46d3-4173-ab1e-a61765f77d61/c9a29eca-a7d2-4be5-b06e-7fab67c7ffa0"
-					(reference "J9")
+					(reference "J8")
 					(unit 1)
 				)
@@
 		(on_board yes)
 		(dnp no)
-		(property "Reference" "R33"
+		(property "Reference" "R37"
 			(at 145.542 104.14 90)
 			(effects
@@
 			(project "turbofrank"
 				(path "/8c0b3d8b-46d3-4173-ab1e-a61765f77d61/c9a29eca-a7d2-4be5-b06e-7fab67c7ffa0"
-					(reference "R33")
+					(reference "R37")
 					(unit 1)
 				)
@@
 		(on_board yes)
 		(dnp no)
-		(property "Reference" "#PWR051"
+		(property "Reference" "#PWR058"
 			(at 135.89 78.74 0)
 			(effects
@@
 			(project "turbofrank"
 				(path "/8c0b3d8b-46d3-4173-ab1e-a61765f77d61/c9a29eca-a7d2-4be5-b06e-7fab67c7ffa0"
-					(reference "#PWR051")
+					(reference "#PWR058")
 					(unit 1)
 				)
@@
 		(on_board yes)
 		(dnp no)
-		(property "Reference" "#PWR053"
+		(property "Reference" "#PWR060"
 			(at 165.1 95.25 0)
 			(effects
@@
 			(project "turbofrank"
 				(path "/8c0b3d8b-46d3-4173-ab1e-a61765f77d61/c9a29eca-a7d2-4be5-b06e-7fab67c7ffa0"
-					(reference "#PWR053")
+					(reference "#PWR060")
 					(unit 1)
 				)
@@
 		(on_board yes)
 		(dnp no)
-		(property "Reference" "R32"
+		(property "Reference" "R36"
 			(at 154.432 102.87 90)
 			(effects
@@
 			(project "turbofrank"
 				(path "/8c0b3d8b-46d3-4173-ab1e-a61765f77d61/c9a29eca-a7d2-4be5-b06e-7fab67c7ffa0"
-					(reference "R32")
+					(reference "R36")
 					(unit 1)
 				)
@@
 		(on_board yes)
 		(dnp no)
-		(property "Reference" "#PWR054"
+		(property "Reference" "#PWR061"
 			(at 176.53 95.25 0)
 			(effects
@@
 			(project "turbofrank"
 				(path "/8c0b3d8b-46d3-4173-ab1e-a61765f77d61/c9a29eca-a7d2-4be5-b06e-7fab67c7ffa0"
-					(reference "#PWR054")
+					(reference "#PWR061")
 					(unit 1)
 				)
@@
 		(on_board yes)
 		(dnp no)
-		(property "Reference" "R31"
+		(property "Reference" "R35"
 			(at 141.732 97.79 90)
 			(effects
@@
 			(project "turbofrank"
 				(path "/8c0b3d8b-46d3-4173-ab1e-a61765f77d61/c9a29eca-a7d2-4be5-b06e-7fab67c7ffa0"
-					(reference "R31")
+					(reference "R35")
 					(unit 1)
 				)
@@
 		(on_board yes)
 		(dnp no)
-		(property "Reference" "#PWR052"
+		(property "Reference" "#PWR059"
 			(at 142.24 78.74 0)
 			(effects
@@
 			(project "turbofrank"
 				(path "/8c0b3d8b-46d3-4173-ab1e-a61765f77d61/c9a29eca-a7d2-4be5-b06e-7fab67c7ffa0"
-					(reference "#PWR052")
+					(reference "#PWR059")
 					(unit 1)
 				)
@@
 		(dnp no)
 		(fields_autoplaced yes)
-		(property "Reference" "#PWR055"
+		(property "Reference" "#PWR062"
 			(at 121.92 111.76 0)
 			(effects
@@
 			(project "turbofrank"
 				(path "/8c0b3d8b-46d3-4173-ab1e-a61765f77d61/c9a29eca-a7d2-4be5-b06e-7fab67c7ffa0"
-					(reference "#PWR055")
+					(reference "#PWR062")
 					(unit 1)
 				)
@@
 		(on_board yes)
 		(dnp no)
-		(property "Reference" "R34"
+		(property "Reference" "R38"
 			(at 158.242 109.22 90)
 			(effects
@@
 			(project "turbofrank"
 				(path "/8c0b3d8b-46d3-4173-ab1e-a61765f77d61/c9a29eca-a7d2-4be5-b06e-7fab67c7ffa0"
-					(reference "R34")
-					(unit 1)
-				)
+					(reference "R38")
+					(unit 1)
+				)
