File: usbstack.kicad_sch (KiCad schematic)
At the start: 7 parts, among them J10 SS-52100-004

Commit message: HW Rev 1.03
Parts:
- renumbered C37 to C36, C38 to C37
Changed lines of the file:
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@@
 	(title_block
 		(title "${NAME}")
-		(date "2025-06-23")
+		(date "2025-07-20")
 		(rev "${VERSION}")
 		(company "Mikhail Matveev")
@@
 		(on_board yes)
 		(dnp no)
-		(property "Reference" "C37"
+		(property "Reference" "C36"
 			(at 178.181 89.0016 0)
 			(effects
@@
 			(project "echo"
 				(path "/8c0b3d8b-46d3-4173-ab1e-a61765f77d61/5ab659b6-5cfd-43f0-936c-acd4035c4ca5"
-					(reference "C37")
+					(reference "C36")
 					(unit 1)
 				)
@@
 		(on_board yes)
 		(dnp no)
-		(property "Reference" "C38"
+		(property "Reference" "C37"
 			(at 189.611 89.0016 0)
 			(effects
@@
 			(project "echo"
 				(path "/8c0b3d8b-46d3-4173-ab1e-a61765f77d61/5ab659b6-5cfd-43f0-936c-acd4035c4ca5"
-					(reference "C38")
+					(reference "C37")
 					(unit 1)
 				)
