File: zero.kicad_sch (KiCad schematic)
At the start: 1 part, among them J7 RP2040-Zero

Commit message: Work-in-progress
Parts:
- renumbered J7 to J8
Connections:
- net ZVBUS renamed VBUS
Changed lines of the file:
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@@
 	(title_block
 		(title "${NAME}")
-		(date "2025-04-29")
+		(date "2025-04-30")
 		(rev "${VERSION}")
 		(company "Mikhail Matveev")
@@
 	(wire
 		(pts
-			(xy 134.62 86.36) (xy 137.16 86.36)
+			(xy 127 88.9) (xy 137.16 88.9)
 		)
 		(stroke
@@
 		)
 	)
+	(wire
+		(pts
+			(xy 127 86.36) (xy 137.16 86.36)
+		)
+		(stroke
+			(width 0)
+			(type default)
+		)
+	)
 	(hierarchical_label "ZGPIO26"
 		(shape input)
@@
 		)
 	)
-	(hierarchical_label "ZVBUS"
-		(shape input)
-		(at 134.62 86.36 180)
-		(effects
-			(font
-				(size 1.27 1.27)
-			)
-			(justify right)
-		)
-	)
 	(hierarchical_label "ZGPIO28"
 		(shape input)
@@
 			)
 			(justify left)
+		)
+	)
+	(symbol
+		(lib_id "power:VBUS")
+		(at 127 86.36 90)
+		(unit 1)
+		(exclude_from_sim no)
+		(in_bom yes)
+		(on_board yes)
+		(dnp no)
+		(fields_autoplaced yes)
+		(property "Reference" "#PWR049"
+			(at 130.81 86.36 0)
+			(effects
+				(font
+					(size 1.27 1.27)
+				)
+				(hide yes)
+			)
+		)
+		(property "Value" "VBUS"
+			(at 123.19 86.3599 90)
+			(effects
+				(font
+					(size 1.27 1.27)
+				)
+				(justify left)
+			)
+		)
+		(property "Footprint" ""
+			(at 127 86.36 0)
+			(effects
+				(font
+					(size 1.27 1.27)
+				)
+				(hide yes)
+			)
+		)
+		(property "Datasheet" ""
+			(at 127 86.36 0)
+			(effects
+				(font
+					(size 1.27 1.27)
+				)
+				(hide yes)
+			)
+		)
+		(property "Description" "Power symbol creates a global label with name \"VBUS\""
+			(at 127 86.36 0)
+			(effects
+				(font
+					(size 1.27 1.27)
+				)
+				(hide yes)
+			)
+		)
+		(pin "1"
+		)
+		(instances
+			(project ""
+				(path "/8c0b3d8b-46d3-4173-ab1e-a61765f77d61/f571fbde-621b-4d45-898a-1392038e5d8f"
+					(reference "#PWR049")
+					(unit 1)
+				)
+			)
 		)
 	)
@@
 		(dnp no)
 		(fields_autoplaced yes)
-		(property "Reference" "J7"
+		(property "Reference" "J8"
 			(at 149.86 78.74 0)
 			(effects
@@
 			(project "frank2"
 				(path "/8c0b3d8b-46d3-4173-ab1e-a61765f77d61/f571fbde-621b-4d45-898a-1392038e5d8f"
-					(reference "J7")
+					(reference "J8")
 					(unit 1)
 				)
@@
 		(lib_name "GND_1")
 		(lib_id "power:GND")
-		(at 137.16 88.9 270)
+		(at 127 88.9 270)
 		(unit 1)
 		(exclude_from_sim no)
@@
 		(dnp no)
 		(fields_autoplaced yes)
-		(property "Reference" "#PWR040"
-			(at 130.81 88.9 0)
+		(property "Reference" "#PWR050"
+			(at 120.65 88.9 0)
 			(effects
 				(font
@@
 		)
 		(property "Value" "GND"
-			(at 133.35 88.8999 90)
+			(at 123.19 88.8999 90)
 			(effects
 				(font
@@
 		)
 		(property "Footprint" ""
-			(at 137.16 88.9 0)
+			(at 127 88.9 0)
 			(effects
 				(font
@@
 		)
 		(property "Datasheet" ""
-			(at 137.16 88.9 0)
+			(at 127 88.9 0)
 			(effects
 				(font
@@
 		)
 		(property "Description" "Power symbol creates a global label with name \"GND\" , ground"
-			(at 137.16 88.9 0)
+			(at 127 88.9 0)
 			(effects
 				(font
@@
 			(project "frank2"
 				(path "/8c0b3d8b-46d3-4173-ab1e-a61765f77d61/f571fbde-621b-4d45-898a-1392038e5d8f"
-					(reference "#PWR040")
+					(reference "#PWR050")
 					(unit 1)
 				)

Commit message: 1.01 WIP
Parts:
- renumbered J8 to J7
Changed lines of the file:
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@@
 		(dnp no)
 		(fields_autoplaced yes)
-		(property "Reference" "#PWR049"
+		(property "Reference" "#PWR056"
 			(at 130.81 86.36 0)
 			(effects
@@
 			(project ""
 				(path "/8c0b3d8b-46d3-4173-ab1e-a61765f77d61/f571fbde-621b-4d45-898a-1392038e5d8f"
-					(reference "#PWR049")
+					(reference "#PWR056")
 					(unit 1)
 				)
@@
 		(dnp no)
 		(fields_autoplaced yes)
-		(property "Reference" "J8"
+		(property "Reference" "J7"
 			(at 149.86 78.74 0)
 			(effects
@@
 			(project "frank2"
 				(path "/8c0b3d8b-46d3-4173-ab1e-a61765f77d61/f571fbde-621b-4d45-898a-1392038e5d8f"
-					(reference "J8")
+					(reference "J7")
 					(unit 1)
 				)
@@
 		(dnp no)
 		(fields_autoplaced yes)
-		(property "Reference" "#PWR050"
+		(property "Reference" "#PWR057"
 			(at 120.65 88.9 0)
 			(effects
@@
 			(project "frank2"
 				(path "/8c0b3d8b-46d3-4173-ab1e-a61765f77d61/f571fbde-621b-4d45-898a-1392038e5d8f"
-					(reference "#PWR050")
+					(reference "#PWR057")
 					(unit 1)
 				)
