File: audio.kicad_sch (KiCad schematic)
At the start: 5 parts, among them J6 PJ-320D

Commit message: Work-in-progress
Parts:
- C13: renamed from C12; LCSC C1711 -> (none)
- C14: renamed from C13; LCSC C1711 -> (none)
- J7: renamed from J6; LCSC C95562 -> (none)
- renumbered R23 to R29, R24 to R30
Changed lines of the file:
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@@
 	(title_block
 		(title "${NAME}")
-		(date "2025-04-29")
+		(date "2025-04-30")
 		(rev "${VERSION}")
 		(company "Mikhail Matveev")
@@
 		(on_board yes)
 		(dnp no)
-		(property "Reference" "R23"
+		(property "Reference" "R29"
 			(at 95.25 80.01 90)
 			(effects
@@
 			(project "echo"
 				(path "/8c0b3d8b-46d3-4173-ab1e-a61765f77d61/e5a22cbe-b729-4e7e-adb7-cba874b6c2eb"
-					(reference "R23")
+					(reference "R29")
 					(unit 1)
 				)
@@
 		(on_board yes)
 		(dnp no)
-		(property "Reference" "#PWR038"
+		(property "Reference" "#PWR047"
 			(at 199.39 104.14 0)
 			(effects
@@
 			(project "minifrank_rm1"
 				(path "/8c0b3d8b-46d3-4173-ab1e-a61765f77d61/e5a22cbe-b729-4e7e-adb7-cba874b6c2eb"
-					(reference "#PWR038")
+					(reference "#PWR047")
 					(unit 1)
 				)
@@
 		(on_board yes)
 		(dnp no)
-		(property "Reference" "J6"
+		(property "Reference" "J7"
 			(at 217.9319 84.8903 0)
 			(effects
@@
 			)
 		)
-		(property "LCSC" "C95562"
+		(property "LCSC" ""
 			(at 210.82 88.9 0)
 			(effects
@@
 			(project "minifrank_rm1"
 				(path "/8c0b3d8b-46d3-4173-ab1e-a61765f77d61/e5a22cbe-b729-4e7e-adb7-cba874b6c2eb"
-					(reference "J6")
+					(reference "J7")
 					(unit 1)
 				)
@@
 		(dnp no)
 		(fields_autoplaced yes)
-		(property "Reference" "#PWR039"
+		(property "Reference" "#PWR048"
 			(at 133.35 130.81 0)
 			(effects
@@
 			(project ""
 				(path "/8c0b3d8b-46d3-4173-ab1e-a61765f77d61/e5a22cbe-b729-4e7e-adb7-cba874b6c2eb"
-					(reference "#PWR039")
+					(reference "#PWR048")
 					(unit 1)
 				)
@@
 		(on_board yes)
 		(dnp no)
-		(property "Reference" "R24"
+		(property "Reference" "R30"
 			(at 129.286 96.266 0)
 			(effects
@@
 			(project "echo"
 				(path "/8c0b3d8b-46d3-4173-ab1e-a61765f77d61/e5a22cbe-b729-4e7e-adb7-cba874b6c2eb"
-					(reference "R24")
+					(reference "R30")
 					(unit 1)
 				)
@@
 		(on_board yes)
 		(dnp no)
-		(property "Reference" "C12"
+		(property "Reference" "C13"
 			(at 139.7 79.502 90)
 			(effects
@@
 			)
 		)
-		(property "LCSC" "C1711"
+		(property "LCSC" ""
 			(at 146.05 81.28 0)
 			(effects
@@
 			(project "echo"
 				(path "/8c0b3d8b-46d3-4173-ab1e-a61765f77d61/e5a22cbe-b729-4e7e-adb7-cba874b6c2eb"
-					(reference "C12")
+					(reference "C13")
 					(unit 1)
 				)
@@
 		(on_board yes)
 		(dnp no)
-		(property "Reference" "C13"
+		(property "Reference" "C14"
 			(at 113.919 96.4184 0)
 			(effects
@@
 			)
 		)
-		(property "LCSC" "C1711"
+		(property "LCSC" ""
 			(at 116.84 95.25 0)
 			(effects
@@
 			(project "echo"
 				(path "/8c0b3d8b-46d3-4173-ab1e-a61765f77d61/e5a22cbe-b729-4e7e-adb7-cba874b6c2eb"
-					(reference "C13")
+					(reference "C14")
 					(unit 1)
 				)

Commit message: 1.01 WIP
Parts:
- renumbered C13 to C12, C14 to C13, R29 to R27, R30 to R28
Changed lines of the file:
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@@
 		(on_board yes)
 		(dnp no)
-		(property "Reference" "R29"
+		(property "Reference" "R27"
 			(at 95.25 80.01 90)
 			(effects
@@
 			(project "echo"
 				(path "/8c0b3d8b-46d3-4173-ab1e-a61765f77d61/e5a22cbe-b729-4e7e-adb7-cba874b6c2eb"
-					(reference "R29")
+					(reference "R27")
 					(unit 1)
 				)
@@
 		(on_board yes)
 		(dnp no)
-		(property "Reference" "#PWR047"
+		(property "Reference" "#PWR050"
 			(at 199.39 104.14 0)
 			(effects
@@
 			(project "minifrank_rm1"
 				(path "/8c0b3d8b-46d3-4173-ab1e-a61765f77d61/e5a22cbe-b729-4e7e-adb7-cba874b6c2eb"
-					(reference "#PWR047")
+					(reference "#PWR050")
 					(unit 1)
 				)
@@
 		(dnp no)
 		(fields_autoplaced yes)
-		(property "Reference" "#PWR048"
+		(property "Reference" "#PWR051"
 			(at 133.35 130.81 0)
 			(effects
@@
 			(project ""
 				(path "/8c0b3d8b-46d3-4173-ab1e-a61765f77d61/e5a22cbe-b729-4e7e-adb7-cba874b6c2eb"
-					(reference "#PWR048")
+					(reference "#PWR051")
 					(unit 1)
 				)
@@
 		(on_board yes)
 		(dnp no)
-		(property "Reference" "R30"
+		(property "Reference" "R28"
 			(at 129.286 96.266 0)
 			(effects
@@
 			(project "echo"
 				(path "/8c0b3d8b-46d3-4173-ab1e-a61765f77d61/e5a22cbe-b729-4e7e-adb7-cba874b6c2eb"
-					(reference "R30")
+					(reference "R28")
 					(unit 1)
 				)
@@
 		(on_board yes)
 		(dnp no)
-		(property "Reference" "C13"
+		(property "Reference" "C12"
 			(at 139.7 79.502 90)
 			(effects
@@
 			(project "echo"
 				(path "/8c0b3d8b-46d3-4173-ab1e-a61765f77d61/e5a22cbe-b729-4e7e-adb7-cba874b6c2eb"
-					(reference "C13")
+					(reference "C12")
 					(unit 1)
 				)
@@
 		(on_board yes)
 		(dnp no)
-		(property "Reference" "C14"
+		(property "Reference" "C13"
 			(at 113.919 96.4184 0)
 			(effects
@@
 			(project "echo"
 				(path "/8c0b3d8b-46d3-4173-ab1e-a61765f77d61/e5a22cbe-b729-4e7e-adb7-cba874b6c2eb"
-					(reference "C14")
-					(unit 1)
-				)
+					(reference "C13")
+					(unit 1)
+				)
