File: audio.kicad_sch (KiCad schematic)
At the start: 5 parts, among them J7 PJ-320D

Commit message: HW Rev 1.03
Parts:
- renumbered C13 to C12, C14 to C13
Changed lines of the file:
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@@
 	(title_block
 		(title "${NAME}")
-		(date "2025-06-23")
+		(date "2025-07-20")
 		(rev "${VERSION}")
 		(company "Mikhail Matveev")
@@
 		(on_board yes)
 		(dnp no)
-		(property "Reference" "C13"
+		(property "Reference" "C12"
 			(at 139.7 79.502 90)
 			(effects
@@
 			(project "echo"
 				(path "/8c0b3d8b-46d3-4173-ab1e-a61765f77d61/e5a22cbe-b729-4e7e-adb7-cba874b6c2eb"
-					(reference "C13")
+					(reference "C12")
 					(unit 1)
 				)
@@
 		(on_board yes)
 		(dnp no)
-		(property "Reference" "C14"
+		(property "Reference" "C13"
 			(at 113.919 96.4184 0)
 			(effects
@@
 			(project "echo"
 				(path "/8c0b3d8b-46d3-4173-ab1e-a61765f77d61/e5a22cbe-b729-4e7e-adb7-cba874b6c2eb"
-					(reference "C14")
+					(reference "C13")
 					(unit 1)
 				)

Commit message: WIP
Parts:
- renumbered C12 to C13, C13 to C14, J7 to J8, R28 to R37, R29 to R38
Changed lines of the file:
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@@
 	(title_block
 		(title "${NAME}")
-		(date "2025-07-20")
+		(date "2025-08-08")
 		(rev "${VERSION}")
 		(company "Mikhail Matveev")
@@
 		(on_board yes)
 		(dnp no)
-		(property "Reference" "R28"
+		(property "Reference" "R37"
 			(at 95.25 80.01 90)
 			(effects
@@
 			(project "echo"
 				(path "/8c0b3d8b-46d3-4173-ab1e-a61765f77d61/e5a22cbe-b729-4e7e-adb7-cba874b6c2eb"
-					(reference "R28")
+					(reference "R37")
 					(unit 1)
 				)
@@
 		(on_board yes)
 		(dnp no)
-		(property "Reference" "#PWR054"
+		(property "Reference" "#PWR066"
 			(at 199.39 104.14 0)
 			(effects
@@
 			(project "minifrank_rm1"
 				(path "/8c0b3d8b-46d3-4173-ab1e-a61765f77d61/e5a22cbe-b729-4e7e-adb7-cba874b6c2eb"
-					(reference "#PWR054")
+					(reference "#PWR066")
 					(unit 1)
 				)
@@
 		(on_board yes)
 		(dnp no)
-		(property "Reference" "J7"
+		(property "Reference" "J8"
 			(at 217.9319 84.8903 0)
 			(effects
@@
 			(project "minifrank_rm1"
 				(path "/8c0b3d8b-46d3-4173-ab1e-a61765f77d61/e5a22cbe-b729-4e7e-adb7-cba874b6c2eb"
-					(reference "J7")
+					(reference "J8")
 					(unit 1)
 				)
@@
 		(dnp no)
 		(fields_autoplaced yes)
-		(property "Reference" "#PWR055"
+		(property "Reference" "#PWR067"
 			(at 133.35 130.81 0)
 			(effects
@@
 			(project ""
 				(path "/8c0b3d8b-46d3-4173-ab1e-a61765f77d61/e5a22cbe-b729-4e7e-adb7-cba874b6c2eb"
-					(reference "#PWR055")
+					(reference "#PWR067")
 					(unit 1)
 				)
@@
 		(on_board yes)
 		(dnp no)
-		(property "Reference" "R29"
+		(property "Reference" "R38"
 			(at 129.286 96.266 0)
 			(effects
@@
 			(project "echo"
 				(path "/8c0b3d8b-46d3-4173-ab1e-a61765f77d61/e5a22cbe-b729-4e7e-adb7-cba874b6c2eb"
-					(reference "R29")
+					(reference "R38")
 					(unit 1)
 				)
@@
 		(on_board yes)
 		(dnp no)
-		(property "Reference" "C12"
+		(property "Reference" "C13"
 			(at 139.7 79.502 90)
 			(effects
@@
 			(project "echo"
 				(path "/8c0b3d8b-46d3-4173-ab1e-a61765f77d61/e5a22cbe-b729-4e7e-adb7-cba874b6c2eb"
-					(reference "C12")
+					(reference "C13")
 					(unit 1)
 				)
@@
 		(on_board yes)
 		(dnp no)
-		(property "Reference" "C13"
+		(property "Reference" "C14"
 			(at 113.919 96.4184 0)
 			(effects
@@
 			(project "echo"
 				(path "/8c0b3d8b-46d3-4173-ab1e-a61765f77d61/e5a22cbe-b729-4e7e-adb7-cba874b6c2eb"
-					(reference "C13")
+					(reference "C14")
 					(unit 1)
 				)

Commit message: Rev 1.05 WIP
Parts:
- C39: renamed from C13; footprint FRANK:Capacitor (0805) -> FRANK:Capacitor (0603)
- C40: renamed from C14; footprint FRANK:Capacitor (0805) -> FRANK:Capacitor (0603)
- R45: renamed from R37; footprint FRANK:Resistor (0805) -> FRANK:Resistor (0603)
- R46: renamed from R38; footprint FRANK:Resistor (0805) -> FRANK:Resistor (0603)
- renumbered J8 to J6
Changed lines of the file:
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@@
 		)
 	)
-	(label "A_OUT"
-		(at 171.45 81.28 180)
+	(hierarchical_label "A_OUT"
+		(shape input)
+		(at 171.45 81.28 0)
 		(effects
 			(font
 				(size 1.27 1.27)
 			)
-			(justify right bottom)
-		)
-	)
-	(label "A_OUT"
-		(at 194.31 88.9 0)
+			(justify left)
+		)
+	)
+	(hierarchical_label "A_OUT"
+		(shape input)
+		(at 194.31 83.82 180)
 		(effects
 			(font
 				(size 1.27 1.27)
 			)
-			(justify left bottom)
-		)
-	)
-	(label "A_OUT"
-		(at 194.31 83.82 0)
+			(justify right)
+		)
+	)
+	(hierarchical_label "A_OUT"
+		(shape input)
+		(at 194.31 88.9 180)
 		(effects
 			(font
 				(size 1.27 1.27)
 			)
-			(justify left bottom)
+			(justify right)
 		)
 	)
@@
 		(on_board yes)
 		(dnp no)
-		(property "Reference" "R37"
+		(property "Reference" "R45"
 			(at 95.25 80.01 90)
 			(effects
@@
 			)
 		)
-		(property "Footprint" "FRANK:Resistor (0805)"
+		(property "Footprint" "FRANK:Resistor (0603)"
 			(at 100.33 83.058 90)
 			(effects
@@
 			(project "echo"
 				(path "/8c0b3d8b-46d3-4173-ab1e-a61765f77d61/e5a22cbe-b729-4e7e-adb7-cba874b6c2eb"
-					(reference "R37")
+					(reference "R45")
 					(unit 1)
 				)
@@
 		(on_board yes)
 		(dnp no)
-		(property "Reference" "#PWR066"
+		(property "Reference" "#PWR096"
 			(at 199.39 104.14 0)
 			(effects
@@
 			(project "minifrank_rm1"
 				(path "/8c0b3d8b-46d3-4173-ab1e-a61765f77d61/e5a22cbe-b729-4e7e-adb7-cba874b6c2eb"
-					(reference "#PWR066")
+					(reference "#PWR096")
 					(unit 1)
 				)
@@
 		(on_board yes)
 		(dnp no)
-		(property "Reference" "J8"
+		(property "Reference" "J6"
 			(at 217.9319 84.8903 0)
 			(effects
@@
 			(project "minifrank_rm1"
 				(path "/8c0b3d8b-46d3-4173-ab1e-a61765f77d61/e5a22cbe-b729-4e7e-adb7-cba874b6c2eb"
-					(reference "J8")
+					(reference "J6")
 					(unit 1)
 				)
@@
 		(dnp no)
 		(fields_autoplaced yes)
-		(property "Reference" "#PWR067"
+		(property "Reference" "#PWR097"
 			(at 133.35 130.81 0)
 			(effects
@@
 			(project ""
 				(path "/8c0b3d8b-46d3-4173-ab1e-a61765f77d61/e5a22cbe-b729-4e7e-adb7-cba874b6c2eb"
-					(reference "#PWR067")
+					(reference "#PWR097")
 					(unit 1)
 				)
@@
 		(on_board yes)
 		(dnp no)
-		(property "Reference" "R38"
+		(property "Reference" "R46"
 			(at 129.286 96.266 0)
 			(effects
@@
 			)
 		)
-		(property "Footprint" "FRANK:Resistor (0805)"
+		(property "Footprint" "FRANK:Resistor (0603)"
 			(at 135.128 95.25 90)
 			(effects
@@
 			(project "echo"
 				(path "/8c0b3d8b-46d3-4173-ab1e-a61765f77d61/e5a22cbe-b729-4e7e-adb7-cba874b6c2eb"
-					(reference "R38")
+					(reference "R46")
 					(unit 1)
 				)
@@
 		(on_board yes)
 		(dnp no)
-		(property "Reference" "C13"
+		(property "Reference" "C39"
 			(at 139.7 79.502 90)
 			(effects
@@
 			)
 		)
-		(property "Footprint" "FRANK:Capacitor (0805)"
+		(property "Footprint" "FRANK:Capacitor (0603)"
 			(at 142.24 82.2452 0)
 			(effects
@@
 			(project "echo"
 				(path "/8c0b3d8b-46d3-4173-ab1e-a61765f77d61/e5a22cbe-b729-4e7e-adb7-cba874b6c2eb"
-					(reference "C13")
+					(reference "C39")
 					(unit 1)
 				)
@@
 		(on_board yes)
 		(dnp no)
-		(property "Reference" "C14"
+		(property "Reference" "C40"
 			(at 113.919 96.4184 0)
 			(effects
@@
 			)
 		)
-		(property "Footprint" "FRANK:Capacitor (0805)"
+		(property "Footprint" "FRANK:Capacitor (0603)"
 			(at 115.8748 91.44 0)
 			(effects
@@
 			(project "echo"
 				(path "/8c0b3d8b-46d3-4173-ab1e-a61765f77d61/e5a22cbe-b729-4e7e-adb7-cba874b6c2eb"
-					(reference "C14")
-					(unit 1)
-				)
+					(reference "C40")
+					(unit 1)
+				)

Commit message: HW 1.06 WIP
Parts:
- renumbered C40 to C53, C39 to C54, R45 to R52, R46 to R53
Changed lines of the file:
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@@
 		(on_board yes)
 		(dnp no)
-		(property "Reference" "R45"
+		(property "Reference" "R52"
 			(at 95.25 80.01 90)
 			(effects
@@
 			(project "echo"
 				(path "/8c0b3d8b-46d3-4173-ab1e-a61765f77d61/e5a22cbe-b729-4e7e-adb7-cba874b6c2eb"
-					(reference "R45")
+					(reference "R52")
 					(unit 1)
 				)
@@
 		(on_board yes)
 		(dnp no)
-		(property "Reference" "#PWR096"
+		(property "Reference" "#PWR0118"
 			(at 199.39 104.14 0)
 			(effects
@@
 			(project "minifrank_rm1"
 				(path "/8c0b3d8b-46d3-4173-ab1e-a61765f77d61/e5a22cbe-b729-4e7e-adb7-cba874b6c2eb"
-					(reference "#PWR096")
+					(reference "#PWR0118")
 					(unit 1)
 				)
@@
 		(dnp no)
 		(fields_autoplaced yes)
-		(property "Reference" "#PWR097"
+		(property "Reference" "#PWR0117"
 			(at 133.35 130.81 0)
 			(effects
@@
 			(project ""
 				(path "/8c0b3d8b-46d3-4173-ab1e-a61765f77d61/e5a22cbe-b729-4e7e-adb7-cba874b6c2eb"
-					(reference "#PWR097")
+					(reference "#PWR0117")
 					(unit 1)
 				)
@@
 		(on_board yes)
 		(dnp no)
-		(property "Reference" "R46"
+		(property "Reference" "R53"
 			(at 129.286 96.266 0)
 			(effects
@@
 			(project "echo"
 				(path "/8c0b3d8b-46d3-4173-ab1e-a61765f77d61/e5a22cbe-b729-4e7e-adb7-cba874b6c2eb"
-					(reference "R46")
+					(reference "R53")
 					(unit 1)
 				)
@@
 		(on_board yes)
 		(dnp no)
-		(property "Reference" "C39"
+		(property "Reference" "C54"
 			(at 139.7 79.502 90)
 			(effects
@@
 			(project "echo"
 				(path "/8c0b3d8b-46d3-4173-ab1e-a61765f77d61/e5a22cbe-b729-4e7e-adb7-cba874b6c2eb"
-					(reference "C39")
+					(reference "C54")
 					(unit 1)
 				)
@@
 		(on_board yes)
 		(dnp no)
-		(property "Reference" "C40"
+		(property "Reference" "C53"
 			(at 113.919 96.4184 0)
 			(effects
@@
 			(project "echo"
 				(path "/8c0b3d8b-46d3-4173-ab1e-a61765f77d61/e5a22cbe-b729-4e7e-adb7-cba874b6c2eb"
-					(reference "C40")
-					(unit 1)
-				)
+					(reference "C53")
+					(unit 1)
+				)
