File: sd.kicad_sch (KiCad schematic)
At the start: 3 parts, among them J4 0475710001, J5 104031-0811

Commit message: Work-in-progress
Parts:
- C12: renamed from C11; LCSC C1711 -> (none)
- renumbered J4 to J5, J5 to J6
Changed lines of the file:
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@@
 	(title_block
 		(title "${NAME}")
-		(date "2025-04-29")
+		(date "2025-04-30")
 		(rev "${VERSION}")
 		(company "Mikhail Matveev")
@@
 		(on_board yes)
 		(dnp no)
-		(property "Reference" "C11"
+		(property "Reference" "C12"
 			(at 172.6184 70.231 0)
 			(effects
@@
 			)
 		)
-		(property "LCSC" "C1711"
+		(property "LCSC" ""
 			(at 171.45 67.31 0)
 			(effects
@@
 			(project "minifrank_rm1"
 				(path "/8c0b3d8b-46d3-4173-ab1e-a61765f77d61/b68ee207-ff62-4120-93b6-b15e01f03b46"
-					(reference "C11")
+					(reference "C12")
 					(unit 1)
 				)
@@
 		(dnp no)
 		(fields_autoplaced yes)
-		(property "Reference" "#PWR033"
+		(property "Reference" "#PWR042"
 			(at 161.29 71.12 0)
 			(effects
@@
 			(project "minifrank_rm1"
 				(path "/8c0b3d8b-46d3-4173-ab1e-a61765f77d61/b68ee207-ff62-4120-93b6-b15e01f03b46"
-					(reference "#PWR033")
+					(reference "#PWR042")
 					(unit 1)
 				)
@@
 		(on_board yes)
 		(dnp no)
-		(property "Reference" "#PWR034"
+		(property "Reference" "#PWR043"
 			(at 181.61 67.31 0)
 			(effects
@@
 			(project "minifrank_rm1"
 				(path "/8c0b3d8b-46d3-4173-ab1e-a61765f77d61/b68ee207-ff62-4120-93b6-b15e01f03b46"
-					(reference "#PWR034")
+					(reference "#PWR043")
 					(unit 1)
 				)
@@
 		(dnp no)
 		(fields_autoplaced yes)
-		(property "Reference" "#PWR032"
+		(property "Reference" "#PWR041"
 			(at 88.9 67.31 0)
 			(effects
@@
 			(project "minifrank_rm1"
 				(path "/8c0b3d8b-46d3-4173-ab1e-a61765f77d61/b68ee207-ff62-4120-93b6-b15e01f03b46"
-					(reference "#PWR032")
+					(reference "#PWR041")
 					(unit 1)
 				)
@@
 		(dnp no)
 		(fields_autoplaced yes)
-		(property "Reference" "J4"
+		(property "Reference" "J5"
 			(at 111.76 57.15 0)
 			(effects
@@
 			(project "minifrank_rm1"
 				(path "/8c0b3d8b-46d3-4173-ab1e-a61765f77d61/b68ee207-ff62-4120-93b6-b15e01f03b46"
-					(reference "J4")
+					(reference "J5")
 					(unit 1)
 				)
@@
 		(dnp no)
 		(fields_autoplaced yes)
-		(property "Reference" "#PWR036"
+		(property "Reference" "#PWR045"
 			(at 134.62 72.39 0)
 			(effects
@@
 			(project "minifrank_rm1"
 				(path "/8c0b3d8b-46d3-4173-ab1e-a61765f77d61/b68ee207-ff62-4120-93b6-b15e01f03b46"
-					(reference "#PWR036")
+					(reference "#PWR045")
 					(unit 1)
 				)
@@
 		(dnp no)
 		(fields_autoplaced yes)
-		(property "Reference" "#PWR037"
+		(property "Reference" "#PWR046"
 			(at 165.1 113.03 0)
 			(effects
@@
 			(project "minifrank_rm1"
 				(path "/8c0b3d8b-46d3-4173-ab1e-a61765f77d61/b68ee207-ff62-4120-93b6-b15e01f03b46"
-					(reference "#PWR037")
+					(reference "#PWR046")
 					(unit 1)
 				)
@@
 		(dnp no)
 		(fields_autoplaced yes)
-		(property "Reference" "J5"
+		(property "Reference" "J6"
 			(at 194.945 88.9 0)
 			(effects
@@
 			(project "minifrank_rm1"
 				(path "/8c0b3d8b-46d3-4173-ab1e-a61765f77d61/b68ee207-ff62-4120-93b6-b15e01f03b46"
-					(reference "J5")
+					(reference "J6")
 					(unit 1)
 				)
@@
 		(dnp no)
 		(fields_autoplaced yes)
-		(property "Reference" "#PWR035"
+		(property "Reference" "#PWR044"
 			(at 88.9 69.85 0)
 			(effects
@@
 			(project "minifrank_rm1"
 				(path "/8c0b3d8b-46d3-4173-ab1e-a61765f77d61/b68ee207-ff62-4120-93b6-b15e01f03b46"
-					(reference "#PWR035")
+					(reference "#PWR044")
 					(unit 1)
 				)
@@
 		(dnp no)
 		(fields_autoplaced yes)
-		(property "Reference" "#PWR031"
+		(property "Reference" "#PWR040"
 			(at 88.9 64.77 0)
 			(effects
@@
 			(project "minifrank_rm1"
 				(path "/8c0b3d8b-46d3-4173-ab1e-a61765f77d61/b68ee207-ff62-4120-93b6-b15e01f03b46"
-					(reference "#PWR031")
+					(reference "#PWR040")
 					(unit 1)
 				)

Commit message: 1.01 WIP
Parts:
- renumbered C12 to C11
Changed lines of the file:
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@@
 		(on_board yes)
 		(dnp no)
-		(property "Reference" "C12"
+		(property "Reference" "C11"
 			(at 172.6184 70.231 0)
 			(effects
@@
 			(project "minifrank_rm1"
 				(path "/8c0b3d8b-46d3-4173-ab1e-a61765f77d61/b68ee207-ff62-4120-93b6-b15e01f03b46"
-					(reference "C12")
+					(reference "C11")
 					(unit 1)
 				)
@@
 		(dnp no)
 		(fields_autoplaced yes)
-		(property "Reference" "#PWR042"
+		(property "Reference" "#PWR045"
 			(at 161.29 71.12 0)
 			(effects
@@
 			(project "minifrank_rm1"
 				(path "/8c0b3d8b-46d3-4173-ab1e-a61765f77d61/b68ee207-ff62-4120-93b6-b15e01f03b46"
-					(reference "#PWR042")
+					(reference "#PWR045")
 					(unit 1)
 				)
@@
 		(on_board yes)
 		(dnp no)
-		(property "Reference" "#PWR043"
+		(property "Reference" "#PWR046"
 			(at 181.61 67.31 0)
 			(effects
@@
 			(project "minifrank_rm1"
 				(path "/8c0b3d8b-46d3-4173-ab1e-a61765f77d61/b68ee207-ff62-4120-93b6-b15e01f03b46"
-					(reference "#PWR043")
+					(reference "#PWR046")
 					(unit 1)
 				)
@@
 		(dnp no)
 		(fields_autoplaced yes)
-		(property "Reference" "#PWR041"
+		(property "Reference" "#PWR044"
 			(at 88.9 67.31 0)
 			(effects
@@
 			(project "minifrank_rm1"
 				(path "/8c0b3d8b-46d3-4173-ab1e-a61765f77d61/b68ee207-ff62-4120-93b6-b15e01f03b46"
-					(reference "#PWR041")
+					(reference "#PWR044")
 					(unit 1)
 				)
@@
 		(dnp no)
 		(fields_autoplaced yes)
-		(property "Reference" "#PWR045"
+		(property "Reference" "#PWR048"
 			(at 134.62 72.39 0)
 			(effects
@@
 			(project "minifrank_rm1"
 				(path "/8c0b3d8b-46d3-4173-ab1e-a61765f77d61/b68ee207-ff62-4120-93b6-b15e01f03b46"
-					(reference "#PWR045")
+					(reference "#PWR048")
 					(unit 1)
 				)
@@
 		(dnp no)
 		(fields_autoplaced yes)
-		(property "Reference" "#PWR046"
+		(property "Reference" "#PWR049"
 			(at 165.1 113.03 0)
 			(effects
@@
 			(project "minifrank_rm1"
 				(path "/8c0b3d8b-46d3-4173-ab1e-a61765f77d61/b68ee207-ff62-4120-93b6-b15e01f03b46"
-					(reference "#PWR046")
+					(reference "#PWR049")
 					(unit 1)
 				)
@@
 		(dnp no)
 		(fields_autoplaced yes)
-		(property "Reference" "#PWR044"
+		(property "Reference" "#PWR047"
 			(at 88.9 69.85 0)
 			(effects
@@
 			(project "minifrank_rm1"
 				(path "/8c0b3d8b-46d3-4173-ab1e-a61765f77d61/b68ee207-ff62-4120-93b6-b15e01f03b46"
-					(reference "#PWR044")
+					(reference "#PWR047")
 					(unit 1)
 				)
@@
 		(dnp no)
 		(fields_autoplaced yes)
-		(property "Reference" "#PWR040"
+		(property "Reference" "#PWR043"
 			(at 88.9 64.77 0)
 			(effects
@@
 			(project "minifrank_rm1"
 				(path "/8c0b3d8b-46d3-4173-ab1e-a61765f77d61/b68ee207-ff62-4120-93b6-b15e01f03b46"
-					(reference "#PWR040")
-					(unit 1)
-				)
+					(reference "#PWR043")
+					(unit 1)
+				)
