File: sd.kicad_sch (KiCad schematic)
At the start: 3 parts, among them J5 0475710001, J6 104031-0811

Commit message: HW Rev 1.03
Parts:
- renumbered C12 to C11
Changed lines of the file:
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@@
 	(title_block
 		(title "${NAME}")
-		(date "2025-06-23")
+		(date "2025-07-20")
 		(rev "${VERSION}")
 		(company "Mikhail Matveev")
@@
 		(on_board yes)
 		(dnp no)
-		(property "Reference" "C12"
+		(property "Reference" "C11"
 			(at 172.6184 70.231 0)
 			(effects
@@
 			(project "minifrank_rm1"
 				(path "/8c0b3d8b-46d3-4173-ab1e-a61765f77d61/b68ee207-ff62-4120-93b6-b15e01f03b46"
-					(reference "C12")
+					(reference "C11")
 					(unit 1)
 				)

Commit message: WIP
Parts:
- removed J6: 104031-0811, FRANK:MicroSD (SMD, long), symbol Connector:Micro_SD_Card
- renumbered C11 to C12, J5 to J6
Connections:
- no-connect marks 1 -> 0
Other:
- moved on the sheet: C12, J6

Commit message: Rev 1.05 WIP
Parts:
- C38: renamed from C12; footprint FRANK:Capacitor (0805) -> FRANK:Capacitor (0603)
- renumbered J6 to J5
Changed lines of the file:
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@@
 		(on_board yes)
 		(dnp no)
-		(property "Reference" "C12"
+		(property "Reference" "C38"
 			(at 205.6384 93.091 0)
 			(effects
@@
 			)
 		)
-		(property "Footprint" "FRANK:Capacitor (0805)"
+		(property "Footprint" "FRANK:Capacitor (0603)"
 			(at 200.66 91.1352 0)
 			(effects
@@
 			(project "minifrank_rm1"
 				(path "/8c0b3d8b-46d3-4173-ab1e-a61765f77d61/b68ee207-ff62-4120-93b6-b15e01f03b46"
-					(reference "C12")
+					(reference "C38")
 					(unit 1)
 				)
@@
 		(dnp no)
 		(fields_autoplaced yes)
-		(property "Reference" "#PWR057"
+		(property "Reference" "#PWR088"
 			(at 194.31 93.98 0)
 			(effects
@@
 			(project "minifrank_rm1"
 				(path "/8c0b3d8b-46d3-4173-ab1e-a61765f77d61/b68ee207-ff62-4120-93b6-b15e01f03b46"
-					(reference "#PWR057")
+					(reference "#PWR088")
 					(unit 1)
 				)
@@
 		(on_board yes)
 		(dnp no)
-		(property "Reference" "#PWR058"
+		(property "Reference" "#PWR089"
 			(at 214.63 90.17 0)
 			(effects
@@
 			(project "minifrank_rm1"
 				(path "/8c0b3d8b-46d3-4173-ab1e-a61765f77d61/b68ee207-ff62-4120-93b6-b15e01f03b46"
-					(reference "#PWR058")
+					(reference "#PWR089")
 					(unit 1)
 				)
@@
 		(dnp no)
 		(fields_autoplaced yes)
-		(property "Reference" "#PWR056"
+		(property "Reference" "#PWR087"
 			(at 121.92 90.17 0)
 			(effects
@@
 			(project "minifrank_rm1"
 				(path "/8c0b3d8b-46d3-4173-ab1e-a61765f77d61/b68ee207-ff62-4120-93b6-b15e01f03b46"
-					(reference "#PWR056")
+					(reference "#PWR087")
 					(unit 1)
 				)
@@
 		(dnp no)
 		(fields_autoplaced yes)
-		(property "Reference" "J6"
+		(property "Reference" "J5"
 			(at 144.78 80.01 0)
 			(effects
@@
 			(project "minifrank_rm1"
 				(path "/8c0b3d8b-46d3-4173-ab1e-a61765f77d61/b68ee207-ff62-4120-93b6-b15e01f03b46"
-					(reference "J6")
+					(reference "J5")
 					(unit 1)
 				)
@@
 		(dnp no)
 		(fields_autoplaced yes)
-		(property "Reference" "#PWR060"
+		(property "Reference" "#PWR091"
 			(at 167.64 95.25 0)
 			(effects
@@
 			(project "minifrank_rm1"
 				(path "/8c0b3d8b-46d3-4173-ab1e-a61765f77d61/b68ee207-ff62-4120-93b6-b15e01f03b46"
-					(reference "#PWR060")
+					(reference "#PWR091")
 					(unit 1)
 				)
@@
 		(dnp no)
 		(fields_autoplaced yes)
-		(property "Reference" "#PWR059"
+		(property "Reference" "#PWR090"
 			(at 121.92 92.71 0)
 			(effects
@@
 			(project "minifrank_rm1"
 				(path "/8c0b3d8b-46d3-4173-ab1e-a61765f77d61/b68ee207-ff62-4120-93b6-b15e01f03b46"
-					(reference "#PWR059")
+					(reference "#PWR090")
 					(unit 1)
 				)
@@
 		(dnp no)
 		(fields_autoplaced yes)
-		(property "Reference" "#PWR055"
+		(property "Reference" "#PWR086"
 			(at 121.92 87.63 0)
 			(effects
@@
 			(project "minifrank_rm1"
 				(path "/8c0b3d8b-46d3-4173-ab1e-a61765f77d61/b68ee207-ff62-4120-93b6-b15e01f03b46"
-					(reference "#PWR055")
-					(unit 1)
-				)
+					(reference "#PWR086")
+					(unit 1)
+				)

Commit message: HW 1.06 WIP
Parts:
- renumbered C38 to C52
Changed lines of the file:
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@@
 		(on_board yes)
 		(dnp no)
-		(property "Reference" "C38"
+		(property "Reference" "C52"
 			(at 205.6384 93.091 0)
 			(effects
@@
 			(project "minifrank_rm1"
 				(path "/8c0b3d8b-46d3-4173-ab1e-a61765f77d61/b68ee207-ff62-4120-93b6-b15e01f03b46"
-					(reference "C38")
+					(reference "C52")
 					(unit 1)
 				)
@@
 		(dnp no)
 		(fields_autoplaced yes)
-		(property "Reference" "#PWR088"
+		(property "Reference" "#PWR0111"
 			(at 194.31 93.98 0)
 			(effects
@@
 			(project "minifrank_rm1"
 				(path "/8c0b3d8b-46d3-4173-ab1e-a61765f77d61/b68ee207-ff62-4120-93b6-b15e01f03b46"
-					(reference "#PWR088")
+					(reference "#PWR0111")
 					(unit 1)
 				)
@@
 		(on_board yes)
 		(dnp no)
-		(property "Reference" "#PWR089"
+		(property "Reference" "#PWR0112"
 			(at 214.63 90.17 0)
 			(effects
@@
 			(project "minifrank_rm1"
 				(path "/8c0b3d8b-46d3-4173-ab1e-a61765f77d61/b68ee207-ff62-4120-93b6-b15e01f03b46"
-					(reference "#PWR089")
+					(reference "#PWR0112")
 					(unit 1)
 				)
@@
 		(dnp no)
 		(fields_autoplaced yes)
-		(property "Reference" "#PWR087"
+		(property "Reference" "#PWR0108"
 			(at 121.92 90.17 0)
 			(effects
@@
 			(project "minifrank_rm1"
 				(path "/8c0b3d8b-46d3-4173-ab1e-a61765f77d61/b68ee207-ff62-4120-93b6-b15e01f03b46"
-					(reference "#PWR087")
+					(reference "#PWR0108")
 					(unit 1)
 				)
@@
 		(dnp no)
 		(fields_autoplaced yes)
-		(property "Reference" "#PWR091"
+		(property "Reference" "#PWR0110"
 			(at 167.64 95.25 0)
 			(effects
@@
 			(project "minifrank_rm1"
 				(path "/8c0b3d8b-46d3-4173-ab1e-a61765f77d61/b68ee207-ff62-4120-93b6-b15e01f03b46"
-					(reference "#PWR091")
+					(reference "#PWR0110")
 					(unit 1)
 				)
@@
 		(dnp no)
 		(fields_autoplaced yes)
-		(property "Reference" "#PWR090"
+		(property "Reference" "#PWR0109"
 			(at 121.92 92.71 0)
 			(effects
@@
 			(project "minifrank_rm1"
 				(path "/8c0b3d8b-46d3-4173-ab1e-a61765f77d61/b68ee207-ff62-4120-93b6-b15e01f03b46"
-					(reference "#PWR090")
+					(reference "#PWR0109")
 					(unit 1)
 				)
@@
 		(dnp no)
 		(fields_autoplaced yes)
-		(property "Reference" "#PWR086"
+		(property "Reference" "#PWR0107"
 			(at 121.92 87.63 0)
 			(effects
@@
 			(project "minifrank_rm1"
 				(path "/8c0b3d8b-46d3-4173-ab1e-a61765f77d61/b68ee207-ff62-4120-93b6-b15e01f03b46"
-					(reference "#PWR086")
-					(unit 1)
-				)
+					(reference "#PWR0107")
+					(unit 1)
+				)
