File: usba.kicad_sch (KiCad schematic)
At the start: 5 parts, among them J8 676430910, U6 USBLC6-2SC6

Commit message: Echo HW Rev 1.01
Other:
- title: Protea -> ${NAME}
Changed lines of the file:
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@@
 	(paper "A4")
 	(title_block
-		(title "Protea")
-		(date "2025-03-08")
-		(rev "2.03")
+		(title "${NAME}")
+		(date "2025-05-24")
+		(rev "${VERSION}")
 		(company "Mikhail Matveev")
-		(comment 1 "https://github.com/xtremespb/frank")
+		(comment 1 "https://github.com/rh1tech/echo")
 	)
 	(junction
