File: audio_multiplexer.kicad_sch (KiCad schematic)
At the start: 3 parts, among them J5 0475710001, J6 104031-0811

Commit message: Minor fixes
Parts:
- removed C12: 100n, FRANK:Capacitor (0805), symbol Device:C
- removed J5: 0475710001, FRANK:MicroSD (SMD, short), symbol FRANK:MicroSD_Short
- removed J6: 104031-0811, FRANK:MicroSD (SMD, long), symbol Connector:Micro_SD_Card
- added C11: 100n, FRANK:Capacitor (0805), symbol Device:C
- added R34: 10K, FRANK:Resistor (0805), symbol Device:R
- added U4: 74HC4052D, FRANK:74HC4052D653, symbol FRANK:74HC4052D
Connections:
- net +3V3: now also C11.2, U4.16 (VCC)
- net GND: now also C11.1, R34.1, U4.11 (1Y3), U4.15 (1Y2), U4.2 (2Y2), U4.4 (2Y3), U4.6 (~{E}), U4.7 (VEE), U4.8 (GND), U4.9 (S1)
- new net AMP_IN_L: U4.13 (1Z)
- new net AMP_IN_R: U4.3 (2Z)
- new net AUDIOSW: R34.2, U4.10 (S0)
- new net PWM_OUT_L: U4.12 (1Y0)
- new net PWM_OUT_R: U4.1 (2Y0)
- new net TDA_L: U4.14 (1Y1)
- new net TDA_R: U4.5 (2Y1)
- no-connect marks 1 -> 0
Other:
- title: ${NAME} -> MiniFRANK RM1P2
