File: echo.kicad_pcb (KiCad board)
At the start: 2 copper layers, 99 x 70 mm, 128 parts, among them J1 USB4215-03-A, J10 SS-52100-004, J2 D-SUB 9 Male, J3 MDC-036, J4 D-SUB 15 Female, J5 0475710001, J6 104031-0811, J7 PJ-320D, J8 PJ-320D, J9 MDC-036, Q1 BSS138, Q2 BSS138, Q3 AO3400A, Q4 AO3400A, Q5 AO3400A, Q6 AO3400A, U1 SN74CBT3257CDR, U10 TS3USB221RSER, U2 CH340C, U3 NCP1117 3.3, U4 USBLC6-2SC6, U5 ESP32-WROVER-E, U6 W25Q128JVSIQ, U7 RP2040, U8 TS3USB221RSER, U9 MW7211A, Y1 12 MHz

Commit message: Minor updates
Routing:
- net Net-(U9-VD3): track 3.31 -> 4.31 mm
- net /USB1_D2+: track 32.6 -> 31.7 mm, vias 2 -> 0
- net /ESP_IO2: track 38.7 -> 37.8 mm
- net /USB1_D2-: track 30.2 -> 31.1 mm
- net VBUS: track 459.9 -> 460.8 mm
- net /ESP_IO18: track 30.3 -> 29.8 mm
- net /ESP_IO5: track 26.9 -> 26.3 mm
- net /ESP_IO4: track 21.2 -> 20.7 mm
- net /ESP_IO23: track 46.4 -> 45.9 mm
- net /ESP_IO19: track 33.2 -> 32.6 mm
- net GND: vias 28 -> 29

Commit message: HW Rev 1.03
Parts:
- removed the C5 at (120.9, 98.5)
- renumbered C11 to C10, C12 to C11, C13 to C12, C14 to C13, C15 to C14, C16 to C15, C17 to C16, C18 to C17, C19 to C18, C20 to C19, C21 to C20, C22 to C21, C23 to C22, C24 to C23, C25 to C24, C26 to C25, C27 to C26, C28 to C27, C29 to C28, C30 to C29, C31 to C30, C32 to C31, C33 to C32, C34 to C33, C35 to C34, C36 to C35, C37 to C36, C38 to C37, C6 to C5, C7 to C6, C8 to C7, C9 to C8, C10 to C9
Connections:
- C4 pad 1: VBUS -> +3V3
- R4 pad 2: VBUS -> +3V3
- R5 pad 1: VBUS -> +3V3
- U2 pad 16: VBUS -> +3V3
- U2 pad 4: Net-(U2-3V) -> +3V3
Routing:
- net +3V3: track 245.8 -> 278.2 mm, vias 11 -> 15
- net VBUS: track 460.8 -> 441.6 mm, vias 4 -> 3
- net Net-(U2-3V): track 4.08 -> 0.00 mm
- net /ESP_IO34: track 116.1 -> 119.0 mm
- net Net-(Q2-E): track 21.0 -> 21.9 mm
- net GND: vias 29 -> 30

Commit message: WIP
Parts:
- removed the C21 at (90.4, 102.8)
- removed the C30 at (91.0, 93.9)
- removed the J3 at (100.2, 57.6)
- removed the J5 at (168.7, 87.2)
- removed J7: PJ-320D, FRANK:Jack (3.5mm, PJ-320D)
- removed the R23 at (115.2, 68.0)
- removed the R24 at (124.0, 71.5)
- removed the R25 at (113.5, 78.0)
- removed the R26 at (113.5, 74.5)
- removed the R27 at (118.0, 78.8)
- removed the R28 at (79.8, 64.5)
- removed the R29 at (84.0, 64.5)
- removed the R30 at (95.5, 68.8)
- removed the R42 at (126.5, 71.5)
- removed the U8 at (113.8, 104.4)
- added C19: 100n, FRANK:Capacitor (0805), F.Cu at (107.8, 85.3)
- added C29: 1u, FRANK:Capacitor (0805), F.Cu at (121.9, 90.3)
- added J11: SS-52100-004, FRANK:USB Type A (stacked), F.Cu at (94.0, 100.1)
- added J2: USB4215-03-A, FRANK:USB Type C, F.Cu at (123.6, 112.3)
- added J4: MDC-036, FRANK:MiniDIN (6 Pin, female), F.Cu at (107.8, 57.6)
- added R14: 22R, FRANK:Resistor (0805), F.Cu at (137.7, 101.0)
- added R15: 5.1K, FRANK:Resistor (0805), F.Cu at (140.1, 99.8)
- added R16: 1M, FRANK:Resistor (0805), F.Cu at (149.2, 104.2)
- added R17: 1K, FRANK:Resistor (0805), F.Cu at (108.5, 90.8)
- added R18: 5.1K, FRANK:Resistor (0805), F.Cu at (121.2, 101.2)
- added R19: 22R, FRANK:Resistor (0805), F.Cu at (123.5, 100.2)
- added R20: 22R, FRANK:Resistor (0805), F.Cu at (125.5, 100.2)
- added R21: 5.1K, FRANK:Resistor (0805), F.Cu at (127.8, 101.2)
- added R33: 22K, FRANK:Resistor (0805), F.Cu at (118.2, 70.5)
- added R49: 22K, FRANK:Resistor (0805), F.Cu at (97.5, 69.8)
- added R50: 4.7K, FRANK:Resistor (0805), F.Cu at (97.5, 72.0)
- added R51: 22K, FRANK:Resistor (0805), F.Cu at (100.0, 75.0)
- added R52: 22R, FRANK:Resistor (0805), F.Cu at (109.2, 93.2)
- added R53: 22R, FRANK:Resistor (0805), F.Cu at (101.7, 93.2)
- added R54: 22R, FRANK:Resistor (0805), F.Cu at (109.5, 95.8)
- added R55: 22R, FRANK:Resistor (0805), F.Cu at (97.6, 94.3)
- added R56: 10K, FRANK:Resistor (0805), F.Cu at (118.2, 97.0)
- added S5: RP Boot, FRANK:Button (SMD, 3x3mm, 1-1), F.Cu at (85.2, 60.2)
- added U5: USBLC6-2SC6, FRANK:SOT-23-6, F.Cu at (124.0, 95.0)
- C12, C37: value 10u -> 100n
- C13: value 33n -> 10u
- C14: value 100n -> 33n
- C27: value 1u -> 100n
- C32: value 100n -> 15p
- C34: value 4.7u -> 10u
- C35, C8: value 100n -> 10u
- C36: value 10u -> 4.7u
- J10: value SS-52100-004 -> MDC-036; footprint FRANK:USB Type A (stacked) -> FRANK:MiniDIN (6 Pin, female)
- J6: value 104031-0811 -> 0475710001; footprint FRANK:MicroSD (SMD, long) -> FRANK:MicroSD (SMD, short)
- J9: value MDC-036 -> PJ-320D; footprint FRANK:MiniDIN (6 Pin, female) -> FRANK:Jack (3.5mm, PJ-320D)
- LD3: value Green (Power) -> Green
- R10: value 22R -> 2.2K
- R11: value 5.1K -> 2.2K
- R12: value 1M -> 5.1K
- R13: value 1K -> 22R
- R22: value 22K -> 1M
- R31: value 10K -> 22K
- R32: value 27R -> 4.7K
- R34: value 27R -> 22K
- R35: value 1K -> 4.7K
- R36: value 1K -> 22K
- R37: value 22K -> 100R
- R38: value 4.7K -> 150R
- R39, R40: value 22K -> 10K
- R4, R5: value 1.5K -> 10K
- R41: value 4.7K -> 27R
- R43: value 10K -> 27R
- R44: value 10K -> 1K
- R45: value 22R -> 1K
- R46, R48: value 22R -> 22K
- R47: value 22R -> 4.7K
- R6, R7: value 2.2K -> 10K
- R8: value 5.1K -> 1.5K
- R9: value 22R -> 1.5K
- S1: footprint FRANK:TACT-SIDE-4623 -> FRANK:Button (SMD, 3x3mm, 1-1)
- S4: value RP Boot -> Power; footprint FRANK:TACT-SIDE-4623 -> FRANK:Switch (MSK12C02)
- moved C12 93.5 mm to (171.5, 57.0)
- moved H1 93.5 mm to (171.5, 52.0)
- moved C15 85.1 mm to (171.2, 102.2), turned to 180 degrees
- moved H2 84.0 mm to (87.0, 52.0)
- moved C9 81.6 mm to (167.5, 86.8), turned to 90 degrees
- moved D1 76.9 mm to (169.8, 79.0), turned to 90 degrees
- moved C16 73.4 mm to (156.0, 102.0), turned to 180 degrees
- moved C17 65.5 mm to (156.0, 104.8)
- moved LD3 63.5 mm to (108.5, 88.5)
- moved C32 61.7 mm to (102.4, 81.2), turned to -90 degrees
- moved R3 60.8 mm to (98.5, 81.5), turned to 180 degrees
- moved C13 60.3 mm to (137.5, 67.2)
- moved R2 60.0 mm to (98.5, 79.2), turned to 180 degrees
- moved JP2 59.1 mm to (141.2, 62.5)
- moved C36 57.8 mm to (113.0, 109.5)
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- renumbered C19 to C20, C20 to C21, C29 to C30, J2 to J3, J4 to J5, R14 to R23, R15 to R24, R16 to R25, R17 to R26, R18 to R27, R19 to R28, R20 to R29, R21 to R30, R33 to R42, U5 to U6, U6 to U7, U7 to U8
Connections:
- C11 pad 1: GND -> VBUS
- C11 pad 2: +3V3 -> GND
- C12 pad 1: /Audio Out/A_OUT -> GND
- C12 pad 2: Net-(C12-Pad2) -> +3V3
- C13 pad 1: GND -> /Audio Out/A_OUT
- C13 pad 2: Net-(C12-Pad2) -> Net-(C13-Pad2)
- C14 pad 2: /Tape In/G -> Net-(C13-Pad2)
- C15 pad 1: /ESP_IO34 -> GND
- C15 pad 2: /Tape In/L -> /Tape In/G
- C16 pad 2: /Tape In/R -> /Tape In/L
- C17 pad 1: Net-(U7-VREG_VOUT) -> /ESP_IO34
- C17 pad 2: GND -> /Tape In/R
- C18 pad 1: Net-(U7-VREG_VOUT) -> Net-(U8-VREG_VOUT)
- C27 pad 1: Net-(U7-VREG_VOUT) -> +3V3
- C28 pad 1: +3V3 -> Net-(U8-VREG_VOUT)
- C31 pad 1: /RP2040/XIN -> Net-(C31-Pad1)
- C32 pad 1: VBUS -> /RP2040/XIN
- C33 pad 1: GND -> VBUS
- C33 pad 2: +3V3 -> GND
- C35 pad 1: GND -> VBUS
- C35 pad 2: +3V3 -> GND
- C37 pad 1: VBUS -> GND
- C37 pad 2: GND -> +3V3
- C7 pad 1: +3V3 -> VBUS
- C9 pad 1: VBUS -> +3V3
- J1 pad 11: VBUS -> Net-(S4-B)
- J1 pad 2: VBUS -> Net-(S4-B)
- J10 pad 1: VBUS -> /MS_DATA
- J10 pad 2: Net-(J10-D1-) -> unconnected-(J10-Pad2)
- J10 pad 3: Net-(J10-D1+) -> GND
- J10 pad 4: GND -> VBUS
- J10 pad 5: VBUS -> /MS_CLK
- J10 pad 6: Net-(J10-D2-) -> unconnected-(J10-Pad6)
- J8 pad R: /Tape In/R -> /Audio Out/A_OUT
- J8 pad S: /Tape In/G -> GND
- J8 pad T: /Tape In/L -> /Audio Out/A_OUT
- JP2 pad 2: /UMSW1 -> /UMSW
- JP2 pad 3: /UMSW2 -> /AUDIO_IN
- JP2 pad 4: GND -> /ESP_IO25
- R10 pad 1: Net-(R10-Pad1) -> Net-(Q1-B)
- R10 pad 2: Net-(J1-DP1) -> Net-(Q2-E)
- R11 pad 1: GND -> Net-(Q2-B)
- R11 pad 2: Net-(J1-CC2) -> Net-(Q1-E)
- R12 pad 1: Net-(J1-SHIELD) -> GND
- R12 pad 2: GND -> Net-(J1-CC1)
- R13 pad 1: Net-(LD3-A) -> Net-(R13-Pad1)
- R13 pad 2: +3V3 -> Net-(J1-DN1)
- R2 pad 1: /ESP_EN -> /GPIO11
- R2 pad 2: +3V3 -> GND
- R22 pad 1: +3V3 -> Net-(J2-SHIELD)
- R22 pad 2: /KB_DATA_3V -> GND
- R3 pad 1: /ESP_IO36 -> /GPIO12
- R3 pad 2: +3V3 -> GND
- R31 pad 1: /ESP_IO34 -> +3V3
- R31 pad 2: VBUS -> /KB_DATA_3V
- R32 pad 1: /RP_D+ -> +3V3
- R32 pad 2: Net-(U7-USB_DP) -> Net-(Q3-G)
- R34 pad 1: /RP_D- -> +3V3
- R34 pad 2: Net-(U7-USB_DM) -> /MS_CLK_3V
- R35 pad 1: /RP2040/XOUT -> +3V3
- R35 pad 2: Net-(C30-Pad1) -> Net-(Q4-G)
- R36 pad 1: Net-(LD4-A) -> VBUS
- R36 pad 2: /RP2040/GPIO25 -> /MS_CLK
- R37 pad 1: +3V3 -> /AUDIO_IN
- R37 pad 2: /MS_DATA_3V -> Net-(C13-Pad2)
- R38 pad 1: +3V3 -> GND
- R38 pad 2: Net-(Q5-G) -> Net-(C13-Pad2)
- R39 pad 1: VBUS -> /ESP_IO34
- R39 pad 2: /MS_DATA -> GND
- R4 pad 1: Net-(LD1-A) -> /GPIO14
- R4 pad 2: +3V3 -> GND
- R40 pad 1: +3V3 -> /ESP_IO34
- R40 pad 2: /KB_CLK_3V -> VBUS
- R41 pad 1: +3V3 -> /RP_D+
- R41 pad 2: Net-(Q6-G) -> Net-(U8-USB_DP)
- R42 pad 2: Net-(R33-Pad2) -> Net-(R42-Pad2)
- R43 pad 1: +3V3 -> /RP_D-
- R43 pad 2: /UMSW2 -> Net-(U8-USB_DM)
- R44 pad 1: +3V3 -> /RP2040/XOUT
- R44 pad 2: /UMSW1 -> Net-(C31-Pad1)
- R45 pad 1: /USB1_D1+ -> Net-(LD4-A)
- R45 pad 2: Net-(J10-D1+) -> /RP2040/GPIO25
- R46 pad 1: /USB1_D2+ -> +3V3
- R46 pad 2: Net-(J10-D2+) -> /MS_DATA_3V
- R47 pad 1: /USB1_D1- -> +3V3
- R47 pad 2: Net-(J10-D1-) -> Net-(Q5-G)
- R48 pad 1: /USB1_D2- -> VBUS
- R48 pad 2: Net-(J10-D2-) -> /MS_DATA
- R5 pad 1: +3V3 -> /GPIO15
- R5 pad 2: Net-(LD2-A) -> GND
- R6 pad 1: Net-(Q1-B) -> /ESP_EN
- R6 pad 2: Net-(Q2-E) -> +3V3
- R7 pad 1: Net-(Q2-B) -> /ESP_IO36
- R7 pad 2: Net-(Q1-E) -> +3V3
- R8 pad 1: GND -> Net-(LD1-A)
- R8 pad 2: Net-(J1-CC1) -> +3V3
- R9 pad 1: Net-(R9-Pad1) -> +3V3
- R9 pad 2: Net-(J1-DN1) -> Net-(LD2-A)
- S4 pad 1: Net-(R33-Pad2) -> unconnected-(S4-C-Pad1)
- S4 pad 2: GND -> Net-(S4-B)
- U10 pad 1: /UTC_D+ -> /TC2_D+
- U10 pad 2: /UTC_D- -> /TC2_D-
- U10 pad 3: /MP1_D+ -> /UH_D+
- U10 pad 4: /MP1_D- -> /UH_D-
- U10 pad 7: /PW_D- -> /RP_D-
- U10 pad 8: /PW_D+ -> /RP_D+
- U10 pad 9: /UMSW1 -> /UMSW
- U2 pad 5: /UTC_D+ -> /TC1_D+
- U2 pad 6: /UTC_D- -> /TC1_D-
- U4 pad 1: Net-(R9-Pad1) -> Net-(R13-Pad1)
- U4 pad 3: Net-(R10-Pad1) -> Net-(R14-Pad1)
- U4 pad 4: /PW_D+ -> /TC1_D+
- U4 pad 6: /PW_D- -> /TC1_D-
- U8 pad 23: Net-(U7-VREG_VOUT) -> Net-(U8-VREG_VOUT)
- U8 pad 45: Net-(U7-VREG_VOUT) -> Net-(U8-VREG_VOUT)
- U8 pad 46: Net-(U7-USB_DM) -> Net-(U8-USB_DM)
- U8 pad 47: Net-(U7-USB_DP) -> Net-(U8-USB_DP)
- U8 pad 50: Net-(U7-VREG_VOUT) -> Net-(U8-VREG_VOUT)
- U9 pad 1: /USB Hub/DM4 -> /USB Hub/D1-
- U9 pad 10: /HUB_D- -> /UH_D-
- U9 pad 11: /HUB_D+ -> /UH_D+
- U9 pad 2: /USB Hub/DP4 -> /USB Hub/D1+
- U9 pad 3: /USB Hub/DM3 -> /USB Hub/D2-
- U9 pad 4: /USB Hub/DP3 -> /USB Hub/D2+
- U9 pad 5: /USB1_D2- -> unconnected-(U9-DM2-Pad5)
- U9 pad 6: /USB1_D2+ -> unconnected-(U9-DP2-Pad6)
- U9 pad 7: /USB1_D1- -> unconnected-(U9-DM3-Pad7)
- U9 pad 8: /USB1_D1+ -> unconnected-(U9-DP3-Pad8)
- Y1 pad 3: Net-(C30-Pad1) -> Net-(C31-Pad1)
Routing:
- net /ESP_IO34: track 119.0 -> 0.00 mm, vias 2 -> 0
- net /ESP_IO25: track 100.5 -> 0.00 mm, vias 4 -> 0
- net /MS_DATA: track 79.0 -> 0.00 mm, vias 1 -> 0
- net /MS_CLK: track 62.9 -> 0.00 mm, vias 1 -> 0
- net /SN74_S: track 59.9 -> 0.00 mm, vias 2 -> 0
- net /ESP_IO26: track 59.1 -> 0.00 mm, vias 4 -> 0
- net /ESP_EN: track 56.6 -> 0.00 mm, vias 2 -> 0
- net /KB_CLK: track 51.3 -> 0.00 mm, vias 1 -> 0
- net VBUS: track 441.6 -> 392.6 mm, vias 3 -> 11
- net /ESP_IO23: track 45.9 -> 0.00 mm
- net /ESP_IO32: track 45.0 -> 0.00 mm, vias 2 -> 0
- net /ESP_IO22: track 43.1 -> 0.00 mm
- net /GPIO12: track 54.3 -> 11.7 mm, vias 2 -> 0
- net /GPIO14: track 56.2 -> 14.2 mm
- net /GPIO5: track 50.8 -> 9.13 mm, vias 0 -> 1
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- added copper zone on B.Cu, net Net-(U8-VREG_VOUT)
- added copper zone on F.Cu, net Net-(U8-VREG_VOUT)
- removed copper zone on B.Cu, net +3V3
- removed copper zone on B.Cu, net Net-(U7-VREG_VOUT)
- removed copper zone on F.Cu, net Net-(U7-VREG_VOUT)
Other:
- board size 99 x 70 mm -> 90.9 x 61.9 mm
- board text removed: "AUDIO OUT"
- board text removed: "ESP BTN"
- board text removed: "ESP RESET"
- board text removed: "PS/2 / USB"
- board text removed: "PS/2 KEYBOARD"
- board text removed: "PS/2 MOUSE"
- board text removed: "RP BOOT"
- board text removed: "RP HUB / BOOT"
- board text removed: "RP RESET"
- board text removed: "TAPE IN"
- board text removed: "USB-TTL / RP"

Commit message: HW 1.04
Parts:
- moved S5 56.3 mm to (139.8, 74.1), turned to 0 degrees
- moved R4 29.0 mm to (87.2, 57.0)
- moved R3 24.9 mm to (87.2, 59.2)
- moved R2 21.0 mm to (87.2, 61.5)
- moved R5 4.78 mm to (98.0, 81.2)
- moved R33 0.32 mm to (118.2, 70.2)
- moved H1 0.24 mm to (171.7, 52.0)
- moved H2 0.18 mm to (86.8, 52.0)
Routing:
- net /ESP_IO27: track 0.00 -> 98.6 mm, vias 0 -> 2
- net /ESP_IO33: track 0.00 -> 98.3 mm, vias 0 -> 2
- net /ESP_IO32: track 0.00 -> 96.3 mm, vias 0 -> 2
- net /ESP_IO26: track 0.00 -> 89.4 mm, vias 0 -> 2
- net /ESP_EN: track 0.00 -> 83.7 mm, vias 0 -> 4
- net /Audio Out/A_OUT: track 0.00 -> 67.9 mm, vias 0 -> 4
- net /MS_DATA_3V: track 0.00 -> 57.1 mm, vias 0 -> 4
- net /GPIO2: track 11.6 -> 65.5 mm
- net /SN74_S: track 0.00 -> 51.5 mm, vias 0 -> 7
- net /GPIO12: track 11.7 -> 59.8 mm, vias 0 -> 2
- net /UMSW: track 5.55 -> 51.7 mm, vias 0 -> 2
- net /GPIO6: track 8.24 -> 50.2 mm
- net /GPIO11: track 13.4 -> 54.4 mm, vias 0 -> 2
- net /ESP_IO34: track 0.00 -> 39.1 mm
- net /GPIO8: track 9.31 -> 47.9 mm, vias 1 -> 2
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Other:
- outline, holes or cut-outs redrawn
- board text added: "AUDIO OUT"
- board text added: "BTN 36"
- board text added: "DH"
- board text added: "KEYBOARD"
- board text added: "MOUSE"
- board text added: "PU"
- board text added: "PWR/ESP"
- board text added: "RESET"
- board text added: "RP"
- board text added: "RP BOOT"
- board text added: "RP RESET"
- board text added: "TAPE IN"
- board text added: "TI"
- board text added: "VGA VIDEO"

Commit message: Rev 1.05 WIP
Parts:
- removed J10: MDC-036, FRANK:MiniDIN (6 Pin, female)
- removed J11: SS-52100-004, FRANK:USB Type A (stacked)
- removed J9: PJ-320D, FRANK:Jack (3.5mm, PJ-320D)
- removed JP1: ESP-RP RST, FRANK:Jumper (solder)
- removed S4: Power, FRANK:Switch (MSK12C02)
- added AJ1: PJ-320D, FRANK:Jack (3.5mm, PJ-320D), F.Cu at (149.8, 78.8)
- added C38: 100n, FRANK:Capacitor (0603), F.Cu at (146.2, 101.0)
- added C39: 10u, FRANK:Capacitor (0603), F.Cu at (149.5, 61.8)
- added C40: 33n, FRANK:Capacitor (0603), F.Cu at (152.0, 61.5)
- added C41: 100n, FRANK:Capacitor (0603), F.Cu at (177.2, 92.5)
- added C42: 100n, FRANK:Capacitor (0603), F.Cu at (166.5, 89.0)
- added C43: 100n, FRANK:Capacitor (0603), F.Cu at (221.5, 104.2)
- added C44: 100n, FRANK:Capacitor (0603), F.Cu at (219.5, 87.2)
- added C45: 100n, FRANK:Capacitor (0603), F.Cu at (232.0, 97.0)
- added C46: 100n, FRANK:Capacitor (0603), F.Cu at (232.0, 94.8)
- added C47: 100n, FRANK:Capacitor (0603), F.Cu at (221.2, 87.2)
- added C48: 100n, FRANK:Capacitor (0603), F.Cu at (216.2, 102.0)
- added C49: 100n, FRANK:Capacitor (0603), F.Cu at (218.0, 103.8)
- added C50: 100n, FRANK:Capacitor (0603), F.Cu at (215.2, 98.5)
- added C51: 100n, FRANK:Capacitor (0603), F.Cu at (226.8, 104.2)
- added C52: 100n, FRANK:Capacitor (0603), F.Cu at (215.2, 94.8)
- added C53: 1u, FRANK:Capacitor (0603), F.Cu at (228.5, 104.2)
- added C54: 1u, FRANK:Capacitor (0603), F.Cu at (219.8, 104.2)
- added C55: 100n, FRANK:Capacitor (0603), F.Cu at (237.8, 103.2)
- added C56: 15p, FRANK:Capacitor (0603), F.Cu at (232.0, 86.8)
- added C57: 15p, FRANK:Capacitor (0603), F.Cu at (224.8, 87.2)
- added C58: 100n, FRANK:Capacitor (0603), F.Cu at (162.8, 60.2)
- added C59: 10u, FRANK:Capacitor (0603), F.Cu at (177.8, 99.2)
- added C60: 10u, FRANK:Capacitor (0603), F.Cu at (177.8, 103.0)
- added C61: 4.7u, FRANK:Capacitor (0603), F.Cu at (206.8, 79.8)
- added C62: 100n, FRANK:Capacitor (0603), F.Cu at (215.2, 105.0)
- added D2: 1N4148, FRANK:Diode (SOD-323), F.Cu at (174.0, 85.5)
- added FB1: 220R, FRANK:Inductor (0805), F.Cu at (238.8, 68.8)
- added FB2: 220R, FRANK:Inductor (0805), F.Cu at (238.8, 53.2)
- added J7: MDC-036, FRANK:MiniDIN (6 Pin, female), F.Cu at (156.5, 54.2)
- added JP3: Main Jumpers, FRANK:SW_DS05-127-2-03BK-SMT-TR, F.Cu at (192.5, 84.5)
- added Q7: AO3400A, FRANK:SOT-23, F.Cu at (161.0, 65.5)
- added Q8: AO3400A, FRANK:SOT-23, F.Cu at (173.2, 63.2)
- added R57: 22K, FRANK:Resistor (0603), F.Cu at (161.0, 69.5)
- added R58: 4.7K, FRANK:Resistor (0603), F.Cu at (158.0, 68.2)
- added R59: 22K, FRANK:Resistor (0603), F.Cu at (162.0, 62.2)
- added R60: 22K, FRANK:Resistor (0603), F.Cu at (174.2, 60.2)
- added R61: 4.7K, FRANK:Resistor (0603), F.Cu at (172.0, 66.8)
- added R62: 22K, FRANK:Resistor (0603), F.Cu at (176.5, 63.0)
- added R63: 22R, FRANK:Resistor (0603), F.Cu at (188.0, 92.2)
- added R64: 22R, FRANK:Resistor (0603), F.Cu at (190.8, 92.2)
- added R65: 22R, FRANK:Resistor (0603), F.Cu at (193.2, 92.2)
- added R66: 22R, FRANK:Resistor (0603), F.Cu at (195.8, 92.2)
- added R67: 10K, FRANK:Resistor (0603), F.Cu at (220.0, 107.2)
- added TP1: MS9288_SCL, FRANK:TestPoint (Pad 1.0x1.0mm), B.Cu at (212.9, 62.8)
- added TP2: MS9288_SDA, FRANK:TestPoint (Pad 1.0x1.0mm), B.Cu at (212.9, 64.8)
- added U11: RP2040, FRANK:QFN 56, F.Cu at (224.0, 96.0)
- added U12: MW7211A, FRANK:SOP-16, F.Cu at (206.2, 84.8)
- added U13: TS3USB221RSER, FRANK:UQFN-10, F.Cu at (214.8, 108.5)
- added X1: 24.576 MHz, FRANK:Crystal (2520), F.Cu at (217.2, 60.0)
- C1, C10, C12, C15, C16, C17, C18, C2, C22, C23, C3, C4, C5, C6, C7, C8, C9: footprint FRANK:Capacitor (0805) -> FRANK:Capacitor (0603)
- C11, C19, C20, C24, C27: value 100n -> 10u; footprint FRANK:Capacitor (0805) -> FRANK:Capacitor (0603)
- C13: value 10u -> 100n; footprint FRANK:Capacitor (0805) -> FRANK:Capacitor (0603)
- C14: value 33n -> 100n; footprint FRANK:Capacitor (0805) -> FRANK:Capacitor (0603)
- C21, C25, C37: value 100n -> 1u; footprint FRANK:Capacitor (0805) -> FRANK:Capacitor (0603)
- C26: value 100n -> 1n; footprint FRANK:Capacitor (0805) -> FRANK:Capacitor (0603)
- C28: value 1u -> 220n; footprint FRANK:Capacitor (0805) -> FRANK:Capacitor (0603)
- C29: value 1u -> 4.7u; footprint FRANK:Capacitor (0805) -> FRANK:Capacitor (0603)
- C30: value 100n -> 220n; footprint FRANK:Capacitor (0805) -> FRANK:Capacitor (0603)
- C31: value 15p -> 4.7u; footprint FRANK:Capacitor (0805) -> FRANK:Capacitor (0603)
- C32: value 15p -> 220n; footprint FRANK:Capacitor (0805) -> FRANK:Capacitor (0603)
- C33: value 100n -> 4.7u; footprint FRANK:Capacitor (0805) -> FRANK:Capacitor (0603)
- C34, C35: value 10u -> 15p; footprint FRANK:Capacitor (0805) -> FRANK:Capacitor (0603)
- C36: value 4.7u -> 1u; footprint FRANK:Capacitor (0805) -> FRANK:Capacitor (0603)
- D1: value Zener 3V3 -> 1N5819WS; footprint FRANK:Diode (0805) -> FRANK:Diode (SOD-323)
- J3: value D-SUB 9 Male -> MDC-036; footprint FRANK:D-SUB (9 pin, male, top mount) -> FRANK:MiniDIN (6 Pin, female)
- J4: value MDC-036 -> DC3RX19JA2; footprint FRANK:MiniDIN (6 Pin, female) -> FRANK:HDMI (female)
- J5: value D-SUB 15 Female -> 0475710001; footprint FRANK:D-SUB (15 pin, female) -> FRANK:MicroSD (SMD, short)
- J6: value 0475710001 -> PJ-320D; footprint FRANK:MicroSD (SMD, short) -> FRANK:Jack (3.5mm, PJ-320D)
- J8: value PJ-320D -> SS-52100-004; footprint FRANK:Jack (3.5mm, PJ-320D) -> FRANK:USB Type A (stacked)
- JP2: value Main Jumpers -> VGA AUDIO L; footprint FRANK:SW_DS05-127-2-03BK-SMT-TR -> FRANK:Jumper (solder, 3 pins); moved to B.Cu
- Q5, Q6: value AO3400A -> BC850
- R1, R10, R11, R12, R13, R14, R15, R16, R17, R18, R19, R2, R20, R21, R22, R3, R4, R5, R6, R7, R8, R9: footprint FRANK:Resistor (0805) -> FRANK:Resistor (0603)
- R23, R25: value 330R -> 806R; footprint FRANK:Resistor (0805) -> FRANK:Resistor (0603)
- R24: value 330R -> 402R; footprint FRANK:Resistor (0805) -> FRANK:Resistor (0603)
- R26, R28: value 1K -> 402R; footprint FRANK:Resistor (0805) -> FRANK:Resistor (0603)
- R27: value 1K -> 806R; footprint FRANK:Resistor (0805) -> FRANK:Resistor (0603)
- R29, R30: value 100R -> 75R; footprint FRANK:Resistor (0805) -> FRANK:Resistor (0603)
- R31: value 22K -> 75R; footprint FRANK:Resistor (0805) -> FRANK:Resistor (0603)
- R32: value 4.7K -> 100R; footprint FRANK:Resistor (0805) -> FRANK:Resistor (0603)
- R33, R51: value 22K -> 100R; footprint FRANK:Resistor (0805) -> FRANK:Resistor (0603)
- R34: value 22K -> 2K; footprint FRANK:Resistor (0805) -> FRANK:Resistor (0603)
- R35: value 4.7K -> 2K; footprint FRANK:Resistor (0805) -> FRANK:Resistor (0603)
- R36, R48: value 22K -> 1K; footprint FRANK:Resistor (0805) -> FRANK:Resistor (0603)
- R37: value 100R -> 4.7K; footprint FRANK:Resistor (0805) -> FRANK:Resistor (0603)
- R38: value 150R -> 4.7K; footprint FRANK:Resistor (0805) -> FRANK:Resistor (0603)
- R39: value 10K -> 22K; footprint FRANK:Resistor (0805) -> FRANK:Resistor (0603)
- R40: value 10K -> 4.7K; footprint FRANK:Resistor (0805) -> FRANK:Resistor (0603)
- R41: value 27R -> 22K; footprint FRANK:Resistor (0805) -> FRANK:Resistor (0603)
- R42, R44: value 1K -> 22K; footprint FRANK:Resistor (0805) -> FRANK:Resistor (0603)
- R43: value 27R -> 4.7K; footprint FRANK:Resistor (0805) -> FRANK:Resistor (0603)
- R45: value 1K -> 100R; footprint FRANK:Resistor (0805) -> FRANK:Resistor (0603)
- R46: value 22K -> 150R; footprint FRANK:Resistor (0805) -> FRANK:Resistor (0603)
- R47, R50: value 4.7K -> 10K; footprint FRANK:Resistor (0805) -> FRANK:Resistor (0603)
- R49: value 22K -> 10K; footprint FRANK:Resistor (0805) -> FRANK:Resistor (0603)
- R52, R54: value 22R -> 27R; footprint FRANK:Resistor (0805) -> FRANK:Resistor (0603)
- R53, R55: value 22R -> 1K; footprint FRANK:Resistor (0805) -> FRANK:Resistor (0603)
- R56: value 10K -> 1K; footprint FRANK:Resistor (0805) -> FRANK:Resistor (0603)
- U10: value TS3USB221RSER -> W25Q128JVSIQ; footprint FRANK:UQFN-10 -> FRANK:SOIC-8
- U7: value W25Q128JVSIQ -> AMS1117-3.3; footprint FRANK:SOIC-8 -> FRANK:SOT-223
- U8: value RP2040 -> AMS1117-1.8; footprint FRANK:QFN 56 -> FRANK:SOT-223
- U9: value MW7211A -> MS9288A; footprint FRANK:SOP-16 -> FRANK:QFN 48
- moved H2 153.0 mm to (239.8, 48.5)
- moved C35 141.0 mm to (220.0, 60.2)
- moved C34 133.7 mm to (214.5, 60.0), turned to 90 degrees
- moved R35 132.6 mm to (230.2, 68.0)
- moved R34 132.5 mm to (230.2, 66.2)
- moved C19 131.7 mm to (239.5, 82.8)
- moved C24 131.2 mm to (235.5, 52.8), turned to 90 degrees
- moved R53 129.2 mm to (230.5, 103.0), turned to -90 degrees
- moved R36 128.2 mm to (225.9, 60.7), turned to -90 degrees
- moved R55 125.6 mm to (223.0, 87.2), turned to 90 degrees
- moved C25 125.5 mm to (233.8, 52.8), turned to 90 degrees
- moved C11 123.2 mm to (238.5, 70.8)
- moved U8 122.3 mm to (236.0, 59.5), turned to 90 degrees
- moved U10 120.9 mm to (238.2, 96.8), turned to -90 degrees
- moved C21 120.8 mm to (234.5, 68.5), turned to 180 degrees
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Connections:
- net /MS_DATA renamed /TAPE_IN
- C11 pad 1: VBUS -> /VGA/AMS_3V3A
- C12 pad 1: GND -> /VGA/B
- C12 pad 2: +3V3 -> Net-(C12-Pad2)
- C13 pad 1: /Audio Out/A_OUT -> /VGA/AMS_1V8A
- C13 pad 2: Net-(C13-Pad2) -> GND
- C14 pad 1: GND -> /VGA/AMS_1V8A
- C14 pad 2: Net-(C13-Pad2) -> GND
- C15 pad 1: GND -> /VGA/AMS_1V8
- C15 pad 2: /Tape In/G -> GND
- C16 pad 1: /ESP_IO34 -> /VGA/AMS_3V3A
- C16 pad 2: /Tape In/L -> GND
- C17 pad 1: /ESP_IO34 -> /VGA/AMS_3V3
- C17 pad 2: /Tape In/R -> GND
- C18 pad 1: Net-(U8-VREG_VOUT) -> /VGA/G
- C18 pad 2: GND -> /VGA/SOG_G
- C19 pad 1: Net-(U8-VREG_VOUT) -> VBUS
- C20 pad 1: +3V3 -> /VGA/AMS_3V3
- C21 pad 1: +3V3 -> /VGA/AMS_3V3
- C22 pad 1: +3V3 -> /VGA/R
- C22 pad 2: GND -> Net-(C22-Pad2)
- C23 pad 1: +3V3 -> VBUS
- C24 pad 1: +3V3 -> /VGA/AMS_1V8
- C25 pad 1: +3V3 -> /VGA/AMS_1V8
- C26 pad 1: +3V3 -> Net-(U9-SOG/Y)
- C26 pad 2: GND -> /VGA/SOG_G
- C27 pad 1: +3V3 -> /VGA/AMS_1V8A
- C28 pad 1: Net-(U8-VREG_VOUT) -> Net-(U9-REFQ0)
- C29 pad 1: +3V3 -> Net-(U9-REFQ0)
- C30 pad 1: +3V3 -> Net-(U9-REFQ1)
- C31 pad 1: Net-(C31-Pad1) -> Net-(U9-REFQ1)
- C32 pad 1: /RP2040/XIN -> Net-(U9-REFP)
- C33 pad 1: VBUS -> Net-(U9-REFP)
- C34 pad 1: VBUS -> Net-(U9-XTO)
- C35 pad 1: VBUS -> Net-(U9-XTI)
- C36 pad 1: VBUS -> /VGA/ALIN
- C36 pad 2: GND -> /VGA_AIN
- C37 pad 1: GND -> /VGA/ARIN
- C37 pad 2: +3V3 -> /VGA_AIN
- D1 pad 1: /ESP_IO34 -> Net-(D1-K)
- D1 pad 2: GND -> VBUS
- J1 pad 11: Net-(S4-B) -> VBUS
- J1 pad 2: Net-(S4-B) -> VBUS
- J3 pad 1: /GPIO2 -> /KB_DATA
- J3 pad 2: /GPIO3 -> unconnected-(J3-Pad2)
- J3 pad 3: /GPIO4 -> GND
- J3 pad 4: /GPIO5 -> VBUS
- J3 pad 5: VBUS -> /KB_CLK
- J3 pad 6: /GPIO6 -> unconnected-(J3-Pad6)
- J4 pad 1: /KB_DATA -> /VGA/TMDS_D2+
- J4 pad 2: unconnected-(J4-Pad2) -> GND
- J4 pad 3: GND -> /VGA/TMDS_D2-
- J4 pad 4: VBUS -> /VGA/TMDS_D1+
- J4 pad 5: /KB_CLK -> GND
- J4 pad 6: unconnected-(J4-Pad6) -> /VGA/TMDS_D1-
- JP2 pad 1: /SN74_S -> /ESP_IO25
- JP2 pad 2: /UMSW -> /VGA_AIN
- JP2 pad 3: /AUDIO_IN -> /A_OUT
- Q5 pad 1: Net-(Q5-G) -> Net-(Q5-B)
- Q5 pad 2: /MS_DATA_3V -> GND
- Q6 pad 2: /KB_CLK_3V -> GND
- Q6 pad 3: /KB_CLK -> Net-(D2-A)
- R2 pad 2: GND -> +3V3
- R23 pad 1: /ESP_IO22 -> /ESP_IO4
- R23 pad 2: Net-(J5-Pad1) -> Net-(C12-Pad2)
- R24 pad 1: /ESP_IO19 -> /ESP_IO5
- R24 pad 2: Net-(J5-Pad2) -> Net-(C12-Pad2)
- R25 pad 1: /ESP_IO5 -> /ESP_IO18
- R25 pad 2: Net-(J5-Pad3) -> /VGA/SOG_G
- R26 pad 1: /ESP_IO21 -> /ESP_IO19
- R26 pad 2: Net-(J5-Pad1) -> /VGA/SOG_G
- R27 pad 1: /ESP_IO18 -> /ESP_IO21
- R27 pad 2: Net-(J5-Pad2) -> Net-(C22-Pad2)
- R28 pad 1: /ESP_IO4 -> /ESP_IO22
- R28 pad 2: Net-(J5-Pad3) -> Net-(C22-Pad2)
- R29 pad 1: Net-(J5-Pad13) -> Net-(C22-Pad2)
- R29 pad 2: /ESP_IO23 -> GND
- R3 pad 2: GND -> +3V3
- R30 pad 1: Net-(J5-Pad14) -> /VGA/SOG_G
- R30 pad 2: /ESP_IO15 -> GND
- R31 pad 1: +3V3 -> Net-(C12-Pad2)
- R31 pad 2: /KB_DATA_3V -> GND
- R32 pad 1: +3V3 -> /ESP_IO23
- R32 pad 2: Net-(Q3-G) -> Net-(U9-HSIN)
- R33 pad 1: VBUS -> /ESP_IO15
- R33 pad 2: /KB_DATA -> Net-(U9-VSIN)
- R34 pad 1: +3V3 -> /VGA/DCCSCL
- R34 pad 2: /MS_CLK_3V -> VBUS
- R35 pad 1: +3V3 -> /VGA/DDCSDA
- R35 pad 2: Net-(Q4-G) -> VBUS
- R36 pad 1: VBUS -> GND
- R36 pad 2: /MS_CLK -> Net-(U9-SWREF1k)
- R37 pad 1: /AUDIO_IN -> /VGA/SCL
- R37 pad 2: Net-(C13-Pad2) -> VBUS
- R38 pad 1: GND -> /VGA/SDA
- R38 pad 2: Net-(C13-Pad2) -> VBUS
- R39 pad 1: /ESP_IO34 -> +3V3
- R39 pad 2: GND -> /KB_DATA_3V
- R4 pad 2: GND -> +3V3
- R40 pad 1: /ESP_IO34 -> +3V3
- R40 pad 2: VBUS -> Net-(Q3-G)
- R41 pad 1: /RP_D+ -> VBUS
- R41 pad 2: Net-(U8-USB_DP) -> /KB_DATA
- R42 pad 1: /RP2040/QSPI_SS -> +3V3
- R42 pad 2: Net-(R42-Pad2) -> /MS_CLK_3V
- R43 pad 1: /RP_D- -> +3V3
- R43 pad 2: Net-(U8-USB_DM) -> Net-(Q4-G)
- R44 pad 1: /RP2040/XOUT -> VBUS
- R44 pad 2: Net-(C31-Pad1) -> /MS_CLK
- R45 pad 1: Net-(LD4-A) -> /ESP_IO25
- R45 pad 2: /RP2040/GPIO25 -> Net-(C39-Pad2)
- R46 pad 1: +3V3 -> GND
- R46 pad 2: /MS_DATA_3V -> Net-(C39-Pad2)
- R47 pad 2: Net-(Q5-G) -> Net-(D2-A)
- R48 pad 1: VBUS -> +3V3
- R49 pad 1: +3V3 -> Net-(D2-A)
- R49 pad 2: /KB_CLK_3V -> Net-(Q5-B)
- R5 pad 2: GND -> +3V3
- R50 pad 1: +3V3 -> Net-(C42-Pad2)
- R51 pad 1: VBUS -> Net-(AJ1-PadT)
- R51 pad 2: /KB_CLK -> GND
- R52 pad 1: /USB Hub/D1+ -> /RP_D+
- R53 pad 1: /USB Hub/D2+ -> /RP2040/QSPI_SS
- R53 pad 2: Net-(J11-D2+) -> Net-(R53-Pad2)
- R54 pad 1: /USB Hub/D1- -> /RP_D-
- R55 pad 1: /USB Hub/D2- -> /RP2040/XOUT
- R55 pad 2: Net-(J11-D2-) -> Net-(C56-Pad1)
- R56 pad 1: +3V3 -> Net-(LD4-A)
- R56 pad 2: /UMSW -> /RP2040/GPIO25
- S5 pad 1: Net-(R42-Pad2) -> Net-(R53-Pad2)
- U10 pad 1: /TC2_D+ -> /RP2040/QSPI_SS
- U10 pad 2: /TC2_D- -> /RP2040/QSPI_SD1
- U10 pad 3: /UH_D+ -> /RP2040/QSPI_SD2
- U10 pad 4: /UH_D- -> GND
- U10 pad 5: GND -> /RP2040/QSPI_SD0
- U10 pad 6: GND -> /RP2040/QSPI_SCLK
- U10 pad 7: /RP_D- -> /RP2040/QSPI_SD3
- U10 pad 8: /RP_D+ -> +3V3
- U7 pad 1: /RP2040/QSPI_SS -> GND
- U7 pad 2: /RP2040/QSPI_SD1 -> /VGA/AMS_3V3
- U7 pad 3: /RP2040/QSPI_SD2 -> VBUS
- U8 pad 1: +3V3 -> GND
- U8 pad 2: /GPIO0 -> /VGA/AMS_1V8
- U8 pad 3: /GPIO1 -> VBUS
- U9 pad 1: /USB Hub/D1- -> /VGA/AMS_1V8A
- U9 pad 10: /UH_D- -> /VGA/DCCSCL
- U9 pad 11: /UH_D+ -> /VGA/AMS_3V3
- U9 pad 12: Net-(U9-VD3) -> /VGA/AMS_3V3A
- U9 pad 13: VBUS -> Net-(U9-SWREF1k)
- U9 pad 14: Net-(U9-VD3) -> /VGA/TMDS_CLK-
- U9 pad 15: GND -> /VGA/TMDS_CLK+
- U9 pad 16: GND -> /VGA/AMS_1V8
- U9 pad 2: /USB Hub/D1+ -> GND
- U9 pad 3: /USB Hub/D2- -> unconnected-(U9-??-Pad3)
- U9 pad 4: /USB Hub/D2+ -> unconnected-(U9-MCUSEL-Pad4)
- U9 pad 5: unconnected-(U9-DM2-Pad5) -> /VGA/AMS_3V3
- U9 pad 6: unconnected-(U9-DP2-Pad6) -> GND
- U9 pad 7: unconnected-(U9-DM3-Pad7) -> /VGA/AMS_1V8
- U9 pad 8: unconnected-(U9-DP3-Pad8) -> /VGA/HPDT
- U9 pad 9: unconnected-(U9-LED-Pad9) -> /VGA/DDCSDA
- Y1 pad 3: Net-(C31-Pad1) -> Net-(C56-Pad1)
Routing:
- net VBUS: track 379.3 -> 2.68 mm, vias 11 -> 0
- net +3V3: track 266.6 -> 0.00 mm, vias 24 -> 1
- net /ESP_IO27: track 98.6 -> 0.00 mm, vias 2 -> 0
- net /ESP_IO33: track 98.3 -> 0.00 mm, vias 2 -> 0
- net /ESP_IO32: track 96.3 -> 0.00 mm, vias 2 -> 0
- net /ESP_IO26: track 89.4 -> 0.00 mm, vias 2 -> 0
- net /ESP_EN: track 83.7 -> 0.00 mm, vias 4 -> 0
- net /VGA/AMS_1V8A: track 0.00 -> 70.9 mm, vias 0 -> 4
- net /Audio Out/A_OUT: track 67.9 -> 0.00 mm, vias 4 -> 0
- net /GPIO2: track 65.5 -> 0.00 mm, vias 1 -> 0
- net /GPIO12: track 59.8 -> 0.00 mm, vias 2 -> 0
- net /MS_DATA_3V: track 57.1 -> 0.00 mm, vias 4 -> 0
- net /VGA/AMS_3V3: track 0.00 -> 55.6 mm, vias 0 -> 6
- net /GPIO11: track 54.4 -> 0.00 mm, vias 2 -> 0
- net /SN74_S: track 51.5 -> 0.00 mm, vias 7 -> 0
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- added copper zone on In2.Cu, net +3V3
- added copper zone on F.Cu, net /VGA/AMS_1V8
- added copper zone on In2.Cu, net /VGA/AMS_1V8
- added copper zone on F.Cu, net /VGA/AMS_3V3
- added copper zone on In2.Cu, net /VGA/AMS_3V3
- added copper zone on F.Cu, net /VGA/AMS_3V3A
- added copper zone on In2.Cu, net /VGA/AMS_3V3A
- added copper zone on In1.Cu, net GND
- removed copper zone on F.Cu, net +3V3
- removed copper zone on B.Cu, net GND
- removed copper zone on B.Cu, net Net-(U8-VREG_VOUT)
- removed copper zone on F.Cu, net Net-(U8-VREG_VOUT)
Other:
- board size 90.9 x 61.9 mm -> 99.5 x 65 mm
- copper layers 2 -> 4
- board text removed: "AUDIO OUT"
- board text removed: "BTN 36"
- board text removed: "DH"
- board text removed: "KEYBOARD"
- board text removed: "MOUSE"
- board text removed: "PU"
- board text removed: "PWR/ESP"
- board text removed: "RESET"
- board text removed: "RP"
- board text removed: "RP BOOT"
- board text removed: "RP RESET"
- board text removed: "TAPE IN"
- board text removed: "TI"
- board text removed: "VGA VIDEO"
- board text removed: "rh1.tech"

Commit message: 1.05 WIP
Parts:
- moved C4 51.1 mm to (149.2, 85.2), turned to 180 degrees
- moved R65 7.50 mm to (185.8, 92.2), turned to -90 degrees
- moved R66 7.25 mm to (188.5, 92.2), turned to -90 degrees
- moved R63 5.75 mm to (193.8, 92.2), turned to -90 degrees
- moved R53 4.23 mm to (232.0, 99.0), turned to 0 degrees
- moved R22 2.61 mm to (198.8, 109.2), turned to 180 degrees
- moved JP3 1.80 mm to (190.7, 84.7)
- moved C38 1.55 mm to (146.2, 102.5)
- moved J5 1.55 mm to (146.3, 93.8)
- moved U4 0.39 mm to (155.2, 94.4)
- moved R64 0.33 mm to (191.1, 92.2), turned to -90 degrees
- turned R13 to -90 degrees
Routing:
- net VBUS: track 2.68 -> 317.8 mm, vias 0 -> 25
- net /GPIO11: track 0.00 -> 81.8 mm, vias 0 -> 2
- net /GPIO12: track 0.00 -> 77.7 mm, vias 0 -> 2
- net /GPIO14: track 0.00 -> 70.6 mm, vias 0 -> 2
- net /GPIO15: track 0.00 -> 69.0 mm, vias 0 -> 2
- net /UH_D-: track 0.00 -> 49.3 mm
- net /ESP_IO0: track 0.00 -> 49.0 mm
- net /UH_D+: track 0.00 -> 44.2 mm
- net /ESP_EN: track 0.00 -> 38.1 mm
- net /TC2_D-: track 0.00 -> 33.1 mm
- net /TC2_D+: track 0.00 -> 31.8 mm
- net Net-(AJ1-PadT): track 0.00 -> 30.1 mm
- net /MS_CLK: track 0.00 -> 26.4 mm
- net /RP2040/QSPI_SS: track 0.00 -> 22.9 mm
- net /RP2040/QSPI_SD2: track 0.00 -> 22.5 mm
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- added copper zone on F.Cu, net +3V3
- added copper zone on F.Cu, net Net-(U11-VREG_VOUT)

Commit message: Update echo.kicad_pcb
Parts:
- moved C41 4.01 mm to (181.2, 92.8), turned to 0 degrees
Routing:
- net /ESP_IO2: track 0.00 -> 118.9 mm, vias 0 -> 2
- net /ESP_IO1: track 18.3 -> 123.6 mm
- net /A_OUT: track 2.93 -> 80.9 mm, vias 0 -> 1
- net /ESP_IO3: track 10.5 -> 87.9 mm, vias 0 -> 2
- net /ESP_IO12: track 0.00 -> 70.1 mm, vias 0 -> 2
- net /ESP_IO25: track 0.00 -> 60.0 mm, vias 0 -> 3
- net /ESP_IO13: track 0.00 -> 56.7 mm, vias 0 -> 2
- net /ESP_IO14: track 0.00 -> 51.0 mm, vias 0 -> 2
- net /UMSW: track 3.91 -> 53.4 mm, vias 0 -> 2
- net /ESP_EN: track 38.1 -> 85.3 mm
- net /ESP_IO19: track 0.00 -> 43.9 mm, vias 0 -> 2
- net /ESP_IO21: track 0.00 -> 41.6 mm, vias 0 -> 2
- net /ESP_IO36: track 5.36 -> 46.7 mm, vias 0 -> 2
- net /ESP_IO22: track 0.00 -> 36.8 mm, vias 0 -> 2
- net /ESP_IO18: track 0.00 -> 36.6 mm, vias 0 -> 2
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