File: gamepad.kicad_sch (KiCad schematic)
At the start: 2 parts, among them J2 D-SUB 9 Male

Commit message: HW Rev 1.03
Parts:
- renumbered C10 to C9
Changed lines of the file:
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@@
 	(title_block
 		(title "${NAME}")
-		(date "2025-06-23")
+		(date "2025-07-20")
 		(rev "${VERSION}")
 		(company "Mikhail Matveev")
@@
 		(on_board yes)
 		(dnp no)
-		(property "Reference" "C10"
+		(property "Reference" "C9"
 			(at 137.668 97.79 0)
 			(effects
@@
 			(project "echo"
 				(path "/8c0b3d8b-46d3-4173-ab1e-a61765f77d61/3f0a2a41-81d6-4e1a-97c7-801d84353ad4"
-					(reference "C10")
+					(reference "C9")
 					(unit 1)
 				)

Commit message: WIP
Parts:
- renumbered C9 to C10, J2 to J3
Changed lines of the file:
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@@
 	(title_block
 		(title "${NAME}")
-		(date "2025-07-20")
+		(date "2025-08-08")
 		(rev "${VERSION}")
 		(company "Mikhail Matveev")
@@
 		(on_board yes)
 		(dnp no)
-		(property "Reference" "#PWR036"
+		(property "Reference" "#PWR048"
 			(at 137.16 90.17 0)
 			(effects
@@
 			(project "echo"
 				(path "/8c0b3d8b-46d3-4173-ab1e-a61765f77d61/3f0a2a41-81d6-4e1a-97c7-801d84353ad4"
-					(reference "#PWR036")
+					(reference "#PWR048")
 					(unit 1)
 				)
@@
 		(on_board yes)
 		(dnp no)
-		(property "Reference" "J2"
+		(property "Reference" "J3"
 			(at 175.26 87.63 0)
 			(effects
@@
 			(project "echo"
 				(path "/8c0b3d8b-46d3-4173-ab1e-a61765f77d61/3f0a2a41-81d6-4e1a-97c7-801d84353ad4"
-					(reference "J2")
+					(reference "J3")
 					(unit 1)
 				)
@@
 		(on_board yes)
 		(dnp no)
-		(property "Reference" "#PWR037"
+		(property "Reference" "#PWR049"
 			(at 147.32 97.79 0)
 			(effects
@@
 			(project "echo"
 				(path "/8c0b3d8b-46d3-4173-ab1e-a61765f77d61/3f0a2a41-81d6-4e1a-97c7-801d84353ad4"
-					(reference "#PWR037")
+					(reference "#PWR049")
 					(unit 1)
 				)
@@
 		(on_board yes)
 		(dnp no)
-		(property "Reference" "C9"
+		(property "Reference" "C10"
 			(at 137.668 97.79 0)
 			(effects
@@
 			(project "echo"
 				(path "/8c0b3d8b-46d3-4173-ab1e-a61765f77d61/3f0a2a41-81d6-4e1a-97c7-801d84353ad4"
-					(reference "C9")
+					(reference "C10")
 					(unit 1)
 				)
@@
 		(on_board yes)
 		(dnp no)
-		(property "Reference" "#PWR038"
+		(property "Reference" "#PWR050"
 			(at 137.16 111.76 0)
 			(effects
@@
 			(project "echo"
 				(path "/8c0b3d8b-46d3-4173-ab1e-a61765f77d61/3f0a2a41-81d6-4e1a-97c7-801d84353ad4"
-					(reference "#PWR038")
+					(reference "#PWR050")
 					(unit 1)
 				)
