File: echo.kicad_sch (KiCad schematic)
At the start: 4 parts

Commit message: Work-in-progress
Parts:
- added C1: 100n, FRANK:Capacitor (0805), symbol Device:C
- added C2: 1u, FRANK:Capacitor (0805), symbol Device:C
- added J1: Input Control, FRANK:Pin Header (1x02), symbol Connector:Conn_01x02_Pin
- added R1, R2: 10K, FRANK:Resistor (0805), symbol Device:R
- added S1: Reset, FRANK:Button (SMD, 3x3mm, 1-1), symbol Switch:SW_Push
- added U1: SN74CBT3257CDR, FRANK:SOP-16, symbol SN74CBT3257CDR:SN74CBT3257CDR
Connections:
- net ESP_EN: now also C2.1, R1.1, S1.2
- net ESP_IO26: now also U1.9 (3A)
- net ESP_IO27: now also U1.12 (4A)
- net ESP_IO32: now also U1.7 (2A)
- net ESP_IO33: now also U1.4 (1A)
- net ZGPIO11: now also U1.6 (2B2)
- net ZGPIO12: now also U1.3 (1B2)
- net ZGPIO14: now also U1.13 (4B2)
- net ZGPIO15: now also U1.10 (3B2)
- new net +3V3: R1.2
- new net GND: C1.1, C2.2, R2.1, S1.1, U1.15 (~{OE}), U1.8 (GND)
- new net KB_CLK_3V: U1.2 (1B1)
- new net KB_DATA_3V: U1.5 (2B1)
- new net MS_CLK_3V: U1.11 (3B1)
- new net MS_DATA_3V: U1.14 (4B1)
- new net SN74_S: J1.2 (Pin_2), R2.2, U1.1 (S)
- new net VCC: C1.2, J1.1 (Pin_1), U1.16 (VCC)
Other:
- sheet ESP32-WROOM-32E renamed ESP32
- added sheet PSRAM (psram.kicad_sch)
- sheet ESP32: file ESP32-WROOM-32E.kicad_sch -> esp32.kicad_sch
- sheet ESP32 ports: added SCK_CLK, SCS_CMD, SDI_SD1, SDO_SD0, SHD_SD2, SWP_SD3; removed none
- sheet PS2 ports: added none; removed KB_CLK, KB_DATA, MS_CLK, MS_DATA
- sheet RP2040-Zero ports: added none; removed ZVBUS

Commit message: HW Revision 1.00
Parts:
- renumbered J1 to JP2
Changed lines of the file:
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@@
 		(dnp no)
 		(fields_autoplaced yes)
-		(property "Reference" "J1"
+		(property "Reference" "JP2"
 			(at 234.315 149.86 0)
 			(effects
@@
 			(project ""
 				(path "/8c0b3d8b-46d3-4173-ab1e-a61765f77d61"
-					(reference "J1")
+					(reference "JP2")
 					(unit 1)
 				)

Commit message: 1.01 WIP
Parts:
- removed JP2: Input Control, FRANK:Pin Header (1x02), symbol Connector:Conn_01x02_Pin
- added JP1: Main Jumpers, FRANK:SW_DS05-127-2-03BK-SMT-TR, symbol Switch:SW_DIP_x03
- S1: footprint FRANK:Button (SMD, 3x3mm, 1-1) -> FRANK:TACT-SIDE-4623
Connections:
- net GND: now also JP1.5
- net SN74_S: now also JP1.1
- net VCC renamed VBUS
- net VBUS: now also JP1.6
- net ZGPIO11 renamed GPIO11
- net ZGPIO12 renamed GPIO12
- net ZGPIO14 renamed GPIO14
- net ZGPIO15 renamed GPIO15
- new net ESP_IO34: JP1.4
- new net GPIO0: JP1.2
- new net LOAD_IN: JP1.3
- no-connect marks 24 -> 20
Other:
- sheet PS2 renamed PS2 KB
- removed sheet PSRAM
- removed sheet RP2040-Zero
- removed sheet USB A Stacked
- added sheet Gamepad 1 (gamepad.kicad_sch)
- added sheet Gamepad 2 (gamepad.kicad_sch)
- added sheet PS2 MS (ps2.kicad_sch)
- added sheet RP2040 (rp2040.kicad_sch)
- added sheet Tape In (tape.kicad_sch)
- added sheet USB A (usba.kicad_sch)
- sheet ESP32 ports: added none; removed IO16, IO17, SCK_CLK, SCS_CMD, SDI_SD1, SDO_SD0, SHD_SD2, SWP_SD3
- sheet PS2 KB ports: added CLK_3V, DATA_3V; removed KB_CLK_3V, KB_DATA_3V, MS_CLK_3V, MS_DATA_3V

Commit message: Echo HW Rev 1.01
Changed lines of the file:
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@@
 	(title_block
 		(title "${NAME}")
-		(date "2025-04-30")
+		(date "2025-05-24")
 		(rev "${VERSION}")
 		(company "Mikhail Matveev")
@@
 			(color 0 0 0 0.0000)
 		)
-		(property "Sheetname" "Gamepad 2"
+		(property "Sheetname" "Gamepad 1"
 			(at 86.36 137.7184 0)
 			(effects
@@
 			(color 0 0 0 0.0000)
 		)
-		(property "Sheetname" "Gamepad 1"
+		(property "Sheetname" "Gamepad 2"
 			(at 86.36 111.0484 0)
 			(effects

Commit message: Minor fixes
Parts:
- added C3: 1u, FRANK:Capacitor (0805), symbol Device:C
- added JP1: ESP-RP RST, FRANK:Jumper (solder), symbol Jumper:SolderJumper_2_Open
- added R3: 10K, FRANK:Resistor (0805), symbol Device:R
- added S1: RP Reset, FRANK:TACT-SIDE-4623, symbol Switch:SW_Push
- added S3: ESP Ctrl, FRANK:TACT-SIDE-4623, symbol Switch:SW_Push
- S2: renamed from S1; value Reset -> ESP Reset; AliExpress (none) -> https://www.aliexpress.com/item/1005007359248990.html
- renumbered JP1 to JP2, R2 to R1, R1 to R2
Connections:
- net +3V3: now also R3.2
- net ESP_EN: now also JP1.2 (B)
- net ESP_IO34: no longer JP2.4
- net GND: now also JP2.4, C3.2, S1.2, S3.1
- net GPIO0: no longer JP2.2
- net GPIO16: now also JP1.1 (A)
- net RUN: now also S1.1
- net LOAD_IN renamed UMSW2
- new net ESP_IO36: C3.1, R3.1, S3.2
- new net UMSW1: JP2.2
- no-connect marks 20 -> 30
Other:
- sheet Gamepad 1 renamed Gamepad
- removed sheet Gamepad 2
- added sheet Shifter1 (level_shifter.kicad_sch)
- added sheet Shifter2 (level_shifter.kicad_sch)
- added sheet Shifter3 (level_shifter.kicad_sch)
- added sheet Shifter4 (level_shifter.kicad_sch)
- added sheet USB Hub (usb_hub.kicad_sch)
- added sheet USB Multiplexer 1 (usb_multiplexer.kicad_sch)
- added sheet USB Multiplexer 2 (usb_multiplexer.kicad_sch)
- sheet ESP32 ports: added IO36, IO39; removed SENSOR_VN, SENSOR_VP
- sheet PS2 KB ports: added CLK, DATA; removed CLK_3V, DATA_3V
- sheet PS2 MS ports: added CLK, DATA; removed CLK_3V, DATA_3V
- sheet USB A: file usba.kicad_sch -> usbstack.kicad_sch
- sheet USB A ports: added D1+, D1-, D2+, D2-; removed D+, D-
- moved on the sheet: C1, C2, JP2, R1, R2, S2, U1

Commit message: WIP
Parts:
- added R2, R3, R4, R5: 10K, FRANK:Resistor (0805), symbol Device:R
- S1: footprint FRANK:TACT-SIDE-4623 -> FRANK:Button (SMD, 3x3mm, 1-1)
- renumbered R2 to R6, R3 to R7
Connections:
- net ESP_IO25: now also JP2.4
- net GND: now also R2.2, R3.2, R4.2, R5.2; no longer JP2.4
- net GPIO11: now also R2.1
- net GPIO12: now also R3.1
- net GPIO14: now also R4.1
- net GPIO15: now also R5.1
- net UMSW1 renamed UMSW
- net UMSW2 renamed AUDIO_IN
- no-connect marks 30 -> 26
Other:
- sheet USB Multiplexer 1 renamed USB Multiplexer
- removed sheet USB A
- removed sheet USB Multiplexer 2
- sheet Power ports: added D1+, D1-, D2+, D2-; removed D+, D-
- sheet USB Hub ports: added none; removed DM1, DM2, DM3, DM4, DP1, DP2, DP3, DP4
- moved on the sheet: C1, C2, C3, H1, H2, H3, H4, JP1, JP2, R1, R6, R7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

Commit message: Rev 1.05 WIP
Parts:
- removed JP1: ESP-RP RST, FRANK:Jumper (solder), symbol Jumper:SolderJumper_2_Open
- added JP2: VGA AUDIO L, FRANK:Jumper (solder, 3 pins), symbol Connector:Conn_01x03_Pin
- C1, C2, C3: footprint FRANK:Capacitor (0805) -> FRANK:Capacitor (0603)
- R1, R2, R3, R4, R5, R6, R7: footprint FRANK:Resistor (0805) -> FRANK:Resistor (0603)
- renumbered JP2 to JP3
Connections:
- net +3V3: now also R2.2, R3.2, R4.2, R5.2
- net ESP_IO25: now also JP2.1 (Pin_1); no longer JP3.4
- net ESP_IO34: now also JP3.4
- net GND: no longer R2.2, R3.2, R4.2, R5.2
- net AUDIO_IN renamed TAPE_IN
- new net A_OUT: JP2.3 (Pin_3)
- new net VGA_AIN: JP2.2 (Pin_2)
- no-connect marks 26 -> 33
Other:
- removed sheet Gamepad
- sheet Audio Out ports: added A_OUT; removed none
- sheet VGA ports: added AUDIO_IN_L, AUDIO_IN_R; removed none
- moved on the sheet: C2, C3, JP3, R6, R7, S2, S3
