File: echo.kicad_sch (KiCad schematic)
At the start: 20 parts, among them U1 SN74CBT3257CDR

Commit message: 1.05 WIP
Connections:
- no-connect marks 33 -> 34
Changed lines of the file:
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@@
+	)
+	(no_connect
+		(at 104.14 72.39)
 	)
 	(no_connect

Commit message: HW 1.06 WIP
Parts:
- renumbered C2 to C1, C1 to C2, JP3 to JP1, R6 to R2, R7 to R3, R2 to R4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
Connections:
- no-connect marks 34 -> 35
Other:
- sheet ESP32 ports: added IO16, IO17, IO37, IO38; removed none
