File: power.kicad_sch (KiCad schematic)
At the start: 10 parts, among them J1 USB4215-03-A, U2 NCP1117 3.3, U4 USBLC6-2SC6

Commit message: Work-in-progress
Parts:
- added R8, R9: 22R, FRANK:Resistor (0805), symbol Device:R
- C7: LCSC C1713 -> (none)
- C8: renamed from C6; LCSC C1713 -> (none)
- J2: renamed from J1; LCSC C165948 -> (none)
- LD3: value Green -> Power
- R10: renamed from R5; LCSC C3152211 -> (none)
- R11: renamed from R6; LCSC C3152182 -> (none)
- R12: renamed from R4; LCSC C17513 -> (none)
- R7: renamed from R3; LCSC C3152211 -> (none)
- U3: renamed from U2; LCSC C5346136 -> (none)
- U4: footprint Package_TO_SOT_SMD:SOT-23-6 -> FRANK:SOT-23-6
Connections:
- net at J2.5 (DN2), J2.7 (DN1): now also R8.2; no longer U4.1 (I/O1)
- net at J2.6 (DP1), J2.8 (DP2): now also R9.2; no longer U4.3 (I/O2)
- new net: R8.1, U4.1 (I/O1)
- new net: R9.1, U4.3 (I/O2)
Other:
- moved on the sheet: C7, C8, U3, U4

Commit message: 1.01 WIP
Parts:
- renumbered C7 to C5, C8 to C6, J2 to J1
Connections:
- net VCC is gone; now on net VBUS: U4.5 (VBUS)
Changed lines of the file:
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@@
 		(on_board yes)
 		(dnp no)
-		(property "Reference" "#PWR024"
+		(property "Reference" "#PWR023"
 			(at 171.45 104.14 0)
 			(effects
@@
 			(project "frank2"
 				(path "/8c0b3d8b-46d3-4173-ab1e-a61765f77d61/4ea27ee4-1edc-4e10-ab5a-91b9933087c0"
-					(reference "#PWR024")
+					(reference "#PWR023")
 					(unit 1)
 				)
@@
 		(dnp no)
 		(fields_autoplaced yes)
-		(property "Reference" "#PWR015"
+		(property "Reference" "#PWR014"
 			(at 135.89 77.47 0)
 			(effects
@@
 			(project ""
 				(path "/8c0b3d8b-46d3-4173-ab1e-a61765f77d61/4ea27ee4-1edc-4e10-ab5a-91b9933087c0"
-					(reference "#PWR015")
+					(reference "#PWR014")
 					(unit 1)
 				)
@@
 		(on_board yes)
 		(dnp no)
-		(property "Reference" "#PWR022"
+		(property "Reference" "#PWR021"
 			(at 123.19 97.79 0)
 			(effects
@@
 			(project "frank2"
 				(path "/8c0b3d8b-46d3-4173-ab1e-a61765f77d61/4ea27ee4-1edc-4e10-ab5a-91b9933087c0"
-					(reference "#PWR022")
+					(reference "#PWR021")
 					(unit 1)
 				)
@@
 		(dnp no)
 		(fields_autoplaced yes)
-		(property "Reference" "#PWR026"
+		(property "Reference" "#PWR025"
 			(at 175.26 119.38 0)
 			(effects
@@
 			(project "frank2"
 				(path "/8c0b3d8b-46d3-4173-ab1e-a61765f77d61/4ea27ee4-1edc-4e10-ab5a-91b9933087c0"
-					(reference "#PWR026")
+					(reference "#PWR025")
 					(unit 1)
 				)
@@
 		(dnp no)
 		(fields_autoplaced yes)
-		(property "Reference" "#PWR023"
+		(property "Reference" "#PWR022"
 			(at 148.59 104.14 0)
 			(effects
@@
 			(project "echo"
 				(path "/8c0b3d8b-46d3-4173-ab1e-a61765f77d61/4ea27ee4-1edc-4e10-ab5a-91b9933087c0"
-					(reference "#PWR023")
+					(reference "#PWR022")
 					(unit 1)
 				)
@@
 		(on_board yes)
 		(dnp no)
-		(property "Reference" "C7"
+		(property "Reference" "C5"
 			(at 208.661 81.3816 0)
 			(effects
@@
 			(project "frank2"
 				(path "/8c0b3d8b-46d3-4173-ab1e-a61765f77d61/4ea27ee4-1edc-4e10-ab5a-91b9933087c0"
-					(reference "C7")
+					(reference "C5")
 					(unit 1)
 				)
@@
 		(on_board yes)
 		(dnp no)
-		(property "Reference" "#PWR025"
+		(property "Reference" "#PWR024"
 			(at 125.73 102.87 0)
 			(effects
@@
 			(project "frank_rm2-2350A"
 				(path "/8c0b3d8b-46d3-4173-ab1e-a61765f77d61/4ea27ee4-1edc-4e10-ab5a-91b9933087c0"
-					(reference "#PWR025")
+					(reference "#PWR024")
 					(unit 1)
 				)
@@
 		(on_board yes)
 		(dnp no)
-		(property "Reference" "J2"
+		(property "Reference" "J1"
 			(at 102.87 78.74 0)
 			(effects
@@
 			(project "frank2"
 				(path "/8c0b3d8b-46d3-4173-ab1e-a61765f77d61/4ea27ee4-1edc-4e10-ab5a-91b9933087c0"
-					(reference "J2")
+					(reference "J1")
+					(unit 1)
+				)
+			)
+		)
+	)
+	(symbol
+		(lib_id "power:VBUS")
+		(at 148.59 82.55 90)
+		(unit 1)
+		(exclude_from_sim no)
+		(in_bom yes)
+		(on_board yes)
+		(dnp no)
+		(fields_autoplaced yes)
+		(property "Reference" "#PWR018"
+			(at 152.4 82.55 0)
+			(effects
+				(font
+					(size 1.27 1.27)
+				)
+				(hide yes)
+			)
+		)
+		(property "Value" "VBUS"
+			(at 144.78 82.5499 90)
+			(effects
+				(font
+					(size 1.27 1.27)
+				)
+				(justify left)
+			)
+		)
+		(property "Footprint" ""
+			(at 148.59 82.55 0)
+			(effects
+				(font
+					(size 1.27 1.27)
+				)
+				(hide yes)
+			)
+		)
+		(property "Datasheet" ""
+			(at 148.59 82.55 0)
+			(effects
+				(font
+					(size 1.27 1.27)
+				)
+				(hide yes)
+			)
+		)
+		(property "Description" "Power symbol creates a global label with name \"VBUS\""
+			(at 148.59 82.55 0)
+			(effects
+				(font
+					(size 1.27 1.27)
+				)
+				(hide yes)
+			)
+		)
+		(pin "1"
+		)
+		(instances
+			(project ""
+				(path "/8c0b3d8b-46d3-4173-ab1e-a61765f77d61/4ea27ee4-1edc-4e10-ab5a-91b9933087c0"
+					(reference "#PWR018")
 					(unit 1)
 				)
@@
 		(on_board yes)
 		(dnp no)
-		(property "Reference" "C8"
+		(property "Reference" "C6"
 			(at 174.371 82.6516 0)
 			(effects
@@
 			(project "frank2"
 				(path "/8c0b3d8b-46d3-4173-ab1e-a61765f77d61/4ea27ee4-1edc-4e10-ab5a-91b9933087c0"
-					(reference "C8")
+					(reference "C6")
 					(unit 1)
 				)
@@
 		(on_board yes)
 		(dnp no)
-		(property "Reference" "#PWR018"
+		(property "Reference" "#PWR017"
 			(at 123.19 82.55 0)
 			(effects
@@
 			(project "frank2"
 				(path "/8c0b3d8b-46d3-4173-ab1e-a61765f77d61/4ea27ee4-1edc-4e10-ab5a-91b9933087c0"
-					(reference "#PWR018")
+					(reference "#PWR017")
 					(unit 1)
 				)
@@
 		(on_board yes)
 		(dnp no)
-		(property "Reference" "#PWR021"
+		(property "Reference" "#PWR020"
 			(at 205.74 93.98 0)
 			(effects
@@
 			(project "frank2"
 				(path "/8c0b3d8b-46d3-4173-ab1e-a61765f77d61/4ea27ee4-1edc-4e10-ab5a-91b9933087c0"
-					(reference "#PWR021")
-					(unit 1)
-				)
-			)
-		)
-	)
-	(symbol
-		(lib_id "power:VCC")
-		(at 148.59 82.55 90)
-		(unit 1)
-		(exclude_from_sim no)
-		(in_bom yes)
-		(on_board yes)
-		(dnp no)
-		(fields_autoplaced yes)
-		(property "Reference" "#PWR019"
-			(at 152.4 82.55 0)
-			(effects
-				(font
-					(size 1.27 1.27)
-				)
-				(hide yes)
-			)
-		)
-		(property "Value" "VCC"
-			(at 144.78 82.5499 90)
-			(effects
-				(font
-					(size 1.27 1.27)
-				)
-				(justify left)
-			)
-		)
-		(property "Footprint" ""
-			(at 148.59 82.55 0)
-			(effects
-				(font
-					(size 1.27 1.27)
-				)
-				(hide yes)
-			)
-		)
-		(property "Datasheet" ""
-			(at 148.59 82.55 0)
-			(effects
-				(font
-					(size 1.27 1.27)
-				)
-				(hide yes)
-			)
-		)
-		(property "Description" "Power symbol creates a global label with name \"VCC\""
-			(at 148.59 82.55 0)
-			(effects
-				(font
-					(size 1.27 1.27)
-				)
-				(hide yes)
-			)
-		)
-		(pin "1"
-		)
-		(instances
-			(project ""
-				(path "/8c0b3d8b-46d3-4173-ab1e-a61765f77d61/4ea27ee4-1edc-4e10-ab5a-91b9933087c0"
-					(reference "#PWR019")
+					(reference "#PWR020")
 					(unit 1)
 				)
@@
 		(on_board yes)
 		(dnp no)
-		(property "Reference" "#PWR017"
+		(property "Reference" "#PWR016"
 			(at 205.74 80.01 0)
 			(effects
@@
 			(project "frank2"
 				(path "/8c0b3d8b-46d3-4173-ab1e-a61765f77d61/4ea27ee4-1edc-4e10-ab5a-91b9933087c0"
-					(reference "#PWR017")
+					(reference "#PWR016")
 					(unit 1)
 				)
@@
 		(on_board yes)
 		(dnp no)
-		(property "Reference" "#PWR016"
+		(property "Reference" "#PWR015"
 			(at 123.19 74.93 0)
 			(effects
@@
 			(project "frank2"
 				(path "/8c0b3d8b-46d3-4173-ab1e-a61765f77d61/4ea27ee4-1edc-4e10-ab5a-91b9933087c0"
-					(reference "#PWR016")
+					(reference "#PWR015")
 					(unit 1)
 				)
@@
 		(dnp no)
 		(fields_autoplaced yes)
-		(property "Reference" "#PWR028"
+		(property "Reference" "#PWR027"
 			(at 118.11 128.27 0)
 			(effects
@@
 			(project ""
 				(path "/8c0b3d8b-46d3-4173-ab1e-a61765f77d61/4ea27ee4-1edc-4e10-ab5a-91b9933087c0"
-					(reference "#PWR028")
+					(reference "#PWR027")
 					(unit 1)
 				)
@@
 		(dnp no)
 		(fields_autoplaced yes)
-		(property "Reference" "#PWR027"
+		(property "Reference" "#PWR026"
 			(at 195.58 119.38 0)
 			(effects
@@
 			(project ""
 				(path "/8c0b3d8b-46d3-4173-ab1e-a61765f77d61/4ea27ee4-1edc-4e10-ab5a-91b9933087c0"
-					(reference "#PWR027")
+					(reference "#PWR026")
 					(unit 1)
 				)
@@
 		(on_board yes)
 		(dnp no)
-		(property "Reference" "#PWR020"
+		(property "Reference" "#PWR019"
 			(at 187.96 92.71 0)
 			(effects
@@
 			(project "frank2"
 				(path "/8c0b3d8b-46d3-4173-ab1e-a61765f77d61/4ea27ee4-1edc-4e10-ab5a-91b9933087c0"
-					(reference "#PWR020")
-					(unit 1)
-				)
+					(reference "#PWR019")
+					(unit 1)
+				)

Commit message: Minor fixes
Parts:
- LD3: value Power -> Green (Power)
- R13: renamed from R12; AliExpress https://www.vishay.com/docs/28952/mcs0402at-mct0603at-mcu08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 -> https://www.aliexpress.com/item/1005005945735199.html
- renumbered C5 to C6, C6 to C7, R9 to R10, R10 to R11, R11 to R12, R7 to R8, R8 to R9
Changed lines of the file:
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@@
 	(title_block
 		(title "${NAME}")
-		(date "2025-05-24")
+		(date "2025-06-23")
 		(rev "${VERSION}")
 		(company "Mikhail Matveev")
@@
 		(on_board yes)
 		(dnp no)
-		(property "Reference" "#PWR023"
+		(property "Reference" "#PWR027"
 			(at 171.45 104.14 0)
 			(effects
@@
 			(project "frank2"
 				(path "/8c0b3d8b-46d3-4173-ab1e-a61765f77d61/4ea27ee4-1edc-4e10-ab5a-91b9933087c0"
-					(reference "#PWR023")
+					(reference "#PWR027")
 					(unit 1)
 				)
@@
 		(dnp no)
 		(fields_autoplaced yes)
-		(property "Reference" "#PWR014"
+		(property "Reference" "#PWR018"
 			(at 135.89 77.47 0)
 			(effects
@@
 			(project ""
 				(path "/8c0b3d8b-46d3-4173-ab1e-a61765f77d61/4ea27ee4-1edc-4e10-ab5a-91b9933087c0"
-					(reference "#PWR014")
+					(reference "#PWR018")
 					(unit 1)
 				)
@@
 		(on_board yes)
 		(dnp no)
-		(property "Reference" "#PWR021"
+		(property "Reference" "#PWR025"
 			(at 123.19 97.79 0)
 			(effects
@@
 			(project "frank2"
 				(path "/8c0b3d8b-46d3-4173-ab1e-a61765f77d61/4ea27ee4-1edc-4e10-ab5a-91b9933087c0"
-					(reference "#PWR021")
+					(reference "#PWR025")
 					(unit 1)
 				)
@@
 		(dnp no)
 		(fields_autoplaced yes)
-		(property "Reference" "#PWR025"
+		(property "Reference" "#PWR029"
 			(at 175.26 119.38 0)
 			(effects
@@
 			(project "frank2"
 				(path "/8c0b3d8b-46d3-4173-ab1e-a61765f77d61/4ea27ee4-1edc-4e10-ab5a-91b9933087c0"
-					(reference "#PWR025")
+					(reference "#PWR029")
 					(unit 1)
 				)
@@
 		(dnp no)
 		(fields_autoplaced yes)
-		(property "Reference" "#PWR022"
+		(property "Reference" "#PWR026"
 			(at 148.59 104.14 0)
 			(effects
@@
 			(project "echo"
 				(path "/8c0b3d8b-46d3-4173-ab1e-a61765f77d61/4ea27ee4-1edc-4e10-ab5a-91b9933087c0"
-					(reference "#PWR022")
+					(reference "#PWR026")
 					(unit 1)
 				)
@@
 			)
 		)
-		(property "Value" "Power"
+		(property "Value" "Green (Power)"
 			(at 183.8325 115.57 0)
 			(effects
@@
 		(on_board yes)
 		(dnp no)
-		(property "Reference" "R8"
+		(property "Reference" "R9"
 			(at 139.192 88.138 90)
 			(effects
@@
 			(project "echo"
 				(path "/8c0b3d8b-46d3-4173-ab1e-a61765f77d61/4ea27ee4-1edc-4e10-ab5a-91b9933087c0"
-					(reference "R8")
+					(reference "R9")
 					(unit 1)
 				)
@@
 		(on_board yes)
 		(dnp no)
-		(property "Reference" "C5"
+		(property "Reference" "C6"
 			(at 208.661 81.3816 0)
 			(effects
@@
 			(project "frank2"
 				(path "/8c0b3d8b-46d3-4173-ab1e-a61765f77d61/4ea27ee4-1edc-4e10-ab5a-91b9933087c0"
-					(reference "C5")
+					(reference "C6")
 					(unit 1)
 				)
@@
 		(on_board yes)
 		(dnp no)
-		(property "Reference" "#PWR024"
+		(property "Reference" "#PWR028"
 			(at 125.73 102.87 0)
 			(effects
@@
 			(project "frank_rm2-2350A"
 				(path "/8c0b3d8b-46d3-4173-ab1e-a61765f77d61/4ea27ee4-1edc-4e10-ab5a-91b9933087c0"
-					(reference "#PWR024")
+					(reference "#PWR028")
 					(unit 1)
 				)
@@
 		(dnp no)
 		(fields_autoplaced yes)
-		(property "Reference" "#PWR018"
+		(property "Reference" "#PWR022"
 			(at 152.4 82.55 0)
 			(effects
@@
 			(project ""
 				(path "/8c0b3d8b-46d3-4173-ab1e-a61765f77d61/4ea27ee4-1edc-4e10-ab5a-91b9933087c0"
-					(reference "#PWR018")
+					(reference "#PWR022")
 					(unit 1)
 				)
@@
 		(on_board yes)
 		(dnp no)
-		(property "Reference" "C6"
+		(property "Reference" "C7"
 			(at 174.371 82.6516 0)
 			(effects
@@
 			(project "frank2"
 				(path "/8c0b3d8b-46d3-4173-ab1e-a61765f77d61/4ea27ee4-1edc-4e10-ab5a-91b9933087c0"
-					(reference "C6")
+					(reference "C7")
 					(unit 1)
 				)
@@
 		(dnp no)
 		(fields_autoplaced yes)
-		(property "Reference" "R12"
+		(property "Reference" "R13"
 			(at 193.04 113.03 90)
 			(effects
@@
 			)
 		)
-		(property "AliExpress" "https://www.vishay.com/docs/28952/mcs0402at-mct0603at-mcu0805at-mca1206at.pdf"
+		(property "AliExpress" "https://www.aliexpress.com/item/1005005945735199.html"
 			(at 193.04 119.38 0)
 			(effects
@@
 			(project "frank2"
 				(path "/8c0b3d8b-46d3-4173-ab1e-a61765f77d61/4ea27ee4-1edc-4e10-ab5a-91b9933087c0"
-					(reference "R12")
+					(reference "R13")
 					(unit 1)
 				)
@@
 		(on_board yes)
 		(dnp no)
-		(property "Reference" "R10"
+		(property "Reference" "R11"
 			(at 114.3 95.25 90)
 			(effects
@@
 			(project "frank2"
 				(path "/8c0b3d8b-46d3-4173-ab1e-a61765f77d61/4ea27ee4-1edc-4e10-ab5a-91b9933087c0"
-					(reference "R10")
+					(reference "R11")
 					(unit 1)
 				)
@@
 		(on_board yes)
 		(dnp no)
-		(property "Reference" "#PWR017"
+		(property "Reference" "#PWR021"
 			(at 123.19 82.55 0)
 			(effects
@@
 			(project "frank2"
 				(path "/8c0b3d8b-46d3-4173-ab1e-a61765f77d61/4ea27ee4-1edc-4e10-ab5a-91b9933087c0"
-					(reference "#PWR017")
+					(reference "#PWR021")
 					(unit 1)
 				)
@@
 		(on_board yes)
 		(dnp no)
-		(property "Reference" "#PWR020"
+		(property "Reference" "#PWR024"
 			(at 205.74 93.98 0)
 			(effects
@@
 			(project "frank2"
 				(path "/8c0b3d8b-46d3-4173-ab1e-a61765f77d61/4ea27ee4-1edc-4e10-ab5a-91b9933087c0"
-					(reference "#PWR020")
+					(reference "#PWR024")
 					(unit 1)
 				)
@@
 		(on_board yes)
 		(dnp no)
-		(property "Reference" "#PWR016"
+		(property "Reference" "#PWR020"
 			(at 205.74 80.01 0)
 			(effects
@@
 			(project "frank2"
 				(path "/8c0b3d8b-46d3-4173-ab1e-a61765f77d61/4ea27ee4-1edc-4e10-ab5a-91b9933087c0"
-					(reference "#PWR016")
+					(reference "#PWR020")
 					(unit 1)
 				)
@@
 		(on_board yes)
 		(dnp no)
-		(property "Reference" "R7"
+		(property "Reference" "R8"
 			(at 114.3 80.01 90)
 			(effects
@@
 			(project "frank2"
 				(path "/8c0b3d8b-46d3-4173-ab1e-a61765f77d61/4ea27ee4-1edc-4e10-ab5a-91b9933087c0"
-					(reference "R7")
+					(reference "R8")
 					(unit 1)
 				)
@@
 		(on_board yes)
 		(dnp no)
-		(property "Reference" "#PWR015"
+		(property "Reference" "#PWR019"
 			(at 123.19 74.93 0)
 			(effects
@@
 			(project "frank2"
 				(path "/8c0b3d8b-46d3-4173-ab1e-a61765f77d61/4ea27ee4-1edc-4e10-ab5a-91b9933087c0"
-					(reference "#PWR015")
+					(reference "#PWR019")
 					(unit 1)
 				)
@@
 		(on_board yes)
 		(dnp no)
-		(property "Reference" "R9"
+		(property "Reference" "R10"
 			(at 139.446 94.996 90)
 			(effects
@@
 			(project "echo"
 				(path "/8c0b3d8b-46d3-4173-ab1e-a61765f77d61/4ea27ee4-1edc-4e10-ab5a-91b9933087c0"
-					(reference "R9")
+					(reference "R10")
 					(unit 1)
 				)
@@
 		(dnp no)
 		(fields_autoplaced yes)
-		(property "Reference" "#PWR027"
+		(property "Reference" "#PWR031"
 			(at 118.11 128.27 0)
 			(effects
@@
 			(project ""
 				(path "/8c0b3d8b-46d3-4173-ab1e-a61765f77d61/4ea27ee4-1edc-4e10-ab5a-91b9933087c0"
-					(reference "#PWR027")
+					(reference "#PWR031")
 					(unit 1)
 				)
@@
 		(dnp no)
 		(fields_autoplaced yes)
-		(property "Reference" "R11"
+		(property "Reference" "R12"
 			(at 120.65 113.0299 0)
 			(effects
@@
 			(project "frank_rm2-2350A"
 				(path "/8c0b3d8b-46d3-4173-ab1e-a61765f77d61/4ea27ee4-1edc-4e10-ab5a-91b9933087c0"
-					(reference "R11")
+					(reference "R12")
 					(unit 1)
 				)
@@
 		(dnp no)
 		(fields_autoplaced yes)
-		(property "Reference" "#PWR026"
+		(property "Reference" "#PWR030"
 			(at 195.58 119.38 0)
 			(effects
@@
 			(project ""
 				(path "/8c0b3d8b-46d3-4173-ab1e-a61765f77d61/4ea27ee4-1edc-4e10-ab5a-91b9933087c0"
-					(reference "#PWR026")
+					(reference "#PWR030")
 					(unit 1)
 				)
@@
 		(on_board yes)
 		(dnp no)
-		(property "Reference" "#PWR019"
+		(property "Reference" "#PWR023"
 			(at 187.96 92.71 0)
 			(effects
@@
 			(project "frank2"
 				(path "/8c0b3d8b-46d3-4173-ab1e-a61765f77d61/4ea27ee4-1edc-4e10-ab5a-91b9933087c0"
-					(reference "#PWR019")
-					(unit 1)
-				)
+					(reference "#PWR023")
+					(unit 1)
+				)

Commit message: HW Rev 1.03
Parts:
- renumbered C6 to C5, C7 to C6
Changed lines of the file:
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@@
 	(title_block
 		(title "${NAME}")
-		(date "2025-06-23")
+		(date "2025-07-20")
 		(rev "${VERSION}")
 		(company "Mikhail Matveev")
@@
 		(on_board yes)
 		(dnp no)
-		(property "Reference" "C6"
+		(property "Reference" "C5"
 			(at 208.661 81.3816 0)
 			(effects
@@
 			(project "frank2"
 				(path "/8c0b3d8b-46d3-4173-ab1e-a61765f77d61/4ea27ee4-1edc-4e10-ab5a-91b9933087c0"
-					(reference "C6")
+					(reference "C5")
 					(unit 1)
 				)
@@
 		(on_board yes)
 		(dnp no)
-		(property "Reference" "C7"
+		(property "Reference" "C6"
 			(at 174.371 82.6516 0)
 			(effects
@@
 			(project "frank2"
 				(path "/8c0b3d8b-46d3-4173-ab1e-a61765f77d61/4ea27ee4-1edc-4e10-ab5a-91b9933087c0"
-					(reference "C7")
+					(reference "C6")
 					(unit 1)
 				)

Commit message: WIP
Parts:
- added C7: 10u, FRANK:Capacitor (0805), symbol Device:C
- added J2: USB4215-03-A, FRANK:USB Type C, symbol FRANK:USB-C
- added R18, R21: 5.1K, FRANK:Resistor (0805), symbol Device:R_Small
- added R19, R20: 22R, FRANK:Resistor (0805), symbol Device:R
- added R22: 1M, FRANK:Resistor (0805), symbol Device:R
- added S4: Power, FRANK:Switch (MSK12C02), symbol Switch:SW_SPDT_321
- added U5: USBLC6-2SC6, FRANK:SOT-23-6, symbol Power_Protection:USBLC6-2SC6
- LD3: value Green (Power) -> Green
- U4: symbol Power_Protection:USBLC6-2SC6 -> FRANK:USBLC6-2SC6; AliExpress (none) -> https://vi.aliexpress.com/item/1005006883533480.html
- renumbered R8 to R12, R9 to R13, R10 to R14, R11 to R15, R12 to R16, R13 to R17
Connections:
- net GND: now also C7.2, J2.1 (GND), J2.12 (GND), R18.1, R21.1, R22.2, U5.2 (GND)
- net VBUS: now also C7.1, J2.11 (VBUS), J2.2 (VBUS), S4.3 (A), U5.5 (VBUS); no longer J1.11 (VBUS), J1.2 (VBUS)
- net D+ renamed D1+
- net D- renamed D1-
- new net: J1.11 (VBUS), J1.2 (VBUS), S4.2 (B)
- new net: J2.13 (SHIELD), R22.1
- new net: J2.4 (CC1), R18.2
- new net: R19.1, U5.1 (I/O1)
- new net: R20.1, U5.3 (I/O2)
- new net: J2.5 (DN2), J2.7 (DN1), R19.2
- new net: J2.6 (DP1), J2.8 (DP2), R20.2
- new net: J2.10 (CC2), R21.2
- new net D2+: U5.4 (I/O2)
- new net D2-: U5.6 (I/O1)
- no-connect marks 2 -> 5
Other:
- moved on the sheet: C5, C6, LD3, R12, R13, R14, R15, R16, R17, U3, U4
