File: power.kicad_sch (KiCad schematic)
At the start: 20 parts, among them J1 USB4215-03-A, J2 USB4215-03-A, U3 NCP1117 3.3, U4 USBLC6-2SC6, U5 USBLC6-2SC6

Commit message: HW 1.06 WIP
Parts:
- renumbered C6 to C5, C7 to C6, C5 to C7, R15 to R13, R16 to R14, R18 to R15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
