File: usb2ttl.kicad_sch (KiCad schematic)
At the start: 13 parts, among them Q1 BSS138, Q2 BSS138, U1 CH340G, X1 12 Mhz

Commit message: Work-in-progress
Parts:
- removed C3: 1u, FRANK:Capacitor (0805), symbol Device:C_Small
- added R5, R6: 2.2K, FRANK:Resistor (0805), symbol Device:R_Small
- renumbered C1 to C3, C2 to C4, C4 to C5, C5 to C6, R1 to R3, R2 to R4, U1 to U2
Connections:
- net at Q1.2 (E), U2.14 (RTS): now also R6.2; no longer Q2.1 (B)
- net at Q2.2 (E), U2.13 (DTR): now also R5.2; no longer Q1.1 (B)
- new net: Q2.1 (B), R6.1
- new net: Q1.1 (B), R5.1
Other:
- moved on the sheet: C5, C6, Q1, Q2

Commit message: 1.01 WIP
Parts:
- removed C5, C6: 15p, FRANK:Capacitor (0805), symbol Device:C_Small
- removed X1: 12 Mhz, FRANK:Crystal (HC49-S), symbol FRANK:Crystal_Generic
- U2: value CH340G -> CH340C
Connections:
- net VCC renamed VBUS
- no-connect marks 5 -> 7

Commit message: Minor fixes
Parts:
- C4: renamed from C3; AliExpress (none) -> https://www.aliexpress.com/item/33008008276.html
- C5: renamed from C4; AliExpress (none) -> https://www.aliexpress.com/item/33008008276.html
- LD1: value TX -> Orange (TX)
- LD2: value RX -> Orange (RX)
- R4: renamed from R3; AliExpress (none) -> https://www.aliexpress.com/item/1005005945735199.html
- R5: renamed from R4; AliExpress (none) -> https://www.aliexpress.com/item/1005005945735199.html
- R6: renamed from R5; AliExpress (none) -> https://www.aliexpress.com/item/1005005945735199.html
- R7: renamed from R6; AliExpress (none) -> https://www.aliexpress.com/item/1005005945735199.html
Changed lines of the file:
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@@
 	(title_block
 		(title "${NAME}")
-		(date "2025-05-24")
+		(date "2025-06-23")
 		(rev "${VERSION}")
 		(company "Mikhail Matveev")
@@
 			)
 		)
-		(property "Value" "TX"
+		(property "Value" "Orange (TX)"
 			(at 188.468 83.82 0)
 			(effects
@@
 		(dnp no)
 		(fields_autoplaced yes)
-		(property "Reference" "#PWR013"
+		(property "Reference" "#PWR017"
 			(at 97.79 96.52 0)
 			(effects
@@
 			(project "echo"
 				(path "/8c0b3d8b-46d3-4173-ab1e-a61765f77d61/f883457e-0c9e-4a1d-9f19-b038d36f033f"
-					(reference "#PWR013")
+					(reference "#PWR017")
 					(unit 1)
 				)
@@
 		(on_board yes)
 		(dnp no)
-		(property "Reference" "R5"
+		(property "Reference" "R6"
 			(at 185.42 104.14 90)
 			(effects
@@
 		)
 		(property "Description" "Resistor, small symbol"
+			(at 185.42 106.68 0)
+			(effects
+				(font
+					(size 1.27 1.27)
+				)
+				(hide yes)
+			)
+		)
+		(property "AliExpress" "https://www.aliexpress.com/item/1005005945735199.html"
 			(at 185.42 106.68 0)
 			(effects
@@
 			(project "echo"
 				(path "/8c0b3d8b-46d3-4173-ab1e-a61765f77d61/f883457e-0c9e-4a1d-9f19-b038d36f033f"
-					(reference "R5")
+					(reference "R6")
 					(unit 1)
 				)
@@
 		(on_board yes)
 		(dnp no)
-		(property "Reference" "R4"
+		(property "Reference" "R5"
 			(at 198.374 74.93 90)
 			(effects
@@
 		)
 		(property "Description" "Resistor, small symbol"
+			(at 195.58 74.93 0)
+			(effects
+				(font
+					(size 1.27 1.27)
+				)
+				(hide yes)
+			)
+		)
+		(property "AliExpress" "https://www.aliexpress.com/item/1005005945735199.html"
 			(at 195.58 74.93 0)
 			(effects
@@
 			(project "echo"
 				(path "/8c0b3d8b-46d3-4173-ab1e-a61765f77d61/f883457e-0c9e-4a1d-9f19-b038d36f033f"
-					(reference "R4")
+					(reference "R5")
 					(unit 1)
 				)
@@
 		(on_board yes)
 		(dnp no)
-		(property "Reference" "C4"
+		(property "Reference" "C5"
 			(at 98.298 82.55 0)
 			(effects
@@
 		)
 		(property "Description" "Unpolarized capacitor, small symbol"
+			(at 97.79 85.09 0)
+			(effects
+				(font
+					(size 1.27 1.27)
+				)
+				(hide yes)
+			)
+		)
+		(property "AliExpress" "https://www.aliexpress.com/item/33008008276.html"
 			(at 97.79 85.09 0)
 			(effects
@@
 			(project "echo"
 				(path "/8c0b3d8b-46d3-4173-ab1e-a61765f77d61/f883457e-0c9e-4a1d-9f19-b038d36f033f"
-					(reference "C4")
+					(reference "C5")
 					(unit 1)
 				)
@@
 		(dnp no)
 		(fields_autoplaced yes)
-		(property "Reference" "#PWR011"
+		(property "Reference" "#PWR015"
 			(at 204.47 67.31 0)
 			(effects
@@
 			(project ""
 				(path "/8c0b3d8b-46d3-4173-ab1e-a61765f77d61/f883457e-0c9e-4a1d-9f19-b038d36f033f"
-					(reference "#PWR011")
+					(reference "#PWR015")
 					(unit 1)
 				)
@@
 		(on_board yes)
 		(dnp no)
-		(property "Reference" "R3"
+		(property "Reference" "R4"
 			(at 187.96 74.93 90)
 			(effects
@@
 		)
 		(property "Description" "Resistor, small symbol"
+			(at 185.42 74.93 0)
+			(effects
+				(font
+					(size 1.27 1.27)
+				)
+				(hide yes)
+			)
+		)
+		(property "AliExpress" "https://www.aliexpress.com/item/1005005945735199.html"
 			(at 185.42 74.93 0)
 			(effects
@@
 			(project "echo"
 				(path "/8c0b3d8b-46d3-4173-ab1e-a61765f77d61/f883457e-0c9e-4a1d-9f19-b038d36f033f"
-					(reference "R3")
+					(reference "R4")
 					(unit 1)
 				)
@@
 		(dnp no)
 		(fields_autoplaced yes)
-		(property "Reference" "#PWR010"
+		(property "Reference" "#PWR014"
 			(at 111.76 67.31 0)
 			(effects
@@
 			(project ""
 				(path "/8c0b3d8b-46d3-4173-ab1e-a61765f77d61/f883457e-0c9e-4a1d-9f19-b038d36f033f"
-					(reference "#PWR010")
+					(reference "#PWR014")
 					(unit 1)
 				)
@@
 		(on_board yes)
 		(dnp no)
-		(property "Reference" "#PWR012"
+		(property "Reference" "#PWR016"
 			(at 175.26 83.82 0)
 			(effects
@@
 			(project "echo"
 				(path "/8c0b3d8b-46d3-4173-ab1e-a61765f77d61/f883457e-0c9e-4a1d-9f19-b038d36f033f"
-					(reference "#PWR012")
+					(reference "#PWR016")
 					(unit 1)
 				)
@@
 			)
 		)
-		(property "Value" "RX"
+		(property "Value" "Orange (RX)"
 			(at 198.374 84.074 0)
 			(effects
@@
 		(on_board yes)
 		(dnp no)
-		(property "Reference" "R6"
+		(property "Reference" "R7"
 			(at 185.42 121.92 90)
 			(effects
@@
 		)
 		(property "Description" "Resistor, small symbol"
+			(at 185.42 124.46 0)
+			(effects
+				(font
+					(size 1.27 1.27)
+				)
+				(hide yes)
+			)
+		)
+		(property "AliExpress" "https://www.aliexpress.com/item/1005005945735199.html"
 			(at 185.42 124.46 0)
 			(effects
@@
 			(project "echo"
 				(path "/8c0b3d8b-46d3-4173-ab1e-a61765f77d61/f883457e-0c9e-4a1d-9f19-b038d36f033f"
-					(reference "R6")
+					(reference "R7")
 					(unit 1)
 				)
@@
 		(on_board yes)
 		(dnp no)
-		(property "Reference" "C3"
+		(property "Reference" "C4"
 			(at 175.768 69.85 0)
 			(effects
@@
 		)
 		(property "Description" "Unpolarized capacitor, small symbol"
+			(at 175.26 72.39 0)
+			(effects
+				(font
+					(size 1.27 1.27)
+				)
+				(hide yes)
+			)
+		)
+		(property "AliExpress" "https://www.aliexpress.com/item/33008008276.html"
 			(at 175.26 72.39 0)
 			(effects
@@
 			(project "echo"
 				(path "/8c0b3d8b-46d3-4173-ab1e-a61765f77d61/f883457e-0c9e-4a1d-9f19-b038d36f033f"
-					(reference "C3")
+					(reference "C4")
 					(unit 1)
 				)

Commit message: HW Rev 1.03
Parts:
- removed C5: 100n, FRANK:Capacitor (0805), symbol Device:C_Small
Connections:
- net VBUS is gone; now on net +3V3: C4.1, R4.2, R5.1, U2.16 (VCC)
- net +3V3: now reaches U2.4 (3V)
Changed lines of the file:
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@@
 	(title_block
 		(title "${NAME}")
-		(date "2025-06-23")
+		(date "2025-07-20")
 		(rev "${VERSION}")
 		(company "Mikhail Matveev")
@@
 	(wire
 		(pts
-			(xy 97.79 74.93) (xy 125.73 74.93)
-		)
-		(stroke
-			(width 0)
-			(type default)
-		)
-	)
-	(wire
-		(pts
 			(xy 175.26 74.93) (xy 175.26 77.47)
 		)
@@
 	(wire
 		(pts
-			(xy 97.79 90.17) (xy 97.79 87.63)
-		)
-		(stroke
-			(width 0)
-			(type default)
-		)
-	)
-	(wire
-		(pts
 			(xy 203.2 129.54) (xy 170.18 129.54)
 		)
@@
 	(wire
 		(pts
-			(xy 97.79 74.93) (xy 97.79 82.55)
-		)
-		(stroke
-			(width 0)
-			(type default)
-		)
-	)
-	(wire
-		(pts
 			(xy 177.8 90.17) (xy 195.58 90.17)
 		)
@@
 		(pts
 			(xy 195.58 77.47) (xy 195.58 80.01)
+		)
+		(stroke
+			(width 0)
+			(type default)
+		)
+	)
+	(wire
+		(pts
+			(xy 118.11 74.93) (xy 125.73 74.93)
 		)
 		(stroke
@@
 			)
 			(justify right)
+		)
+	)
+	(symbol
+		(lib_id "power:+3V3")
+		(at 118.11 74.93 90)
+		(unit 1)
+		(exclude_from_sim no)
+		(in_bom yes)
+		(on_board yes)
+		(dnp no)
+		(fields_autoplaced yes)
+		(property "Reference" "#PWR016"
+			(at 121.92 74.93 0)
+			(effects
+				(font
+					(size 1.27 1.27)
+				)
+				(hide yes)
+			)
+		)
+		(property "Value" "+3V3"
+			(at 114.3 74.9299 90)
+			(effects
+				(font
+					(size 1.27 1.27)
+				)
+				(justify left)
+			)
+		)
+		(property "Footprint" ""
+			(at 118.11 74.93 0)
+			(effects
+				(font
+					(size 1.27 1.27)
+				)
+				(hide yes)
+			)
+		)
+		(property "Datasheet" ""
+			(at 118.11 74.93 0)
+			(effects
+				(font
+					(size 1.27 1.27)
+				)
+				(hide yes)
+			)
+		)
+		(property "Description" "Power symbol creates a global label with name \"+3V3\""
+			(at 118.11 74.93 0)
+			(effects
+				(font
+					(size 1.27 1.27)
+				)
+				(hide yes)
+			)
+		)
+		(pin "1"
+		)
+		(instances
+			(project "echo"
+				(path "/8c0b3d8b-46d3-4173-ab1e-a61765f77d61/f883457e-0c9e-4a1d-9f19-b038d36f033f"
+					(reference "#PWR016")
+					(unit 1)
+				)
+			)
 		)
 	)
@@
 	)
 	(symbol
-		(lib_id "power:GND")
-		(at 97.79 90.17 0)
-		(unit 1)
-		(exclude_from_sim no)
-		(in_bom yes)
-		(on_board yes)
-		(dnp no)
-		(fields_autoplaced yes)
-		(property "Reference" "#PWR017"
-			(at 97.79 96.52 0)
-			(effects
-				(font
-					(size 1.27 1.27)
-				)
-				(hide yes)
-			)
-		)
-		(property "Value" "GND"
-			(at 97.79 95.25 0)
-			(effects
-				(font
-					(size 1.27 1.27)
-				)
-			)
-		)
-		(property "Footprint" ""
-			(at 97.79 90.17 0)
-			(effects
-				(font
-					(size 1.27 1.27)
-				)
-				(hide yes)
-			)
-		)
-		(property "Datasheet" ""
-			(at 97.79 90.17 0)
-			(effects
-				(font
-					(size 1.27 1.27)
-				)
-				(hide yes)
-			)
-		)
-		(property "Description" "Power symbol creates a global label with name \"GND\" , ground"
-			(at 97.79 90.17 0)
-			(effects
-				(font
-					(size 1.27 1.27)
-				)
-				(hide yes)
-			)
-		)
-		(pin "1"
-		)
-		(instances
-			(project "echo"
-				(path "/8c0b3d8b-46d3-4173-ab1e-a61765f77d61/f883457e-0c9e-4a1d-9f19-b038d36f033f"
-					(reference "#PWR017")
-					(unit 1)
-				)
-			)
-		)
-	)
-	(symbol
 		(lib_id "FRANK:CH340G")
 		(at 143.51 77.47 0)
@@
 				(path "/8c0b3d8b-46d3-4173-ab1e-a61765f77d61/f883457e-0c9e-4a1d-9f19-b038d36f033f"
 					(reference "U2")
+					(unit 1)
+				)
+			)
+		)
+	)
+	(symbol
+		(lib_id "power:+3V3")
+		(at 208.28 67.31 270)
+		(unit 1)
+		(exclude_from_sim no)
+		(in_bom yes)
+		(on_board yes)
+		(dnp no)
+		(fields_autoplaced yes)
+		(property "Reference" "#PWR015"
+			(at 204.47 67.31 0)
+			(effects
+				(font
+					(size 1.27 1.27)
+				)
+				(hide yes)
+			)
+		)
+		(property "Value" "+3V3"
+			(at 212.09 67.3099 90)
+			(effects
+				(font
+					(size 1.27 1.27)
+				)
+				(justify left)
+			)
+		)
+		(property "Footprint" ""
+			(at 208.28 67.31 0)
+			(effects
+				(font
+					(size 1.27 1.27)
+				)
+				(hide yes)
+			)
+		)
+		(property "Datasheet" ""
+			(at 208.28 67.31 0)
+			(effects
+				(font
+					(size 1.27 1.27)
+				)
+				(hide yes)
+			)
+		)
+		(property "Description" "Power symbol creates a global label with name \"+3V3\""
+			(at 208.28 67.31 0)
+			(effects
+				(font
+					(size 1.27 1.27)
+				)
+				(hide yes)
+			)
+		)
+		(pin "1"
+		)
+		(instances
+			(project ""
+				(path "/8c0b3d8b-46d3-4173-ab1e-a61765f77d61/f883457e-0c9e-4a1d-9f19-b038d36f033f"
+					(reference "#PWR015")
 					(unit 1)
 				)
@@
 				(path "/8c0b3d8b-46d3-4173-ab1e-a61765f77d61/f883457e-0c9e-4a1d-9f19-b038d36f033f"
 					(reference "R5")
-					(unit 1)
-				)
-			)
-		)
-	)
-	(symbol
-		(lib_id "Device:C_Small")
-		(at 97.79 85.09 0)
-		(unit 1)
-		(exclude_from_sim no)
-		(in_bom yes)
-		(on_board yes)
-		(dnp no)
-		(property "Reference" "C5"
-			(at 98.298 82.55 0)
-			(effects
-				(font
-					(size 1.524 1.524)
-				)
-				(justify left)
-			)
-		)
-		(property "Value" "100n"
-			(at 98.298 87.63 0)
-			(effects
-				(font
-					(size 1.524 1.524)
-				)
-				(justify left)
-			)
-		)
-		(property "Footprint" "FRANK:Capacitor (0805)"
-			(at 97.79 85.09 0)
-			(effects
-				(font
-					(size 1.27 1.27)
-				)
-				(hide yes)
-			)
-		)
-		(property "Datasheet" "~"
-			(at 97.79 85.09 0)
-			(effects
-				(font
-					(size 1.27 1.27)
-				)
-				(hide yes)
-			)
-		)
-		(property "Description" "Unpolarized capacitor, small symbol"
-			(at 97.79 85.09 0)
-			(effects
-				(font
-					(size 1.27 1.27)
-				)
-				(hide yes)
-			)
-		)
-		(property "AliExpress" "https://www.aliexpress.com/item/33008008276.html"
-			(at 97.79 85.09 0)
-			(effects
-				(font
-					(size 1.27 1.27)
-				)
-				(hide yes)
-			)
-		)
-		(pin "1"
-		)
-		(pin "2"
-		)
-		(instances
-			(project "echo"
-				(path "/8c0b3d8b-46d3-4173-ab1e-a61765f77d61/f883457e-0c9e-4a1d-9f19-b038d36f033f"
-					(reference "C5")
-					(unit 1)
-				)
-			)
-		)
-	)
-	(symbol
-		(lib_id "power:VBUS")
-		(at 208.28 67.31 270)
-		(unit 1)
-		(exclude_from_sim no)
-		(in_bom yes)
-		(on_board yes)
-		(dnp no)
-		(fields_autoplaced yes)
-		(property "Reference" "#PWR015"
-			(at 204.47 67.31 0)
-			(effects
-				(font
-					(size 1.27 1.27)
-				)
-				(hide yes)
-			)
-		)
-		(property "Value" "VBUS"
-			(at 212.09 67.3099 90)
-			(effects
-				(font
-					(size 1.27 1.27)
-				)
-				(justify left)
-			)
-		)
-		(property "Footprint" ""
-			(at 208.28 67.31 0)
-			(effects
-				(font
-					(size 1.27 1.27)
-				)
-				(hide yes)
-			)
-		)
-		(property "Datasheet" ""
-			(at 208.28 67.31 0)
-			(effects
-				(font
-					(size 1.27 1.27)
-				)
-				(hide yes)
-			)
-		)
-		(property "Description" "Power symbol creates a global label with name \"VBUS\""
-			(at 208.28 67.31 0)
-			(effects
-				(font
-					(size 1.27 1.27)
-				)
-				(hide yes)
-			)
-		)
-		(pin "1"
-		)
-		(instances
-			(project ""
-				(path "/8c0b3d8b-46d3-4173-ab1e-a61765f77d61/f883457e-0c9e-4a1d-9f19-b038d36f033f"
-					(reference "#PWR015")
 					(unit 1)
 				)
@@
 		(on_board yes)
 		(dnp no)
-		(property "Reference" "#PWR016"
+		(property "Reference" "#PWR017"
 			(at 175.26 83.82 0)
 			(effects
@@
 			(project "echo"
 				(path "/8c0b3d8b-46d3-4173-ab1e-a61765f77d61/f883457e-0c9e-4a1d-9f19-b038d36f033f"
-					(reference "#PWR016")
+					(reference "#PWR017")
 					(unit 1)
 				)

Commit message: WIP
Parts:
- renumbered R6 to R10, R7 to R11, R4 to R8, R5 to R9
Changed lines of the file:
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@@
 	(title_block
 		(title "${NAME}")
-		(date "2025-07-20")
+		(date "2025-08-08")
 		(rev "${VERSION}")
 		(company "Mikhail Matveev")
@@
 		(dnp no)
 		(fields_autoplaced yes)
-		(property "Reference" "#PWR016"
+		(property "Reference" "#PWR019"
 			(at 121.92 74.93 0)
 			(effects
@@
 			(project "echo"
 				(path "/8c0b3d8b-46d3-4173-ab1e-a61765f77d61/f883457e-0c9e-4a1d-9f19-b038d36f033f"
-					(reference "#PWR016")
+					(reference "#PWR019")
 					(unit 1)
 				)
@@
 		(dnp no)
 		(fields_autoplaced yes)
-		(property "Reference" "#PWR015"
+		(property "Reference" "#PWR018"
 			(at 204.47 67.31 0)
 			(effects
@@
 			(project ""
 				(path "/8c0b3d8b-46d3-4173-ab1e-a61765f77d61/f883457e-0c9e-4a1d-9f19-b038d36f033f"
-					(reference "#PWR015")
+					(reference "#PWR018")
 					(unit 1)
 				)
@@
 		(on_board yes)
 		(dnp no)
-		(property "Reference" "R6"
+		(property "Reference" "R10"
 			(at 185.42 104.14 90)
 			(effects
@@
 			(project "echo"
 				(path "/8c0b3d8b-46d3-4173-ab1e-a61765f77d61/f883457e-0c9e-4a1d-9f19-b038d36f033f"
-					(reference "R6")
+					(reference "R10")
 					(unit 1)
 				)
@@
 		(on_board yes)
 		(dnp no)
-		(property "Reference" "R5"
+		(property "Reference" "R9"
 			(at 198.374 74.93 90)
 			(effects
@@
 			(project "echo"
 				(path "/8c0b3d8b-46d3-4173-ab1e-a61765f77d61/f883457e-0c9e-4a1d-9f19-b038d36f033f"
-					(reference "R5")
+					(reference "R9")
 					(unit 1)
 				)
@@
 		(on_board yes)
 		(dnp no)
-		(property "Reference" "R4"
+		(property "Reference" "R8"
 			(at 187.96 74.93 90)
 			(effects
@@
 			(project "echo"
 				(path "/8c0b3d8b-46d3-4173-ab1e-a61765f77d61/f883457e-0c9e-4a1d-9f19-b038d36f033f"
-					(reference "R4")
+					(reference "R8")
 					(unit 1)
 				)
@@
 		(dnp no)
 		(fields_autoplaced yes)
-		(property "Reference" "#PWR014"
+		(property "Reference" "#PWR017"
 			(at 111.76 67.31 0)
 			(effects
@@
 			(project ""
 				(path "/8c0b3d8b-46d3-4173-ab1e-a61765f77d61/f883457e-0c9e-4a1d-9f19-b038d36f033f"
-					(reference "#PWR014")
+					(reference "#PWR017")
 					(unit 1)
 				)
@@
 		(on_board yes)
 		(dnp no)
-		(property "Reference" "#PWR017"
+		(property "Reference" "#PWR020"
 			(at 175.26 83.82 0)
 			(effects
@@
 			(project "echo"
 				(path "/8c0b3d8b-46d3-4173-ab1e-a61765f77d61/f883457e-0c9e-4a1d-9f19-b038d36f033f"
-					(reference "#PWR017")
+					(reference "#PWR020")
 					(unit 1)
 				)
@@
 		(on_board yes)
 		(dnp no)
-		(property "Reference" "R7"
+		(property "Reference" "R11"
 			(at 185.42 121.92 90)
 			(effects
@@
 			(project "echo"
 				(path "/8c0b3d8b-46d3-4173-ab1e-a61765f77d61/f883457e-0c9e-4a1d-9f19-b038d36f033f"
-					(reference "R7")
+					(reference "R11")
 					(unit 1)
 				)

Commit message: Rev 1.05 WIP
Parts:
- C4: footprint FRANK:Capacitor (0805) -> FRANK:Capacitor (0603)
- R10, R11, R8, R9: footprint FRANK:Resistor (0805) -> FRANK:Resistor (0603)
Changed lines of the file:
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@@
 			)
 		)
-		(property "Footprint" "FRANK:Resistor (0805)"
+		(property "Footprint" "FRANK:Resistor (0603)"
 			(at 185.42 106.68 0)
 			(effects
@@
 			)
 		)
-		(property "Footprint" "FRANK:Resistor (0805)"
+		(property "Footprint" "FRANK:Resistor (0603)"
 			(at 195.58 74.93 0)
 			(effects
@@
 			)
 		)
-		(property "Footprint" "FRANK:Resistor (0805)"
+		(property "Footprint" "FRANK:Resistor (0603)"
 			(at 185.42 74.93 0)
 			(effects
@@
 			)
 		)
-		(property "Footprint" "FRANK:Resistor (0805)"
+		(property "Footprint" "FRANK:Resistor (0603)"
 			(at 185.42 124.46 0)
 			(effects
@@
 			)
 		)
-		(property "Footprint" "FRANK:Capacitor (0805)"
+		(property "Footprint" "FRANK:Capacitor (0603)"
 			(at 175.26 72.39 0)
 			(effects

Commit message: HW Revision 1.05
Parts:
- LD1, LD2: footprint FRANK:LED (0805) -> FRANK:LED (0603)
Changed lines of the file:
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@@
 			)
 		)
-		(property "Footprint" "FRANK:LED (0805)"
+		(property "Footprint" "FRANK:LED (0603)"
 			(at 185.42 82.55 90)
 			(effects
@@
 	)
 	(symbol
+		(lib_name "R_Small_3")
 		(lib_id "Device:R_Small")
 		(at 185.42 106.68 270)
@@
 	)
 	(symbol
+		(lib_name "R_Small_2")
 		(lib_id "Device:R_Small")
 		(at 195.58 74.93 0)
@@
 	)
 	(symbol
+		(lib_name "R_Small_1")
 		(lib_id "Device:R_Small")
 		(at 185.42 74.93 180)
@@
 			)
 		)
-		(property "Footprint" "FRANK:LED (0805)"
+		(property "Footprint" "FRANK:LED (0603)"
 			(at 195.58 82.55 90)
 			(effects
