File: vga.kicad_sch (KiCad schematic)
At the start: 9 parts, among them J3 D-SUB 15 Female

Commit message: Work-in-progress
Parts:
- renumbered J3 to J4, R15 to R21, R16 to R22, R17 to R23, R18 to R24, R19 to R25, R20 to R26, R21 to R27, R22 to R28
Changed lines of the file:
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@@
 	(title_block
 		(title "${NAME}")
-		(date "2025-04-29")
+		(date "2025-04-30")
 		(rev "${VERSION}")
 		(company "Mikhail Matveev")
@@
 		(on_board yes)
 		(dnp no)
-		(property "Reference" "R17"
+		(property "Reference" "R23"
 			(at 95.25 73.66 90)
 			(effects
@@
 			(project "turbofrank"
 				(path "/8c0b3d8b-46d3-4173-ab1e-a61765f77d61/8958bb3d-1ab4-4fa9-968d-9ba0bebf85a9"
-					(reference "R17")
+					(reference "R23")
 					(unit 1)
 				)
@@
 		(on_board yes)
 		(dnp no)
-		(property "Reference" "R22"
+		(property "Reference" "R28"
 			(at 177.8 95.25 90)
 			(effects
@@
 			(project "turbofrank"
 				(path "/8c0b3d8b-46d3-4173-ab1e-a61765f77d61/8958bb3d-1ab4-4fa9-968d-9ba0bebf85a9"
-					(reference "R22")
+					(reference "R28")
 					(unit 1)
 				)
@@
 		(dnp no)
 		(fields_autoplaced yes)
-		(property "Reference" "J3"
+		(property "Reference" "J4"
 			(at 151.13 68.58 0)
 			(effects
@@
 			(project "turbofrank"
 				(path "/8c0b3d8b-46d3-4173-ab1e-a61765f77d61/8958bb3d-1ab4-4fa9-968d-9ba0bebf85a9"
-					(reference "J3")
+					(reference "J4")
 					(unit 1)
 				)
@@
 		(on_board yes)
 		(dnp no)
-		(property "Reference" "R19"
+		(property "Reference" "R25"
 			(at 114.3 85.09 90)
 			(effects
@@
 			(project "turbofrank"
 				(path "/8c0b3d8b-46d3-4173-ab1e-a61765f77d61/8958bb3d-1ab4-4fa9-968d-9ba0bebf85a9"
-					(reference "R19")
+					(reference "R25")
 					(unit 1)
 				)
@@
 		(dnp no)
 		(fields_autoplaced yes)
-		(property "Reference" "#PWR030"
+		(property "Reference" "#PWR039"
 			(at 151.13 123.19 0)
 			(effects
@@
 			(project "turbofrank"
 				(path "/8c0b3d8b-46d3-4173-ab1e-a61765f77d61/8958bb3d-1ab4-4fa9-968d-9ba0bebf85a9"
-					(reference "#PWR030")
+					(reference "#PWR039")
 					(unit 1)
 				)
@@
 		(on_board yes)
 		(dnp no)
-		(property "Reference" "R18"
+		(property "Reference" "R24"
 			(at 114.3 80.01 90)
 			(effects
@@
 			(project "turbofrank"
 				(path "/8c0b3d8b-46d3-4173-ab1e-a61765f77d61/8958bb3d-1ab4-4fa9-968d-9ba0bebf85a9"
-					(reference "R18")
+					(reference "R24")
 					(unit 1)
 				)
@@
 		(on_board yes)
 		(dnp no)
-		(property "Reference" "R21"
+		(property "Reference" "R27"
 			(at 177.8 90.17 90)
 			(effects
@@
 			(project "turbofrank"
 				(path "/8c0b3d8b-46d3-4173-ab1e-a61765f77d61/8958bb3d-1ab4-4fa9-968d-9ba0bebf85a9"
-					(reference "R21")
+					(reference "R27")
 					(unit 1)
 				)
@@
 		(on_board yes)
 		(dnp no)
-		(property "Reference" "R16"
+		(property "Reference" "R22"
 			(at 95.25 68.58 90)
 			(effects
@@
 			(project "turbofrank"
 				(path "/8c0b3d8b-46d3-4173-ab1e-a61765f77d61/8958bb3d-1ab4-4fa9-968d-9ba0bebf85a9"
-					(reference "R16")
+					(reference "R22")
 					(unit 1)
 				)
@@
 		(on_board yes)
 		(dnp no)
-		(property "Reference" "R15"
+		(property "Reference" "R21"
 			(at 95.25 63.5 90)
 			(effects
@@
 			(project "turbofrank"
 				(path "/8c0b3d8b-46d3-4173-ab1e-a61765f77d61/8958bb3d-1ab4-4fa9-968d-9ba0bebf85a9"
-					(reference "R15")
+					(reference "R21")
 					(unit 1)
 				)
@@
 		(on_board yes)
 		(dnp no)
-		(property "Reference" "R20"
+		(property "Reference" "R26"
 			(at 114.3 90.17 90)
 			(effects
@@
 			(project "turbofrank"
 				(path "/8c0b3d8b-46d3-4173-ab1e-a61765f77d61/8958bb3d-1ab4-4fa9-968d-9ba0bebf85a9"
-					(reference "R20")
+					(reference "R26")
 					(unit 1)
 				)

Commit message: 1.01 WIP
Parts:
- renumbered R21 to R19, R22 to R20, R23 to R21, R24 to R22, R25 to R23, R26 to R24, R27 to R25, R28 to R26
Changed lines of the file:
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@@
 		(on_board yes)
 		(dnp no)
-		(property "Reference" "R23"
+		(property "Reference" "R21"
 			(at 95.25 73.66 90)
 			(effects
@@
 			(project "turbofrank"
 				(path "/8c0b3d8b-46d3-4173-ab1e-a61765f77d61/8958bb3d-1ab4-4fa9-968d-9ba0bebf85a9"
-					(reference "R23")
+					(reference "R21")
 					(unit 1)
 				)
@@
 		(on_board yes)
 		(dnp no)
-		(property "Reference" "R28"
+		(property "Reference" "R26"
 			(at 177.8 95.25 90)
 			(effects
@@
 			(project "turbofrank"
 				(path "/8c0b3d8b-46d3-4173-ab1e-a61765f77d61/8958bb3d-1ab4-4fa9-968d-9ba0bebf85a9"
-					(reference "R28")
+					(reference "R26")
 					(unit 1)
 				)
@@
 		(on_board yes)
 		(dnp no)
-		(property "Reference" "R25"
+		(property "Reference" "R23"
 			(at 114.3 85.09 90)
 			(effects
@@
 			(project "turbofrank"
 				(path "/8c0b3d8b-46d3-4173-ab1e-a61765f77d61/8958bb3d-1ab4-4fa9-968d-9ba0bebf85a9"
-					(reference "R25")
+					(reference "R23")
 					(unit 1)
 				)
@@
 		(dnp no)
 		(fields_autoplaced yes)
-		(property "Reference" "#PWR039"
+		(property "Reference" "#PWR042"
 			(at 151.13 123.19 0)
 			(effects
@@
 			(project "turbofrank"
 				(path "/8c0b3d8b-46d3-4173-ab1e-a61765f77d61/8958bb3d-1ab4-4fa9-968d-9ba0bebf85a9"
-					(reference "#PWR039")
+					(reference "#PWR042")
 					(unit 1)
 				)
@@
 		(on_board yes)
 		(dnp no)
-		(property "Reference" "R24"
+		(property "Reference" "R22"
 			(at 114.3 80.01 90)
 			(effects
@@
 			(project "turbofrank"
 				(path "/8c0b3d8b-46d3-4173-ab1e-a61765f77d61/8958bb3d-1ab4-4fa9-968d-9ba0bebf85a9"
-					(reference "R24")
+					(reference "R22")
 					(unit 1)
 				)
@@
 		(on_board yes)
 		(dnp no)
-		(property "Reference" "R27"
+		(property "Reference" "R25"
 			(at 177.8 90.17 90)
 			(effects
@@
 			(project "turbofrank"
 				(path "/8c0b3d8b-46d3-4173-ab1e-a61765f77d61/8958bb3d-1ab4-4fa9-968d-9ba0bebf85a9"
-					(reference "R27")
+					(reference "R25")
 					(unit 1)
 				)
@@
 		(on_board yes)
 		(dnp no)
-		(property "Reference" "R22"
+		(property "Reference" "R20"
 			(at 95.25 68.58 90)
 			(effects
@@
 			(project "turbofrank"
 				(path "/8c0b3d8b-46d3-4173-ab1e-a61765f77d61/8958bb3d-1ab4-4fa9-968d-9ba0bebf85a9"
-					(reference "R22")
+					(reference "R20")
 					(unit 1)
 				)
@@
 		(on_board yes)
 		(dnp no)
-		(property "Reference" "R21"
+		(property "Reference" "R19"
 			(at 95.25 63.5 90)
 			(effects
@@
 			(project "turbofrank"
 				(path "/8c0b3d8b-46d3-4173-ab1e-a61765f77d61/8958bb3d-1ab4-4fa9-968d-9ba0bebf85a9"
-					(reference "R21")
+					(reference "R19")
 					(unit 1)
 				)
@@
 		(on_board yes)
 		(dnp no)
-		(property "Reference" "R26"
+		(property "Reference" "R24"
 			(at 114.3 90.17 90)
 			(effects
@@
 			(project "turbofrank"
 				(path "/8c0b3d8b-46d3-4173-ab1e-a61765f77d61/8958bb3d-1ab4-4fa9-968d-9ba0bebf85a9"
-					(reference "R26")
-					(unit 1)
-				)
+					(reference "R24")
+					(unit 1)
+				)

Commit message: Minor fixes
Parts:
- renumbered R19 to R14, R20 to R15, R21 to R16, R22 to R17, R23 to R18, R24 to R19, R25 to R20, R26 to R21
Other:
- moved on the sheet: J4, R14, R15, R16, R17, R18, R19, R20, R21

Commit message: WIP
Parts:
- renumbered J4 to J5, R14 to R23, R15 to R24, R16 to R25, R17 to R26, R18 to R27, R19 to R28, R20 to R29, R21 to R30
Changed lines of the file:
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@@
 	(title_block
 		(title "${NAME}")
-		(date "2025-07-20")
+		(date "2025-08-08")
 		(rev "${VERSION}")
 		(company "Mikhail Matveev")
@@
 		(on_board yes)
 		(dnp no)
-		(property "Reference" "R16"
+		(property "Reference" "R25"
 			(at 100.33 81.28 90)
 			(effects
@@
 			(project "turbofrank"
 				(path "/8c0b3d8b-46d3-4173-ab1e-a61765f77d61/8958bb3d-1ab4-4fa9-968d-9ba0bebf85a9"
-					(reference "R16")
+					(reference "R25")
 					(unit 1)
 				)
@@
 		(on_board yes)
 		(dnp no)
-		(property "Reference" "R21"
+		(property "Reference" "R30"
 			(at 182.88 102.87 90)
 			(effects
@@
 			(project "turbofrank"
 				(path "/8c0b3d8b-46d3-4173-ab1e-a61765f77d61/8958bb3d-1ab4-4fa9-968d-9ba0bebf85a9"
-					(reference "R21")
+					(reference "R30")
 					(unit 1)
 				)
@@
 		(dnp no)
 		(fields_autoplaced yes)
-		(property "Reference" "J4"
+		(property "Reference" "J5"
 			(at 156.21 76.2 0)
 			(effects
@@
 			(project "turbofrank"
 				(path "/8c0b3d8b-46d3-4173-ab1e-a61765f77d61/8958bb3d-1ab4-4fa9-968d-9ba0bebf85a9"
-					(reference "J4")
+					(reference "J5")
 					(unit 1)
 				)
@@
 		(on_board yes)
 		(dnp no)
-		(property "Reference" "R18"
+		(property "Reference" "R27"
 			(at 119.38 92.71 90)
 			(effects
@@
 			(project "turbofrank"
 				(path "/8c0b3d8b-46d3-4173-ab1e-a61765f77d61/8958bb3d-1ab4-4fa9-968d-9ba0bebf85a9"
-					(reference "R18")
+					(reference "R27")
 					(unit 1)
 				)
@@
 		(dnp no)
 		(fields_autoplaced yes)
-		(property "Reference" "#PWR042"
+		(property "Reference" "#PWR054"
 			(at 156.21 130.81 0)
 			(effects
@@
 			(project "turbofrank"
 				(path "/8c0b3d8b-46d3-4173-ab1e-a61765f77d61/8958bb3d-1ab4-4fa9-968d-9ba0bebf85a9"
-					(reference "#PWR042")
+					(reference "#PWR054")
 					(unit 1)
 				)
@@
 		(on_board yes)
 		(dnp no)
-		(property "Reference" "R17"
+		(property "Reference" "R26"
 			(at 119.38 87.63 90)
 			(effects
@@
 			(project "turbofrank"
 				(path "/8c0b3d8b-46d3-4173-ab1e-a61765f77d61/8958bb3d-1ab4-4fa9-968d-9ba0bebf85a9"
-					(reference "R17")
+					(reference "R26")
 					(unit 1)
 				)
@@
 		(on_board yes)
 		(dnp no)
-		(property "Reference" "R20"
+		(property "Reference" "R29"
 			(at 182.88 97.79 90)
 			(effects
@@
 			(project "turbofrank"
 				(path "/8c0b3d8b-46d3-4173-ab1e-a61765f77d61/8958bb3d-1ab4-4fa9-968d-9ba0bebf85a9"
-					(reference "R20")
+					(reference "R29")
 					(unit 1)
 				)
@@
 		(on_board yes)
 		(dnp no)
-		(property "Reference" "R15"
+		(property "Reference" "R24"
 			(at 100.33 76.2 90)
 			(effects
@@
 			(project "turbofrank"
 				(path "/8c0b3d8b-46d3-4173-ab1e-a61765f77d61/8958bb3d-1ab4-4fa9-968d-9ba0bebf85a9"
-					(reference "R15")
+					(reference "R24")
 					(unit 1)
 				)
@@
 		(on_board yes)
 		(dnp no)
-		(property "Reference" "R14"
+		(property "Reference" "R23"
 			(at 100.33 71.12 90)
 			(effects
@@
 			(project "turbofrank"
 				(path "/8c0b3d8b-46d3-4173-ab1e-a61765f77d61/8958bb3d-1ab4-4fa9-968d-9ba0bebf85a9"
-					(reference "R14")
+					(reference "R23")
 					(unit 1)
 				)
@@
 		(on_board yes)
 		(dnp no)
-		(property "Reference" "R19"
+		(property "Reference" "R28"
 			(at 119.38 97.79 90)
 			(effects
@@
 			(project "turbofrank"
 				(path "/8c0b3d8b-46d3-4173-ab1e-a61765f77d61/8958bb3d-1ab4-4fa9-968d-9ba0bebf85a9"
-					(reference "R19")
+					(reference "R28")
 					(unit 1)
 				)

Commit message: Rev 1.05 WIP
Parts:
- removed J5: D-SUB 15 Female, FRANK:D-SUB (15 pin, female), symbol FRANK:VGA
- added C11, C19, C20, C24, C27: 10u, FRANK:Capacitor (0603), symbol Device:C
- added C12, C13, C14, C15, C16, C17, C18, C22, C23: 100n, FRANK:Capacitor (0603), symbol Device:C
- added C21, C25, C36, C37: 1u, FRANK:Capacitor (0603), symbol Device:C
- added C26: 1n, FRANK:Capacitor (0603), symbol Device:C
- added C28, C30, C32: 220n, FRANK:Capacitor (0603), symbol Device:C
- added C29, C31, C33: 4.7u, FRANK:Capacitor (0603), symbol Device:C
- added C34, C35: 15p, FRANK:Capacitor (0603), symbol Device:C
- added D1: 1N5819WS, FRANK:Diode (SOD-323), symbol Device:D_Schottky
- added FB1, FB2: 220R, FRANK:Inductor (0805), symbol Device:FerriteBead
- added J4: DC3RX19JA2, FRANK:HDMI (female), symbol FRANK:HDMI
- added R31: 75R, FRANK:Resistor (0603), symbol Device:R
- added R32, R33: 100R, FRANK:Resistor (0603), symbol Device:R
- added R34, R35: 2K, FRANK:Resistor (0603), symbol Device:R
- added R36: 1K, FRANK:Resistor (0603), symbol Device:R
- added R37, R38: 4.7K, FRANK:Resistor (0603), symbol Device:R
- added TP1: MS9288_SCL, FRANK:TestPoint (Pad 1.0x1.0mm), symbol Connector:TestPoint
- added TP2: MS9288_SDA, FRANK:TestPoint (Pad 1.0x1.0mm), symbol Connector:TestPoint
- added U7: AMS1117-3.3, FRANK:SOT-223, symbol Regulator_Linear:AMS1117-3.3
- added U8: AMS1117-1.8, FRANK:SOT-223, symbol Regulator_Linear:AMS1117-1.8
- added U9: MS9288A, FRANK:QFN 48, symbol FRANK:MS9288A
- added X1: 24.576 MHz, FRANK:Crystal (2520), symbol FRANK:Crystal_25.576MHz
- R23, R25: value 330R -> 806R; footprint FRANK:Resistor (0805) -> FRANK:Resistor (0603)
- R24: value 330R -> 402R; footprint FRANK:Resistor (0805) -> FRANK:Resistor (0603)
- R26, R28: value 1K -> 402R; footprint FRANK:Resistor (0805) -> FRANK:Resistor (0603)
- R27: value 1K -> 806R; footprint FRANK:Resistor (0805) -> FRANK:Resistor (0603)
- R29, R30: value 100R -> 75R; footprint FRANK:Resistor (0805) -> FRANK:Resistor (0603)
Connections:
- net GND: now also R29.2, R30.2, C11.2, C13.2, C14.2, C15.2, C16.2, C17.2, C19.2, C20.2, C21.2, C23.2, C24.2, C25.2, C27.2, C28.2, C29.2, C30.2, C31.2, C32.2, C33.2, C34.2, C35.2, J4.11 (G_CLK), J4.17 (G_DDC/CEC), J4.2 (G_D2), J4.20 (SHIELD1), J4.21 (SHIELD2), J4.22 (SHIELD3), J4.23 (SHIELD4), J4.5 (G_D1), J4.8 (G_D0), R31.2, R36.1, U7.1 (GND), U8.1 (GND), U9.2 (GND), U9.27 (GND), U9.40 (GND), U9.45 (GND), U9.49 (EP), U9.6 (GND), X1.2 (GND), X1.4 (GND)
- net VGA_B: now also R23.1; no longer R28.1
- net VGA_BH: now also R24.1; no longer R25.1
- net VGA_G: now also R25.1; no longer R27.1
- net VGA_GH: now also R26.1; no longer R24.1
- net VGA_HS: now also R32.1; no longer R29.2
- net VGA_R: now also R27.1; no longer R26.1
- net VGA_RH: now also R28.1; no longer R23.1
- net VGA_VS: now also R33.1; no longer R30.2
- net at R28.2: now also R27.2, R29.1, C22.2; no longer R25.2
- net SOG_G: now reaches R30.1
- net SOG_G: now also R25.2, R26.2, C18.2, C26.2
- net at R23.2: now also R24.2, C12.2, R31.1; no longer R26.2
- new net: C34.1, U9.26 (XTO), X1.3 (OSC)
- new net: C28.1, C29.1, U9.31 (REFQ0)
- new net: C30.1, C31.1, U9.32 (REFQ1)
- new net: C32.1, C33.1, U9.37 (REFP)
- new net: R36.2, U9.13 (SWREF1k)
- new net: D1.1 (K), J4.18 (+5V)
- new net: C35.1, U9.25 (XTI), X1.1 (OSC)
- new net: R32.2, U9.34 (HSIN)
- new net: C26.1, U9.42 (SOG/Y)
- new net: R33.2, U9.35 (VSIN)
- new net ALIN: C36.1, U9.30 (ALIN)
- new net AMS_1V8: C15.1, C24.1, C25.1, FB2.1, U8.2 (VO), U9.16 (AVDD18), U9.21 (AVDD18), U9.7 (AVDD18)
- new net AMS_1V8A: C13.1, C14.1, C27.1, FB2.2, U9.1 (AVDD18_ADC), U9.41 (AVDD18_ADC), U9.46 (AVDD18_ADC)
- new net AMS_3V3: C17.1, C20.1, C21.1, FB1.2, U7.2 (VO), U9.11 (DVDD33), U9.24 (DVDD33), U9.36 (DVDD33), U9.5 (DVDD33)
- new net AMS_3V3A: C11.1, C16.1, FB1.1, U9.12 (AVDD33), U9.38 (AVDD33), U9.43 (AVDD33), U9.47 (AVDD33)
- new net ARIN: C37.1, U9.33 (ARIN)
- new net AUDIO_IN_L: C36.2
- new net AUDIO_IN_R: C37.2
- new net B: C12.1, U9.39 (B/Pb)
- new net DCCSCL: J4.15 (SCL), R34.1, U9.10 (DCCSCL)
- new net DDCSDA: J4.16 (SDA), R35.1, U9.9 (DDCSDA)
- new net G: C18.1, U9.44 (G/Y)
- new net HPDT: J4.19 (HOT_PLUG_DET), U9.8 (HotPlugDetect)
- new net R: C22.1, U9.48 (R/Pr)
- new net SCL: R37.1, TP1.1, U9.28 (SCL)
- new net SDA: R38.1, TP2.1, U9.29 (SDA)
- new net TMDS_CLK+: J4.10 (CLKP), U9.15 (TMDS_CLK+)
- new net TMDS_CLK-: J4.12 (CLKN), U9.14 (TMDS_CLK-)
- new net TMDS_D0+: J4.7 (D0P), U9.18 (TMDS-D0+)
- new net TMDS_D0-: J4.9 (D0N), U9.17 (TMDS_D0-)
- new net TMDS_D1+: J4.4 (D1P), U9.20 (TMDS_D1+)
- new net TMDS_D1-: J4.6 (D1N), U9.19 (TMDS_D1-)
- new net TMDS_D2+: J4.1 (D2P), U9.23 (TMDS_D2+)
- new net TMDS_D2-: J4.3 (D2N), U9.22 (TMDS_D2-)
- new net VBUS: C19.1, C23.1, D1.2 (A), R34.2, R35.2, R37.2, R38.2, U7.3 (VI), U8.3 (VI)
- no-connect marks 5 -> 4
