File: vga.kicad_sch (KiCad schematic)
At the start: 53 parts, among them J4 DC3RX19JA2, U7 AMS1117-3.3, U8 AMS1117-1.8, U9 MS9288A, X1 24.576 MHz

Commit message: HW 1.06 WIP
Parts:
- renumbered C28 to C25, C29 to C26, C30 to C27, C31 to C28, C12 to C29, C18 to C30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
