File: esp32.kicad_sch (KiCad schematic)
At the start: 3 parts, among them U5 ESP32-WROOM-32

Commit message: 1.01 WIP
Parts:
- removed C10: 100n, FRANK:Capacitor (0805), symbol Device:C
- removed C9: 10u, FRANK:Capacitor (0805), symbol Device:C
- removed U5: ESP32-WROOM-32, RF_Module:ESP32-WROOM-32, symbol RF_Module:ESP32-WROOM-32
- added C7: 10u, FRANK:Capacitor (0805), symbol Device:C
- added C8: 100n, FRANK:Capacitor (0805), symbol Device:C
- added U5: ESP32-WROVER-E, FRANK:ESP32-WROVER-E, symbol FRANK:ESP32-WROVER-E
Connections:
- net +3V3: now also C7.1, C8.1, U5.2 (3V3)
- net EN: now also U5.3 (EN/CHIP_PU)
- net GND: now also C7.2, C8.2, U5.1 (GND), U5.15 (GND), U5.38 (GND), U5.39 (GND_THERMAL)
- net IO0: now also U5.25 (GPIO0/BOOT/ADC2_CH1)
- net IO1: now also U5.35 (U0TXD/GPIO1)
- net IO12: now also U5.14 (MTDI/GPIO12/ADC2_CH5)
- net IO13: now also U5.16 (MTCK/GPIO13/ADC2_CH4)
- net IO14: now also U5.13 (MTMS/GPIO14/ADC2_CH6)
- net IO15: now also U5.23 (MTDO/GPIO15/ADC2_CH3)
- net IO18: now also U5.30 (GPIO18)
- net IO19: now also U5.31 (GPIO19)
- net IO2: now also U5.24 (ADC2_CH2/GPIO2)
- net IO21: now also U5.33 (GPIO21)
- net IO22: now also U5.36 (GPIO22)
- net IO23: now also U5.37 (GPIO23)
- net IO25: now also U5.10 (DAC_1/ADC2_CH8/GPIO25)
- net IO26: now also U5.11 (DAC_2/ADC2_CH9/GPIO26)
- net IO27: now also U5.12 (ADC2_CH7/GPIO27)
- net IO3: now also U5.34 (U0RXD/GPIO3)
- net IO32: now also U5.8 (32K_XP/GPIO32/ADC1_CH4)
- net IO33: now also U5.9 (32K_XN/GPIO33/ADC1_CH5)
- net IO34: now also U5.6 (GPIO34/ADC1_CH6)
- net IO35: now also U5.7 (GPIO35/ADC1_CH7)
- net IO4: now also U5.26 (ADC2_CH0/GPIO4)
- net IO5: now also U5.29 (GPIO5)
- net SENSOR_VN: now also U5.5 (SENSOR_VN/GPIO39/ADC1_CH3)
- net SENSOR_VP: now also U5.4 (SENSOR_VP/GPIO36/ADC1_CH0)

Commit message: Minor fixes
Parts:
- renumbered C7 to C8, C8 to C9
Connections:
- net SENSOR_VN renamed IO39
- net SENSOR_VP renamed IO36
Changed lines of the file:
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@@
 	(title_block
 		(title "${NAME}")
-		(date "2025-05-24")
+		(date "2025-06-23")
 		(rev "${VERSION}")
 		(company "Mikhail Matveev")
@@
 		)
 	)
-	(hierarchical_label "SENSOR_VP"
+	(hierarchical_label "IO36"
 		(shape input)
 		(at 105.41 115.57 180)
@@
 		)
 	)
-	(hierarchical_label "SENSOR_VN"
+	(hierarchical_label "IO39"
 		(shape input)
 		(at 105.41 118.11 180)
@@
 		(on_board yes)
 		(dnp no)
-		(property "Reference" "#PWR031"
+		(property "Reference" "#PWR035"
 			(at 157.48 143.51 0)
 			(effects
@@
 			(project "echo"
 				(path "/8c0b3d8b-46d3-4173-ab1e-a61765f77d61/77c89b3c-77eb-4110-a91f-a0bd1c85adbc"
-					(reference "#PWR031")
+					(reference "#PWR035")
 					(unit 1)
 				)
@@
 		(on_board yes)
 		(dnp no)
-		(property "Reference" "#PWR028"
+		(property "Reference" "#PWR032"
 			(at 139.7 39.37 0)
 			(effects
@@
 			(project "echo"
 				(path "/8c0b3d8b-46d3-4173-ab1e-a61765f77d61/77c89b3c-77eb-4110-a91f-a0bd1c85adbc"
-					(reference "#PWR028")
+					(reference "#PWR032")
 					(unit 1)
 				)
@@
 		(on_board yes)
 		(dnp no)
-		(property "Reference" "C7"
+		(property "Reference" "C8"
 			(at 136.779 58.3184 0)
 			(effects
@@
 			(project "echo"
 				(path "/8c0b3d8b-46d3-4173-ab1e-a61765f77d61/77c89b3c-77eb-4110-a91f-a0bd1c85adbc"
-					(reference "C7")
+					(reference "C8")
 					(unit 1)
 				)
@@
 		(on_board yes)
 		(dnp no)
-		(property "Reference" "C8"
+		(property "Reference" "C9"
 			(at 149.479 58.3184 0)
 			(effects
@@
 			(project "echo"
 				(path "/8c0b3d8b-46d3-4173-ab1e-a61765f77d61/77c89b3c-77eb-4110-a91f-a0bd1c85adbc"
-					(reference "C8")
+					(reference "C9")
 					(unit 1)
 				)
@@
 		(on_board yes)
 		(dnp no)
-		(property "Reference" "#PWR029"
+		(property "Reference" "#PWR033"
 			(at 165.1 67.31 0)
 			(effects
@@
 			(project "echo"
 				(path "/8c0b3d8b-46d3-4173-ab1e-a61765f77d61/77c89b3c-77eb-4110-a91f-a0bd1c85adbc"
-					(reference "#PWR029")
+					(reference "#PWR033")
 					(unit 1)
 				)
@@
 		(on_board yes)
 		(dnp no)
-		(property "Reference" "#PWR030"
+		(property "Reference" "#PWR034"
 			(at 154.94 143.51 0)
 			(effects
@@
 			(project "echo"
 				(path "/8c0b3d8b-46d3-4173-ab1e-a61765f77d61/77c89b3c-77eb-4110-a91f-a0bd1c85adbc"
-					(reference "#PWR030")
+					(reference "#PWR034")
 					(unit 1)
 				)

Commit message: HW Rev 1.03
Parts:
- renumbered C8 to C7, C9 to C8
Changed lines of the file:
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@@
 	(title_block
 		(title "${NAME}")
-		(date "2025-06-23")
+		(date "2025-07-20")
 		(rev "${VERSION}")
 		(company "Mikhail Matveev")
@@
 		(on_board yes)
 		(dnp no)
-		(property "Reference" "C8"
+		(property "Reference" "C7"
 			(at 136.779 58.3184 0)
 			(effects
@@
 			(project "echo"
 				(path "/8c0b3d8b-46d3-4173-ab1e-a61765f77d61/77c89b3c-77eb-4110-a91f-a0bd1c85adbc"
-					(reference "C8")
+					(reference "C7")
 					(unit 1)
 				)
@@
 		(on_board yes)
 		(dnp no)
-		(property "Reference" "C9"
+		(property "Reference" "C8"
 			(at 149.479 58.3184 0)
 			(effects
@@
 			(project "echo"
 				(path "/8c0b3d8b-46d3-4173-ab1e-a61765f77d61/77c89b3c-77eb-4110-a91f-a0bd1c85adbc"
-					(reference "C9")
+					(reference "C8")
 					(unit 1)
 				)

Commit message: WIP
Parts:
- renumbered C7 to C8, C8 to C9, U5 to U6
Changed lines of the file:
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@@
 	(title_block
 		(title "${NAME}")
-		(date "2025-07-20")
+		(date "2025-08-08")
 		(rev "${VERSION}")
 		(company "Mikhail Matveev")
@@
 		(on_board yes)
 		(dnp no)
-		(property "Reference" "#PWR035"
+		(property "Reference" "#PWR047"
 			(at 157.48 143.51 0)
 			(effects
@@
 			(project "echo"
 				(path "/8c0b3d8b-46d3-4173-ab1e-a61765f77d61/77c89b3c-77eb-4110-a91f-a0bd1c85adbc"
-					(reference "#PWR035")
+					(reference "#PWR047")
 					(unit 1)
 				)
@@
 		(on_board yes)
 		(dnp no)
-		(property "Reference" "#PWR032"
+		(property "Reference" "#PWR044"
 			(at 139.7 39.37 0)
 			(effects
@@
 			(project "echo"
 				(path "/8c0b3d8b-46d3-4173-ab1e-a61765f77d61/77c89b3c-77eb-4110-a91f-a0bd1c85adbc"
-					(reference "#PWR032")
+					(reference "#PWR044")
 					(unit 1)
 				)
@@
 		(on_board yes)
 		(dnp no)
-		(property "Reference" "C7"
+		(property "Reference" "C8"
 			(at 136.779 58.3184 0)
 			(effects
@@
 			(project "echo"
 				(path "/8c0b3d8b-46d3-4173-ab1e-a61765f77d61/77c89b3c-77eb-4110-a91f-a0bd1c85adbc"
-					(reference "C7")
+					(reference "C8")
 					(unit 1)
 				)
@@
 		(on_board yes)
 		(dnp no)
-		(property "Reference" "C8"
+		(property "Reference" "C9"
 			(at 149.479 58.3184 0)
 			(effects
@@
 			(project "echo"
 				(path "/8c0b3d8b-46d3-4173-ab1e-a61765f77d61/77c89b3c-77eb-4110-a91f-a0bd1c85adbc"
-					(reference "C8")
+					(reference "C9")
 					(unit 1)
 				)
@@
 		(on_board yes)
 		(dnp no)
-		(property "Reference" "#PWR033"
+		(property "Reference" "#PWR045"
 			(at 165.1 67.31 0)
 			(effects
@@
 			(project "echo"
 				(path "/8c0b3d8b-46d3-4173-ab1e-a61765f77d61/77c89b3c-77eb-4110-a91f-a0bd1c85adbc"
-					(reference "#PWR033")
+					(reference "#PWR045")
 					(unit 1)
 				)
@@
 		(dnp no)
 		(fields_autoplaced yes)
-		(property "Reference" "U5"
+		(property "Reference" "U6"
 			(at 157.0833 77.47 0)
 			(effects
@@
 			(project ""
 				(path "/8c0b3d8b-46d3-4173-ab1e-a61765f77d61/77c89b3c-77eb-4110-a91f-a0bd1c85adbc"
-					(reference "U5")
+					(reference "U6")
 					(unit 1)
 				)
@@
 		(on_board yes)
 		(dnp no)
-		(property "Reference" "#PWR034"
+		(property "Reference" "#PWR046"
 			(at 154.94 143.51 0)
 			(effects
@@
 			(project "echo"
 				(path "/8c0b3d8b-46d3-4173-ab1e-a61765f77d61/77c89b3c-77eb-4110-a91f-a0bd1c85adbc"
-					(reference "#PWR034")
+					(reference "#PWR046")
 					(unit 1)
 				)

Commit message: Rev 1.05 WIP
Parts:
- C8, C9: footprint FRANK:Capacitor (0805) -> FRANK:Capacitor (0603)
Changed lines of the file:
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@@
 			)
 		)
-		(property "Footprint" "FRANK:Capacitor (0805)"
+		(property "Footprint" "FRANK:Capacitor (0603)"
 			(at 138.7348 53.34 0)
 			(effects
@@
 			)
 		)
-		(property "Footprint" "FRANK:Capacitor (0805)"
+		(property "Footprint" "FRANK:Capacitor (0603)"
 			(at 151.4348 53.34 0)
 			(effects

Commit message: HW 1.06 WIP
Parts:
- removed C8: 10u, FRANK:Capacitor (0603), symbol Device:C
- removed C9: 100n, FRANK:Capacitor (0603), symbol Device:C
- removed U6: ESP32-WROVER-E, FRANK:ESP32-WROVER-E, symbol FRANK:ESP32-WROVER-E
- added AE1: Antenna_Shield, FRANK:Antenna (2.4GHz), symbol Device:Antenna_Shield
- added C10, C11, C14, C15, C21, C22, C23: 100n, FRANK:Capacitor (0603), symbol Device:C
- added C12, C13: 15p, FRANK:Capacitor (0603), symbol Device:C
- added C16: 10uF, FRANK:Capacitor (0603), symbol Device:C
- added C17, C20: 1uF, FRANK:Capacitor (0603), symbol Device:C
- added C18: 10nF, FRANK:Capacitor (0603), symbol Device:C
- added C19: 3.3nF, FRANK:Capacitor (0603), symbol Device:C
- added C8: 2.4pF, FRANK:Capacitor (0603), symbol Device:C_Small
- added C9: 1.5pF, FRANK:Capacitor (0603), symbol Device:C_Small
- added L1: 3nH, FRANK:Inductor (0603 1.05x0.95), symbol Device:L_Small
- added L2: 2.2nH, FRANK:Inductor (0603 1.05x0.95), symbol Device:L_Small
- added LD4: Blue, FRANK:LED (0603), symbol Device:LED
- added R23, R24, R27: 0R, FRANK:Resistor (0603), symbol Device:R
- added R25: 10K, FRANK:Resistor (0603), symbol Device:R
- added R26: 499R, FRANK:Resistor (0603), symbol Device:R
- added R28: 20K, FRANK:Resistor (0603), symbol Device:R
- added R29: 5.1K, FRANK:Resistor (0603), symbol Device:R
- added U6: W25Q32JVSIQ, FRANK:SOIC-8 (Longer), symbol FRANK:Flash_W25Q128JVS
- added U7: ESP32-D0WD, FRANK:QFN48_ESP32-D0WD-V3_EXP, symbol FRANK:ESP32-D0WD-V3
- added U8: ESP-PSRAM32, FRANK:SO-8, symbol FRANK:ESP-PSRAM32
- added Y1: 40 MHz, FRANK:Crystal (3225), symbol Device:Crystal_GND24
Connections:
- net +3V3: now also C10.2, C11.2, C15.2, C16.2, C17.2, C21.2, C22.2, C23.2, L2.2, R29.2
- net EN: now also U7.9 (CHIP_PU)
- net GND: now also AE1.2 (Shield), C12.2, C13.2, C14.1, C15.1, C16.1, C17.1, C18.1, C20.1, C8.2, C9.2, U6.4 (GND), U7.49 (GND), U8.4 (VSS), Y1.2, Y1.4
- net IO0: now also U7.23 (GPIO0)
- net IO1: now also R26.2
- net IO12: now also U7.18 (MTDI)
- net IO13: now also U7.20 (MTCK)
- net IO14: now also U7.17 (MTMS)
- net IO15: now also U7.21 (MTDO)
- net IO18: now also U7.35 (GPIO18)
- net IO19: now also U7.38 (GPIO19)
- net IO2: now also U7.22 (GPIO2)
- net IO21: now also U7.42 (GPIO21)
- net IO22: now also LD4.1 (K), U7.39 (GPIO22)
- net IO23: now also U7.36 (GPIO23)
- net IO25: now also U7.14 (GPIO25)
- net IO26: now also U7.15 (GPIO26)
- net IO27: now also U7.16 (GPIO27)
- net IO3: now also U7.40 (U0RXD)
- net IO32: now also U7.12 (32K_XP)
- net IO33: now also U7.13 (32K_XN)
- net IO34: now also U7.10 (VDET_1)
- net IO35: now also U7.11 (VDET_2)
- net IO36: now also U7.5 (SENSOR_VP)
- net IO39: now also U7.8 (SENSOR_VN)
- net IO4: now also U7.24 (GPIO4)
- net IO5: now also U7.34 (GPIO5)
- new net: R26.1, U7.41 (U0TXD)
- new net: C21.1, U7.46 (VDDA)
- new net: C9.1, L1.2, U7.2 (LNA_IN)
- new net: C13.1, R23.2, Y1.1
- new net: LD4.2 (A), R29.1
- new net: C11.1, U7.19 (VDD3P3_RTC)
- new net: C10.1, U7.1 (VDDA)
- new net: C22.1, U7.43 (VDDA)
- new net: R27.1, U7.25 (GPIO16)
- new net: C23.1, U7.37 (VDD3P3_CPU)
- new net: R24.1, U8.6 (SCLK)
- new net +3.3VP: C14.2, L2.1, U7.3 (VDD3P3), U7.4 (VDD3P3)
- new net ANT: AE1.1 (A), C8.1, L1.1
- new net CAP1: C18.2, C19.2, R28.1, U7.48 (CAP1)
- new net CAP2: C19.1, R28.2, U7.47 (CAP2)
- new net IO16: R25.1, R27.2, U8.1 (~{CE})
- new net IO17: R24.2, U7.27 (GPIO17)
- new net IO37: U7.6 (SENSOR_CAPP)
- new net IO38: U7.7 (SENSOR_CAPN)
- new net SCK/CLK: U6.6 (CLK), U7.31 (SD_CLK)
- new net SCS/CMD: U6.1 (~{CS}), U7.30 (SD_CMD)
- new net SDI/SD1: U6.5 (DI(IO0)), U7.33 (SD_DATA_1), U8.5 (SI/SIO)
- new net SDO/SD0: U6.2 (DO(IO1)), U7.32 (SD_DATA_0), U8.2 (SO/SIO)
- new net SHD/SD2: U6.7 (IO3), U7.28 (SD_DATA_2), U8.7 (SIO3)
- new net SWP/SD3: U6.3 (IO2), U7.29 (SD_DATA_3), U8.3 (SIO2)
- new net VDD_SDIO: C20.2, R25.2, U6.8 (VCC), U7.26 (VDD_SDIO), U8.8 (VCC)
- new net XIN: R23.1, U7.45 (XTAL_P)
- new net XOUT: C12.1, U7.44 (XTAL_N), Y1.3
