File: level_shifter.kicad_sch (KiCad schematic)
At the start: 4 parts, among them Q3 AO3400A

Commit message: WIP
Parts:
- renumbered R22 to R31, R23 to R32, R24 to R33
Changed lines of the file:
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@@
 	(title_block
 		(title "${NAME}")
-		(date "2025-07-20")
+		(date "2025-08-08")
 		(rev "${VERSION}")
 		(company "Mikhail Matveev")
@@
 		(on_board yes)
 		(dnp no)
-		(property "Reference" "R24"
+		(property "Reference" "R33"
 			(at 161.29 93.98 0)
 			(effects
@@
 			(project "echo"
 				(path "/8c0b3d8b-46d3-4173-ab1e-a61765f77d61/4252f457-35b5-4f79-9561-ecba9662200c"
-					(reference "R39")
+					(reference "R48")
 					(unit 1)
 				)
 				(path "/8c0b3d8b-46d3-4173-ab1e-a61765f77d61/ca9d4364-8864-42d1-89eb-99280f8ed67d"
-					(reference "R24")
+					(reference "R33")
 					(unit 1)
 				)
 				(path "/8c0b3d8b-46d3-4173-ab1e-a61765f77d61/f55e411b-ec4b-43e8-a550-3df1b34591c7"
-					(reference "R27")
+					(reference "R36")
 					(unit 1)
 				)
 				(path "/8c0b3d8b-46d3-4173-ab1e-a61765f77d61/f647f155-e741-47c8-b191-8b4f6021bf8f"
-					(reference "R42")
+					(reference "R51")
 					(unit 1)
 				)
@@
 		(on_board yes)
 		(dnp no)
-		(property "Reference" "#PWR051"
+		(property "Reference" "#PWR063"
 			(at 160.02 95.25 0)
 			(effects
@@
 			(project "echo"
 				(path "/8c0b3d8b-46d3-4173-ab1e-a61765f77d61/4252f457-35b5-4f79-9561-ecba9662200c"
-					(reference "#PWR074")
+					(reference "#PWR086")
 					(unit 1)
 				)
 				(path "/8c0b3d8b-46d3-4173-ab1e-a61765f77d61/ca9d4364-8864-42d1-89eb-99280f8ed67d"
-					(reference "#PWR051")
+					(reference "#PWR063")
 					(unit 1)
 				)
 				(path "/8c0b3d8b-46d3-4173-ab1e-a61765f77d61/f55e411b-ec4b-43e8-a550-3df1b34591c7"
-					(reference "#PWR053")
+					(reference "#PWR065")
 					(unit 1)
 				)
 				(path "/8c0b3d8b-46d3-4173-ab1e-a61765f77d61/f647f155-e741-47c8-b191-8b4f6021bf8f"
-					(reference "#PWR076")
+					(reference "#PWR088")
 					(unit 1)
 				)
@@
 		(on_board yes)
 		(dnp no)
-		(property "Reference" "R22"
+		(property "Reference" "R31"
 			(at 139.446 93.98 0)
 			(effects
@@
 			(project "echo"
 				(path "/8c0b3d8b-46d3-4173-ab1e-a61765f77d61/4252f457-35b5-4f79-9561-ecba9662200c"
-					(reference "R37")
+					(reference "R46")
 					(unit 1)
 				)
 				(path "/8c0b3d8b-46d3-4173-ab1e-a61765f77d61/ca9d4364-8864-42d1-89eb-99280f8ed67d"
-					(reference "R22")
+					(reference "R31")
 					(unit 1)
 				)
 				(path "/8c0b3d8b-46d3-4173-ab1e-a61765f77d61/f55e411b-ec4b-43e8-a550-3df1b34591c7"
-					(reference "R25")
+					(reference "R34")
 					(unit 1)
 				)
 				(path "/8c0b3d8b-46d3-4173-ab1e-a61765f77d61/f647f155-e741-47c8-b191-8b4f6021bf8f"
-					(reference "R40")
+					(reference "R49")
 					(unit 1)
 				)
@@
 		(on_board yes)
 		(dnp no)
-		(property "Reference" "R23"
+		(property "Reference" "R32"
 			(at 152.4 93.98 0)
 			(effects
@@
 			(project "echo"
 				(path "/8c0b3d8b-46d3-4173-ab1e-a61765f77d61/4252f457-35b5-4f79-9561-ecba9662200c"
-					(reference "R38")
+					(reference "R47")
 					(unit 1)
 				)
 				(path "/8c0b3d8b-46d3-4173-ab1e-a61765f77d61/ca9d4364-8864-42d1-89eb-99280f8ed67d"
-					(reference "R23")
+					(reference "R32")
 					(unit 1)
 				)
 				(path "/8c0b3d8b-46d3-4173-ab1e-a61765f77d61/f55e411b-ec4b-43e8-a550-3df1b34591c7"
-					(reference "R26")
+					(reference "R35")
 					(unit 1)
 				)
 				(path "/8c0b3d8b-46d3-4173-ab1e-a61765f77d61/f647f155-e741-47c8-b191-8b4f6021bf8f"
-					(reference "R41")
+					(reference "R50")
 					(unit 1)
 				)
@@
 		(dnp no)
 		(fields_autoplaced yes)
-		(property "Reference" "#PWR050"
+		(property "Reference" "#PWR062"
 			(at 151.13 90.17 0)
 			(effects
@@
 			(project "echo"
 				(path "/8c0b3d8b-46d3-4173-ab1e-a61765f77d61/4252f457-35b5-4f79-9561-ecba9662200c"
-					(reference "#PWR073")
+					(reference "#PWR085")
 					(unit 1)
 				)
 				(path "/8c0b3d8b-46d3-4173-ab1e-a61765f77d61/ca9d4364-8864-42d1-89eb-99280f8ed67d"
-					(reference "#PWR050")
+					(reference "#PWR062")
 					(unit 1)
 				)
 				(path "/8c0b3d8b-46d3-4173-ab1e-a61765f77d61/f55e411b-ec4b-43e8-a550-3df1b34591c7"
-					(reference "#PWR052")
+					(reference "#PWR064")
 					(unit 1)
 				)
 				(path "/8c0b3d8b-46d3-4173-ab1e-a61765f77d61/f647f155-e741-47c8-b191-8b4f6021bf8f"
-					(reference "#PWR075")
-					(unit 1)
-				)
+					(reference "#PWR087")
+					(unit 1)
+				)

Commit message: Rev 1.05 WIP
Parts:
- R39: renamed from R31; footprint FRANK:Resistor (0805) -> FRANK:Resistor (0603)
- R40: renamed from R32; footprint FRANK:Resistor (0805) -> FRANK:Resistor (0603)
- R41: renamed from R33; footprint FRANK:Resistor (0805) -> FRANK:Resistor (0603)
Changed lines of the file:
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@@
 		(on_board yes)
 		(dnp no)
-		(property "Reference" "R33"
+		(property "Reference" "R41"
 			(at 161.29 93.98 0)
 			(effects
@@
 			)
 		)
-		(property "Footprint" "FRANK:Resistor (0805)"
+		(property "Footprint" "FRANK:Resistor (0603)"
 			(at 158.242 95.25 90)
 			(effects
@@
 			(project "echo"
 				(path "/8c0b3d8b-46d3-4173-ab1e-a61765f77d61/4252f457-35b5-4f79-9561-ecba9662200c"
-					(reference "R48")
+					(reference "R59")
 					(unit 1)
 				)
 				(path "/8c0b3d8b-46d3-4173-ab1e-a61765f77d61/ca9d4364-8864-42d1-89eb-99280f8ed67d"
-					(reference "R33")
+					(reference "R41")
 					(unit 1)
 				)
 				(path "/8c0b3d8b-46d3-4173-ab1e-a61765f77d61/f55e411b-ec4b-43e8-a550-3df1b34591c7"
-					(reference "R36")
+					(reference "R44")
 					(unit 1)
 				)
 				(path "/8c0b3d8b-46d3-4173-ab1e-a61765f77d61/f647f155-e741-47c8-b191-8b4f6021bf8f"
-					(reference "R51")
+					(reference "R62")
 					(unit 1)
 				)
@@
 		(on_board yes)
 		(dnp no)
-		(property "Reference" "#PWR063"
+		(property "Reference" "#PWR093"
 			(at 160.02 95.25 0)
 			(effects
@@
 			(project "echo"
 				(path "/8c0b3d8b-46d3-4173-ab1e-a61765f77d61/4252f457-35b5-4f79-9561-ecba9662200c"
-					(reference "#PWR086")
+					(reference "#PWR0120")
 					(unit 1)
 				)
 				(path "/8c0b3d8b-46d3-4173-ab1e-a61765f77d61/ca9d4364-8864-42d1-89eb-99280f8ed67d"
-					(reference "#PWR063")
+					(reference "#PWR093")
 					(unit 1)
 				)
 				(path "/8c0b3d8b-46d3-4173-ab1e-a61765f77d61/f55e411b-ec4b-43e8-a550-3df1b34591c7"
-					(reference "#PWR065")
+					(reference "#PWR095")
 					(unit 1)
 				)
 				(path "/8c0b3d8b-46d3-4173-ab1e-a61765f77d61/f647f155-e741-47c8-b191-8b4f6021bf8f"
-					(reference "#PWR088")
+					(reference "#PWR0122")
 					(unit 1)
 				)
@@
 		(on_board yes)
 		(dnp no)
-		(property "Reference" "R31"
+		(property "Reference" "R39"
 			(at 139.446 93.98 0)
 			(effects
@@
 			)
 		)
-		(property "Footprint" "FRANK:Resistor (0805)"
+		(property "Footprint" "FRANK:Resistor (0603)"
 			(at 143.002 95.25 90)
 			(effects
@@
 			(project "echo"
 				(path "/8c0b3d8b-46d3-4173-ab1e-a61765f77d61/4252f457-35b5-4f79-9561-ecba9662200c"
-					(reference "R46")
+					(reference "R57")
 					(unit 1)
 				)
 				(path "/8c0b3d8b-46d3-4173-ab1e-a61765f77d61/ca9d4364-8864-42d1-89eb-99280f8ed67d"
-					(reference "R31")
+					(reference "R39")
 					(unit 1)
 				)
 				(path "/8c0b3d8b-46d3-4173-ab1e-a61765f77d61/f55e411b-ec4b-43e8-a550-3df1b34591c7"
-					(reference "R34")
+					(reference "R42")
 					(unit 1)
 				)
 				(path "/8c0b3d8b-46d3-4173-ab1e-a61765f77d61/f647f155-e741-47c8-b191-8b4f6021bf8f"
-					(reference "R49")
+					(reference "R60")
 					(unit 1)
 				)
@@
 			(project "echo"
 				(path "/8c0b3d8b-46d3-4173-ab1e-a61765f77d61/4252f457-35b5-4f79-9561-ecba9662200c"
-					(reference "Q5")
+					(reference "Q7")
 					(unit 1)
 				)
@@
 				)
 				(path "/8c0b3d8b-46d3-4173-ab1e-a61765f77d61/f647f155-e741-47c8-b191-8b4f6021bf8f"
-					(reference "Q6")
+					(reference "Q8")
 					(unit 1)
 				)
@@
 		(on_board yes)
 		(dnp no)
-		(property "Reference" "R32"
+		(property "Reference" "R40"
 			(at 152.4 93.98 0)
 			(effects
@@
 			)
 		)
-		(property "Footprint" "FRANK:Resistor (0805)"
+		(property "Footprint" "FRANK:Resistor (0603)"
 			(at 149.352 95.25 90)
 			(effects
@@
 			(project "echo"
 				(path "/8c0b3d8b-46d3-4173-ab1e-a61765f77d61/4252f457-35b5-4f79-9561-ecba9662200c"
-					(reference "R47")
+					(reference "R58")
 					(unit 1)
 				)
 				(path "/8c0b3d8b-46d3-4173-ab1e-a61765f77d61/ca9d4364-8864-42d1-89eb-99280f8ed67d"
-					(reference "R32")
+					(reference "R40")
 					(unit 1)
 				)
 				(path "/8c0b3d8b-46d3-4173-ab1e-a61765f77d61/f55e411b-ec4b-43e8-a550-3df1b34591c7"
-					(reference "R35")
+					(reference "R43")
 					(unit 1)
 				)
 				(path "/8c0b3d8b-46d3-4173-ab1e-a61765f77d61/f647f155-e741-47c8-b191-8b4f6021bf8f"
-					(reference "R50")
+					(reference "R61")
 					(unit 1)
 				)
@@
 		(dnp no)
 		(fields_autoplaced yes)
-		(property "Reference" "#PWR062"
+		(property "Reference" "#PWR092"
 			(at 151.13 90.17 0)
 			(effects
@@
 			(project "echo"
 				(path "/8c0b3d8b-46d3-4173-ab1e-a61765f77d61/4252f457-35b5-4f79-9561-ecba9662200c"
-					(reference "#PWR085")
+					(reference "#PWR0119")
 					(unit 1)
 				)
 				(path "/8c0b3d8b-46d3-4173-ab1e-a61765f77d61/ca9d4364-8864-42d1-89eb-99280f8ed67d"
-					(reference "#PWR062")
+					(reference "#PWR092")
 					(unit 1)
 				)
 				(path "/8c0b3d8b-46d3-4173-ab1e-a61765f77d61/f55e411b-ec4b-43e8-a550-3df1b34591c7"
-					(reference "#PWR064")
+					(reference "#PWR094")
 					(unit 1)
 				)
 				(path "/8c0b3d8b-46d3-4173-ab1e-a61765f77d61/f647f155-e741-47c8-b191-8b4f6021bf8f"
-					(reference "#PWR087")
-					(unit 1)
-				)
+					(reference "#PWR0121")
+					(unit 1)
+				)

Commit message: HW Revision 1.05
Parts:
- Q3: footprint FRANK:SOT-23 -> Package_TO_SOT_SMD:SOT-23
Changed lines of the file:
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@@
 			)
 		)
-		(property "Footprint" "FRANK:SOT-23"
+		(property "Footprint" "Package_TO_SOT_SMD:SOT-23"
 			(at 149.225 109.22 0)
 			(effects

Commit message: HW 1.06 WIP
Parts:
- Q3: footprint Package_TO_SOT_SMD:SOT-23 -> FRANK:SOT-23
- renumbered R39 to R46, R40 to R47, R41 to R48
Changed lines of the file:
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@@
 		(on_board yes)
 		(dnp no)
-		(property "Reference" "R41"
+		(property "Reference" "R48"
 			(at 161.29 93.98 0)
 			(effects
@@
 			(project "echo"
 				(path "/8c0b3d8b-46d3-4173-ab1e-a61765f77d61/4252f457-35b5-4f79-9561-ecba9662200c"
-					(reference "R59")
+					(reference "R66")
 					(unit 1)
 				)
 				(path "/8c0b3d8b-46d3-4173-ab1e-a61765f77d61/ca9d4364-8864-42d1-89eb-99280f8ed67d"
-					(reference "R41")
+					(reference "R48")
 					(unit 1)
 				)
 				(path "/8c0b3d8b-46d3-4173-ab1e-a61765f77d61/f55e411b-ec4b-43e8-a550-3df1b34591c7"
-					(reference "R44")
+					(reference "R51")
 					(unit 1)
 				)
 				(path "/8c0b3d8b-46d3-4173-ab1e-a61765f77d61/f647f155-e741-47c8-b191-8b4f6021bf8f"
-					(reference "R62")
+					(reference "R69")
 					(unit 1)
 				)
@@
 		(on_board yes)
 		(dnp no)
-		(property "Reference" "#PWR093"
+		(property "Reference" "#PWR0114"
 			(at 160.02 95.25 0)
 			(effects
@@
 			(project "echo"
 				(path "/8c0b3d8b-46d3-4173-ab1e-a61765f77d61/4252f457-35b5-4f79-9561-ecba9662200c"
-					(reference "#PWR0120")
+					(reference "#PWR0141")
 					(unit 1)
 				)
 				(path "/8c0b3d8b-46d3-4173-ab1e-a61765f77d61/ca9d4364-8864-42d1-89eb-99280f8ed67d"
-					(reference "#PWR093")
+					(reference "#PWR0114")
 					(unit 1)
 				)
 				(path "/8c0b3d8b-46d3-4173-ab1e-a61765f77d61/f55e411b-ec4b-43e8-a550-3df1b34591c7"
-					(reference "#PWR095")
+					(reference "#PWR0116")
 					(unit 1)
 				)
 				(path "/8c0b3d8b-46d3-4173-ab1e-a61765f77d61/f647f155-e741-47c8-b191-8b4f6021bf8f"
-					(reference "#PWR0122")
+					(reference "#PWR0143")
 					(unit 1)
 				)
@@
 		(on_board yes)
 		(dnp no)
-		(property "Reference" "R39"
+		(property "Reference" "R46"
 			(at 139.446 93.98 0)
 			(effects
@@
 			(project "echo"
 				(path "/8c0b3d8b-46d3-4173-ab1e-a61765f77d61/4252f457-35b5-4f79-9561-ecba9662200c"
-					(reference "R57")
+					(reference "R64")
 					(unit 1)
 				)
 				(path "/8c0b3d8b-46d3-4173-ab1e-a61765f77d61/ca9d4364-8864-42d1-89eb-99280f8ed67d"
-					(reference "R39")
+					(reference "R46")
 					(unit 1)
 				)
 				(path "/8c0b3d8b-46d3-4173-ab1e-a61765f77d61/f55e411b-ec4b-43e8-a550-3df1b34591c7"
-					(reference "R42")
+					(reference "R49")
 					(unit 1)
 				)
 				(path "/8c0b3d8b-46d3-4173-ab1e-a61765f77d61/f647f155-e741-47c8-b191-8b4f6021bf8f"
-					(reference "R60")
+					(reference "R67")
 					(unit 1)
 				)
@@
 			)
 		)
-		(property "Footprint" "Package_TO_SOT_SMD:SOT-23"
+		(property "Footprint" "FRANK:SOT-23"
 			(at 149.225 109.22 0)
 			(effects
@@
 		(on_board yes)
 		(dnp no)
-		(property "Reference" "R40"
+		(property "Reference" "R47"
 			(at 152.4 93.98 0)
 			(effects
@@
 			(project "echo"
 				(path "/8c0b3d8b-46d3-4173-ab1e-a61765f77d61/4252f457-35b5-4f79-9561-ecba9662200c"
-					(reference "R58")
+					(reference "R65")
 					(unit 1)
 				)
 				(path "/8c0b3d8b-46d3-4173-ab1e-a61765f77d61/ca9d4364-8864-42d1-89eb-99280f8ed67d"
-					(reference "R40")
+					(reference "R47")
 					(unit 1)
 				)
 				(path "/8c0b3d8b-46d3-4173-ab1e-a61765f77d61/f55e411b-ec4b-43e8-a550-3df1b34591c7"
-					(reference "R43")
+					(reference "R50")
 					(unit 1)
 				)
 				(path "/8c0b3d8b-46d3-4173-ab1e-a61765f77d61/f647f155-e741-47c8-b191-8b4f6021bf8f"
-					(reference "R61")
+					(reference "R68")
 					(unit 1)
 				)
@@
 		(dnp no)
 		(fields_autoplaced yes)
-		(property "Reference" "#PWR092"
+		(property "Reference" "#PWR0113"
 			(at 151.13 90.17 0)
 			(effects
@@
 			(project "echo"
 				(path "/8c0b3d8b-46d3-4173-ab1e-a61765f77d61/4252f457-35b5-4f79-9561-ecba9662200c"
-					(reference "#PWR0119")
+					(reference "#PWR0140")
 					(unit 1)
 				)
 				(path "/8c0b3d8b-46d3-4173-ab1e-a61765f77d61/ca9d4364-8864-42d1-89eb-99280f8ed67d"
-					(reference "#PWR092")
+					(reference "#PWR0113")
 					(unit 1)
 				)
 				(path "/8c0b3d8b-46d3-4173-ab1e-a61765f77d61/f55e411b-ec4b-43e8-a550-3df1b34591c7"
-					(reference "#PWR094")
+					(reference "#PWR0115")
 					(unit 1)
 				)
 				(path "/8c0b3d8b-46d3-4173-ab1e-a61765f77d61/f647f155-e741-47c8-b191-8b4f6021bf8f"
-					(reference "#PWR0121")
-					(unit 1)
-				)
+					(reference "#PWR0142")
+					(unit 1)
+				)
