File: rp2040.kicad_sch (KiCad schematic)
At the start: 25 parts, among them U7 W25Q128JVSIQ, U8 RP2040, Y1 12 MHz

Commit message: Minor fixes
Parts:
- C18: renamed from C19; LCSC C1711 -> (none)
- C19: renamed from C20; LCSC C1711 -> (none)
- C20: renamed from C21; LCSC C1711 -> (none)
- C21: renamed from C22; LCSC C1711 -> (none)
- C22: renamed from C23; LCSC C1711 -> (none)
- C23: renamed from C24; LCSC C1711 -> (none)
- C24: renamed from C25; LCSC C1711 -> (none)
- C25: renamed from C26; LCSC C1711 -> (none)
- C26: renamed from C27; LCSC C1711 -> (none)
- C27: renamed from C28; LCSC C1711 -> (none)
- C28: renamed from C29; LCSC C24123 -> (none)
- C29: renamed from C30; LCSC C24123 -> (none)
- C30: renamed from C31; LCSC C1711 -> (none)
- C31: renamed from C32; LCSC C63339 -> (none)
- C32: renamed from C33; LCSC C63339 -> (none)
- LD4: value Blue -> Blue (GPIO25)
- R33: renamed from R34; LCSC C17513 -> (none)
- R35: renamed from R36; LCSC C17513 -> (none)
- R36: renamed from R37; LCSC C17513 -> (none)
- S4: renamed from S2; value Boot -> RP Boot
- U6: renamed from U7; LCSC C97521 -> (none)
- U7: renamed from U8; LCSC C2040 -> (none)
- Y1: LCSC C9900023240 -> (none)
- renumbered R33 to R32, R35 to R34

Commit message: HW Rev 1.03
Parts:
- renumbered C18 to C17, C19 to C18, C20 to C19, C21 to C20, C22 to C21, C23 to C22, C24 to C23, C25 to C24, C26 to C25, C27 to C26, C28 to C27, C29 to C28, C30 to C29, C31 to C30, C32 to C31
Changed lines of the file:
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@@
 	(title_block
 		(title "${NAME}")
-		(date "2025-06-23")
+		(date "2025-07-20")
 		(rev "${VERSION}")
 		(company "Mikhail Matveev")
@@
 		(on_board yes)
 		(dnp no)
-		(property "Reference" "C19"
+		(property "Reference" "C18"
 			(at 49.911 42.0116 0)
 			(effects
@@
 			(project "frank2"
 				(path "/8c0b3d8b-46d3-4173-ab1e-a61765f77d61/e0efa020-7652-4c53-946d-b42f9a8f5279"
-					(reference "C19")
+					(reference "C18")
 					(unit 1)
 				)
@@
 		(on_board yes)
 		(dnp no)
-		(property "Reference" "C23"
+		(property "Reference" "C22"
 			(at 138.811 42.0116 0)
 			(effects
@@
 			(project "frank2"
 				(path "/8c0b3d8b-46d3-4173-ab1e-a61765f77d61/e0efa020-7652-4c53-946d-b42f9a8f5279"
-					(reference "C23")
+					(reference "C22")
 					(unit 1)
 				)
@@
 		(on_board yes)
 		(dnp no)
-		(property "Reference" "C18"
+		(property "Reference" "C17"
 			(at 38.481 42.0116 0)
 			(effects
@@
 			(project "frank2"
 				(path "/8c0b3d8b-46d3-4173-ab1e-a61765f77d61/e0efa020-7652-4c53-946d-b42f9a8f5279"
-					(reference "C18")
+					(reference "C17")
 					(unit 1)
 				)
@@
 		(on_board yes)
 		(dnp no)
-		(property "Reference" "C20"
+		(property "Reference" "C19"
 			(at 104.521 42.0116 0)
 			(effects
@@
 			(project "frank2"
 				(path "/8c0b3d8b-46d3-4173-ab1e-a61765f77d61/e0efa020-7652-4c53-946d-b42f9a8f5279"
-					(reference "C20")
+					(reference "C19")
 					(unit 1)
 				)
@@
 		(on_board yes)
 		(dnp no)
-		(property "Reference" "C21"
+		(property "Reference" "C20"
 			(at 115.951 42.0116 0)
 			(effects
@@
 			(project "frank2"
 				(path "/8c0b3d8b-46d3-4173-ab1e-a61765f77d61/e0efa020-7652-4c53-946d-b42f9a8f5279"
-					(reference "C21")
+					(reference "C20")
 					(unit 1)
 				)
@@
 		(on_board yes)
 		(dnp no)
-		(property "Reference" "C29"
+		(property "Reference" "C28"
 			(at 104.521 57.2516 0)
 			(effects
@@
 			(project "frank2"
 				(path "/8c0b3d8b-46d3-4173-ab1e-a61765f77d61/e0efa020-7652-4c53-946d-b42f9a8f5279"
-					(reference "C29")
+					(reference "C28")
 					(unit 1)
 				)
@@
 		(on_board yes)
 		(dnp no)
-		(property "Reference" "C30"
+		(property "Reference" "C29"
 			(at 257.7084 79.121 0)
 			(effects
@@
 			(project "frank2"
 				(path "/8c0b3d8b-46d3-4173-ab1e-a61765f77d61/e0efa020-7652-4c53-946d-b42f9a8f5279"
-					(reference "C30")
+					(reference "C29")
 					(unit 1)
 				)
@@
 		(on_board yes)
 		(dnp no)
-		(property "Reference" "C32"
+		(property "Reference" "C31"
 			(at 208.3816 134.239 0)
 			(effects
@@
 			(project "frank2"
 				(path "/8c0b3d8b-46d3-4173-ab1e-a61765f77d61/e0efa020-7652-4c53-946d-b42f9a8f5279"
-					(reference "C32")
+					(reference "C31")
 					(unit 1)
 				)
@@
 		(on_board yes)
 		(dnp no)
-		(property "Reference" "C27"
+		(property "Reference" "C26"
 			(at 184.531 42.0116 0)
 			(effects
@@
 			(project "core"
 				(path "/8c0b3d8b-46d3-4173-ab1e-a61765f77d61/e0efa020-7652-4c53-946d-b42f9a8f5279"
-					(reference "C27")
+					(reference "C26")
 					(unit 1)
 				)
@@
 		(on_board yes)
 		(dnp no)
-		(property "Reference" "C31"
+		(property "Reference" "C30"
 			(at 208.3816 124.079 0)
 			(effects
@@
 			(project "frank2"
 				(path "/8c0b3d8b-46d3-4173-ab1e-a61765f77d61/e0efa020-7652-4c53-946d-b42f9a8f5279"
-					(reference "C31")
+					(reference "C30")
 					(unit 1)
 				)
@@
 		(on_board yes)
 		(dnp no)
-		(property "Reference" "C28"
+		(property "Reference" "C27"
 			(at 49.911 57.2516 0)
 			(effects
@@
 			(project "frank2"
 				(path "/8c0b3d8b-46d3-4173-ab1e-a61765f77d61/e0efa020-7652-4c53-946d-b42f9a8f5279"
-					(reference "C28")
+					(reference "C27")
 					(unit 1)
 				)
@@
 		(on_board yes)
 		(dnp no)
-		(property "Reference" "C22"
+		(property "Reference" "C21"
 			(at 127.381 42.0116 0)
 			(effects
@@
 			(project "frank2"
 				(path "/8c0b3d8b-46d3-4173-ab1e-a61765f77d61/e0efa020-7652-4c53-946d-b42f9a8f5279"
-					(reference "C22")
+					(reference "C21")
 					(unit 1)
 				)
@@
 		(on_board yes)
 		(dnp no)
-		(property "Reference" "C26"
+		(property "Reference" "C25"
 			(at 173.101 42.0116 0)
 			(effects
@@
 			(project "frank2"
 				(path "/8c0b3d8b-46d3-4173-ab1e-a61765f77d61/e0efa020-7652-4c53-946d-b42f9a8f5279"
-					(reference "C26")
+					(reference "C25")
 					(unit 1)
 				)
@@
 		(on_board yes)
 		(dnp no)
-		(property "Reference" "C24"
+		(property "Reference" "C23"
 			(at 150.241 42.0116 0)
 			(effects
@@
 			(project "frank2"
 				(path "/8c0b3d8b-46d3-4173-ab1e-a61765f77d61/e0efa020-7652-4c53-946d-b42f9a8f5279"
-					(reference "C24")
+					(reference "C23")
 					(unit 1)
 				)
@@
 		(on_board yes)
 		(dnp no)
-		(property "Reference" "C25"
+		(property "Reference" "C24"
 			(at 161.671 42.0116 0)
 			(effects
@@
 			(project "frank2"
 				(path "/8c0b3d8b-46d3-4173-ab1e-a61765f77d61/e0efa020-7652-4c53-946d-b42f9a8f5279"
-					(reference "C25")
+					(reference "C24")
 					(unit 1)
 				)

Commit message: WIP
Parts:
- S5: renamed from S4; footprint FRANK:TACT-SIDE-4623 -> FRANK:Button (SMD, 3x3mm, 1-1)
- renumbered C17 to C18, C18 to C19, C19 to C20, C20 to C21, C21 to C22, C22 to C23, C23 to C24, C24 to C25, C25 to C26, C26 to C27, C27 to C28, C28 to C29, C29 to C30, C30 to C31, C31 to C32, R32 to R41, R33 to R42, R34 to R43, R35 to R44, R36 to R45, U6 to U7, U7 to U8

Commit message: Rev 1.05 WIP
Parts:
- C43: renamed from C18; footprint FRANK:Capacitor (0805) -> FRANK:Capacitor (0603)
- C44: renamed from C19; footprint FRANK:Capacitor (0805) -> FRANK:Capacitor (0603)
- C45: renamed from C20; footprint FRANK:Capacitor (0805) -> FRANK:Capacitor (0603)
- C46: renamed from C21; footprint FRANK:Capacitor (0805) -> FRANK:Capacitor (0603)
- C47: renamed from C22; footprint FRANK:Capacitor (0805) -> FRANK:Capacitor (0603)
- C48: renamed from C23; footprint FRANK:Capacitor (0805) -> FRANK:Capacitor (0603)
- C49: renamed from C24; footprint FRANK:Capacitor (0805) -> FRANK:Capacitor (0603)
- C50: renamed from C25; footprint FRANK:Capacitor (0805) -> FRANK:Capacitor (0603)
- C51: renamed from C26; footprint FRANK:Capacitor (0805) -> FRANK:Capacitor (0603)
- C52: renamed from C27; footprint FRANK:Capacitor (0805) -> FRANK:Capacitor (0603)
- C53: renamed from C28; footprint FRANK:Capacitor (0805) -> FRANK:Capacitor (0603)
- C54: renamed from C29; footprint FRANK:Capacitor (0805) -> FRANK:Capacitor (0603)
- C55: renamed from C30; footprint FRANK:Capacitor (0805) -> FRANK:Capacitor (0603)
- C56: renamed from C31; footprint FRANK:Capacitor (0805) -> FRANK:Capacitor (0603)
- C57: renamed from C32; footprint FRANK:Capacitor (0805) -> FRANK:Capacitor (0603)
- R52: renamed from R41; footprint FRANK:Resistor (0805) -> FRANK:Resistor (0603)
- R53: renamed from R42; footprint FRANK:Resistor (0805) -> FRANK:Resistor (0603)
- R54: renamed from R43; footprint FRANK:Resistor (0805) -> FRANK:Resistor (0603)
- R55: renamed from R44; footprint FRANK:Resistor (0805) -> FRANK:Resistor (0603)
- R56: renamed from R45; footprint FRANK:Resistor (0805) -> FRANK:Resistor (0603)
- renumbered U7 to U10, U8 to U11

Commit message: HW Revision 1.05
Parts:
- LD4: footprint FRANK:LED (0805) -> FRANK:LED (0603)
Changed lines of the file:
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@@
 			)
 		)
-		(property "Footprint" "FRANK:LED (0805)"
+		(property "Footprint" "FRANK:LED (0603)"
 			(at 252.73 130.81 0)
 			(effects

Commit message: HW 1.06 WIP
Parts:
- renumbered C43 to C57, C44 to C58, C53 to C59, C45 to C60, C54 to C61, C46 to C62, C47 to C63, C48 to C64, C49 to C65, C50 to C66, C51 to C67, C52 to C68, C56 to C69, C57 to C70, C55 to C71, LD4 to LD5, R52 to R59, R54 to R60, R55 to R61, R53 to R62, R56 to R63, S5 to S4, U11 to U12, U10 to U13, Y1 to Y2
