File: usb_multiplexer.kicad_sch (KiCad schematic)
At the start: 5 parts, among them J7 PJ-320D

Commit message: Minor fixes
Parts:
- removed C13: 10u, FRANK:Capacitor (0805), symbol Device:C
- removed C14: 33n, FRANK:Capacitor (0805), symbol Device:C
- removed J7: PJ-320D, FRANK:Jack (3.5mm, PJ-320D), symbol FRANK:AudioJack_3.5mm
- removed R28: 100R, FRANK:Resistor (0805), symbol Device:R
- removed R29: 150R, FRANK:Resistor (0805), symbol Device:R
- added C34: 100n, FRANK:Capacitor (0805), symbol Device:C
- added R43: 10K, FRANK:Resistor (0805), symbol Device:R
- added U8: TS3USB221RSER, FRANK:UQFN-10, symbol TS3USB221R:TS3USB221RSER
Connections:
- net GND: now also C34.1, U8.5 (GND), U8.6 (~{OE})
- new net +3V3: C34.2, R43.1, U8.10 (VCC)
- new net D+: U8.8 (D+)
- new net D-: U8.7 (D-)
- new net D1+: U8.1 (1D+)
- new net D1-: U8.2 (1D-)
- new net D2+: U8.3 (2D+)
- new net D2-: U8.4 (2D-)
- new net S: R43.2, U8.9 (S)

Commit message: HW Rev 1.03
Parts:
- renumbered C34 to C33
Changed lines of the file:
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@@
 	(title_block
 		(title "${NAME}")
-		(date "2025-06-23")
+		(date "2025-07-20")
 		(rev "${VERSION}")
 		(company "Mikhail Matveev")
@@
 		(on_board yes)
 		(dnp no)
-		(property "Reference" "C34"
+		(property "Reference" "C33"
 			(at 143.6116 79.629 0)
 			(effects
@@
 			(project "echo"
 				(path "/8c0b3d8b-46d3-4173-ab1e-a61765f77d61/21f6980c-fc10-4480-8dc1-86a15fb6d0bb"
-					(reference "C36")
+					(reference "C35")
 					(unit 1)
 				)
 				(path "/8c0b3d8b-46d3-4173-ab1e-a61765f77d61/a27ed13f-fa40-49de-a786-9b8f7712cf33"
-					(reference "C34")
-					(unit 1)
-				)
+					(reference "C33")
+					(unit 1)
+				)

Commit message: WIP
Parts:
- renumbered C33 to C37, R43 to R56, U8 to U10
Other:
- moved on the sheet: C37, R56, U10

Commit message: Rev 1.05 WIP
Parts:
- C62: renamed from C37; footprint FRANK:Capacitor (0805) -> FRANK:Capacitor (0603)
- R67: renamed from R56; footprint FRANK:Resistor (0805) -> FRANK:Resistor (0603)
- renumbered U10 to U13
Changed lines of the file:
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@@
 		(dnp no)
 		(fields_autoplaced yes)
-		(property "Reference" "U10"
+		(property "Reference" "U13"
 			(at 159.6233 83.82 0)
 			(effects
@@
 			(project "echo"
 				(path "/8c0b3d8b-46d3-4173-ab1e-a61765f77d61/21f6980c-fc10-4480-8dc1-86a15fb6d0bb"
-					(reference "U10")
+					(reference "U13")
 					(unit 1)
 				)
@@
 		(dnp no)
 		(fields_autoplaced yes)
-		(property "Reference" "#PWR0103"
+		(property "Reference" "#PWR0137"
 			(at 137.16 99.06 0)
 			(effects
@@
 			(project "echo"
 				(path "/8c0b3d8b-46d3-4173-ab1e-a61765f77d61/21f6980c-fc10-4480-8dc1-86a15fb6d0bb"
-					(reference "#PWR0103")
+					(reference "#PWR0137")
 					(unit 1)
 				)
@@
 		(on_board yes)
 		(dnp no)
-		(property "Reference" "C37"
+		(property "Reference" "C62"
 			(at 143.6116 77.089 0)
 			(effects
@@
 			)
 		)
-		(property "Footprint" "FRANK:Capacitor (0805)"
+		(property "Footprint" "FRANK:Capacitor (0603)"
 			(at 148.59 79.0448 0)
 			(effects
@@
 			(project "echo"
 				(path "/8c0b3d8b-46d3-4173-ab1e-a61765f77d61/21f6980c-fc10-4480-8dc1-86a15fb6d0bb"
-					(reference "C37")
+					(reference "C62")
 					(unit 1)
 				)
@@
 		(dnp no)
 		(fields_autoplaced yes)
-		(property "Reference" "#PWR0100"
+		(property "Reference" "#PWR0134"
 			(at 157.48 77.47 0)
 			(effects
@@
 			(project "echo"
 				(path "/8c0b3d8b-46d3-4173-ab1e-a61765f77d61/21f6980c-fc10-4480-8dc1-86a15fb6d0bb"
-					(reference "#PWR0100")
+					(reference "#PWR0134")
 					(unit 1)
 				)
@@
 		(on_board yes)
 		(dnp no)
-		(property "Reference" "R56"
+		(property "Reference" "R67"
 			(at 125.476 92.202 90)
 			(effects
@@
 			)
 		)
-		(property "Footprint" "FRANK:Resistor (0805)"
+		(property "Footprint" "FRANK:Resistor (0603)"
 			(at 121.412 93.98 90)
 			(effects
@@
 			(project "echo"
 				(path "/8c0b3d8b-46d3-4173-ab1e-a61765f77d61/21f6980c-fc10-4480-8dc1-86a15fb6d0bb"
-					(reference "R56")
+					(reference "R67")
 					(unit 1)
 				)
@@
 		(dnp no)
 		(fields_autoplaced yes)
-		(property "Reference" "#PWR0102"
+		(property "Reference" "#PWR0136"
 			(at 123.19 92.71 0)
 			(effects
@@
 			(project "echo"
 				(path "/8c0b3d8b-46d3-4173-ab1e-a61765f77d61/21f6980c-fc10-4480-8dc1-86a15fb6d0bb"
-					(reference "#PWR0102")
+					(reference "#PWR0136")
 					(unit 1)
 				)
@@
 		(dnp no)
 		(fields_autoplaced yes)
-		(property "Reference" "#PWR0101"
+		(property "Reference" "#PWR0135"
 			(at 134.62 80.01 0)
 			(effects
@@
 			(project "echo"
 				(path "/8c0b3d8b-46d3-4173-ab1e-a61765f77d61/21f6980c-fc10-4480-8dc1-86a15fb6d0bb"
-					(reference "#PWR0101")
+					(reference "#PWR0135")
 					(unit 1)
 				)
@@
 		(dnp no)
 		(fields_autoplaced yes)
-		(property "Reference" "#PWR0104"
+		(property "Reference" "#PWR0138"
 			(at 157.48 125.73 0)
 			(effects
@@
 			(project "echo"
 				(path "/8c0b3d8b-46d3-4173-ab1e-a61765f77d61/21f6980c-fc10-4480-8dc1-86a15fb6d0bb"
-					(reference "#PWR0104")
-					(unit 1)
-				)
+					(reference "#PWR0138")
+					(unit 1)
+				)

Commit message: HW 1.06 WIP
Parts:
- renumbered C62 to C76, R67 to R74, U13 to U15
Changed lines of the file:
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@@
 		(dnp no)
 		(fields_autoplaced yes)
-		(property "Reference" "U13"
+		(property "Reference" "U15"
 			(at 159.6233 83.82 0)
 			(effects
@@
 			(project "echo"
 				(path "/8c0b3d8b-46d3-4173-ab1e-a61765f77d61/21f6980c-fc10-4480-8dc1-86a15fb6d0bb"
-					(reference "U13")
+					(reference "U15")
 					(unit 1)
 				)
@@
 		(dnp no)
 		(fields_autoplaced yes)
-		(property "Reference" "#PWR0137"
+		(property "Reference" "#PWR0157"
 			(at 137.16 99.06 0)
 			(effects
@@
 			(project "echo"
 				(path "/8c0b3d8b-46d3-4173-ab1e-a61765f77d61/21f6980c-fc10-4480-8dc1-86a15fb6d0bb"
-					(reference "#PWR0137")
+					(reference "#PWR0157")
 					(unit 1)
 				)
@@
 		(on_board yes)
 		(dnp no)
-		(property "Reference" "C62"
+		(property "Reference" "C76"
 			(at 143.6116 77.089 0)
 			(effects
@@
 			(project "echo"
 				(path "/8c0b3d8b-46d3-4173-ab1e-a61765f77d61/21f6980c-fc10-4480-8dc1-86a15fb6d0bb"
-					(reference "C62")
+					(reference "C76")
 					(unit 1)
 				)
@@
 		(dnp no)
 		(fields_autoplaced yes)
-		(property "Reference" "#PWR0134"
+		(property "Reference" "#PWR0158"
 			(at 157.48 77.47 0)
 			(effects
@@
 			(project "echo"
 				(path "/8c0b3d8b-46d3-4173-ab1e-a61765f77d61/21f6980c-fc10-4480-8dc1-86a15fb6d0bb"
-					(reference "#PWR0134")
+					(reference "#PWR0158")
 					(unit 1)
 				)
@@
 		(on_board yes)
 		(dnp no)
-		(property "Reference" "R67"
+		(property "Reference" "R74"
 			(at 125.476 92.202 90)
 			(effects
@@
 			(project "echo"
 				(path "/8c0b3d8b-46d3-4173-ab1e-a61765f77d61/21f6980c-fc10-4480-8dc1-86a15fb6d0bb"
-					(reference "R67")
+					(reference "R74")
 					(unit 1)
 				)
@@
 		(dnp no)
 		(fields_autoplaced yes)
-		(property "Reference" "#PWR0136"
+		(property "Reference" "#PWR0155"
 			(at 123.19 92.71 0)
 			(effects
@@
 			(project "echo"
 				(path "/8c0b3d8b-46d3-4173-ab1e-a61765f77d61/21f6980c-fc10-4480-8dc1-86a15fb6d0bb"
-					(reference "#PWR0136")
+					(reference "#PWR0155")
 					(unit 1)
 				)
@@
 		(dnp no)
 		(fields_autoplaced yes)
-		(property "Reference" "#PWR0135"
+		(property "Reference" "#PWR0156"
 			(at 134.62 80.01 0)
 			(effects
@@
 			(project "echo"
 				(path "/8c0b3d8b-46d3-4173-ab1e-a61765f77d61/21f6980c-fc10-4480-8dc1-86a15fb6d0bb"
-					(reference "#PWR0135")
+					(reference "#PWR0156")
 					(unit 1)
 				)
@@
 		(dnp no)
 		(fields_autoplaced yes)
-		(property "Reference" "#PWR0138"
+		(property "Reference" "#PWR0159"
 			(at 157.48 125.73 0)
 			(effects
@@
 			(project "echo"
 				(path "/8c0b3d8b-46d3-4173-ab1e-a61765f77d61/21f6980c-fc10-4480-8dc1-86a15fb6d0bb"
-					(reference "#PWR0138")
-					(unit 1)
-				)
+					(reference "#PWR0159")
+					(unit 1)
+				)
