File: tape.kicad_sch (KiCad schematic)
At the start: 7 parts, among them J9 PJ-320D

Commit message: Minor fixes
Parts:
- J8: renamed from J9; LCSC C95562 -> (none)
- renumbered R31 to R30, R32 to R31
Changed lines of the file:
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@@
 	(title_block
 		(title "${NAME}")
-		(date "2025-05-24")
+		(date "2025-06-23")
 		(rev "${VERSION}")
 		(company "Mikhail Matveev")
@@
 		(dnp no)
 		(fields_autoplaced yes)
-		(property "Reference" "#PWR058"
+		(property "Reference" "#PWR057"
 			(at 172.72 95.25 0)
 			(effects
@@
 			(project "echo"
 				(path "/8c0b3d8b-46d3-4173-ab1e-a61765f77d61/e606b562-b239-4a02-9f90-df2cbefa5295"
-					(reference "#PWR058")
+					(reference "#PWR057")
 					(unit 1)
 				)
@@
 		(on_board yes)
 		(dnp no)
-		(property "Reference" "J9"
+		(property "Reference" "J8"
 			(at 116.0781 92.5103 0)
 			(effects
@@
 			)
 		)
-		(property "LCSC" "C95562"
+		(property "LCSC" ""
 			(at 123.19 96.52 0)
 			(effects
@@
 			(project "echo"
 				(path "/8c0b3d8b-46d3-4173-ab1e-a61765f77d61/e606b562-b239-4a02-9f90-df2cbefa5295"
-					(reference "J9")
+					(reference "J8")
 					(unit 1)
 				)
@@
 		(on_board yes)
 		(dnp no)
-		(property "Reference" "R31"
+		(property "Reference" "R30"
 			(at 164.084 90.17 0)
 			(effects
@@
 			(project "echo"
 				(path "/8c0b3d8b-46d3-4173-ab1e-a61765f77d61/e606b562-b239-4a02-9f90-df2cbefa5295"
-					(reference "R31")
+					(reference "R30")
 					(unit 1)
 				)
@@
 		(on_board yes)
 		(dnp no)
-		(property "Reference" "R32"
+		(property "Reference" "R31"
 			(at 166.37 100.584 0)
 			(effects
@@
 			(project "echo"
 				(path "/8c0b3d8b-46d3-4173-ab1e-a61765f77d61/e606b562-b239-4a02-9f90-df2cbefa5295"
-					(reference "R32")
+					(reference "R31")
 					(unit 1)
 				)
@@
 		(dnp no)
 		(fields_autoplaced yes)
-		(property "Reference" "#PWR057"
+		(property "Reference" "#PWR056"
 			(at 182.88 90.17 0)
 			(effects
@@
 			(project "echo"
 				(path "/8c0b3d8b-46d3-4173-ab1e-a61765f77d61/e606b562-b239-4a02-9f90-df2cbefa5295"
-					(reference "#PWR057")
+					(reference "#PWR056")
 					(unit 1)
 				)

Commit message: HW Rev 1.03
Parts:
- renumbered C15 to C14, C16 to C15, C17 to C16
Changed lines of the file:
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@@
 	(title_block
 		(title "${NAME}")
-		(date "2025-06-23")
+		(date "2025-07-20")
 		(rev "${VERSION}")
 		(company "Mikhail Matveev")
@@
 		(on_board yes)
 		(dnp no)
-		(property "Reference" "C17"
+		(property "Reference" "C16"
 			(at 152.2984 103.251 0)
 			(effects
@@
 			(project "echo"
 				(path "/8c0b3d8b-46d3-4173-ab1e-a61765f77d61/e606b562-b239-4a02-9f90-df2cbefa5295"
-					(reference "C17")
+					(reference "C16")
 					(unit 1)
 				)
@@
 		(on_board yes)
 		(dnp no)
-		(property "Reference" "C16"
+		(property "Reference" "C15"
 			(at 151.9174 87.376 0)
 			(effects
@@
 			(project "echo"
 				(path "/8c0b3d8b-46d3-4173-ab1e-a61765f77d61/e606b562-b239-4a02-9f90-df2cbefa5295"
-					(reference "C16")
+					(reference "C15")
 					(unit 1)
 				)
@@
 		(on_board yes)
 		(dnp no)
-		(property "Reference" "C15"
+		(property "Reference" "C14"
 			(at 151.9174 74.676 0)
 			(effects
@@
 			(project "echo"
 				(path "/8c0b3d8b-46d3-4173-ab1e-a61765f77d61/e606b562-b239-4a02-9f90-df2cbefa5295"
-					(reference "C15")
+					(reference "C14")
 					(unit 1)
 				)

Commit message: WIP
Parts:
- renumbered C14 to C15, C15 to C16, C16 to C17, J8 to J9, R30 to R39, R31 to R40
Changed lines of the file:
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@@
 	(title_block
 		(title "${NAME}")
-		(date "2025-07-20")
+		(date "2025-08-08")
 		(rev "${VERSION}")
 		(company "Mikhail Matveev")
@@
 		(on_board yes)
 		(dnp no)
-		(property "Reference" "C16"
+		(property "Reference" "C17"
 			(at 152.2984 103.251 0)
 			(effects
@@
 			(project "echo"
 				(path "/8c0b3d8b-46d3-4173-ab1e-a61765f77d61/e606b562-b239-4a02-9f90-df2cbefa5295"
-					(reference "C16")
+					(reference "C17")
 					(unit 1)
 				)
@@
 		(dnp no)
 		(fields_autoplaced yes)
-		(property "Reference" "#PWR057"
+		(property "Reference" "#PWR069"
 			(at 172.72 95.25 0)
 			(effects
@@
 			(project "echo"
 				(path "/8c0b3d8b-46d3-4173-ab1e-a61765f77d61/e606b562-b239-4a02-9f90-df2cbefa5295"
-					(reference "#PWR057")
+					(reference "#PWR069")
 					(unit 1)
 				)
@@
 		(on_board yes)
 		(dnp no)
-		(property "Reference" "J8"
+		(property "Reference" "J9"
 			(at 116.0781 92.5103 0)
 			(effects
@@
 			(project "echo"
 				(path "/8c0b3d8b-46d3-4173-ab1e-a61765f77d61/e606b562-b239-4a02-9f90-df2cbefa5295"
-					(reference "J8")
+					(reference "J9")
 					(unit 1)
 				)
@@
 		(on_board yes)
 		(dnp no)
-		(property "Reference" "C15"
+		(property "Reference" "C16"
 			(at 151.9174 87.376 0)
 			(effects
@@
 			(project "echo"
 				(path "/8c0b3d8b-46d3-4173-ab1e-a61765f77d61/e606b562-b239-4a02-9f90-df2cbefa5295"
-					(reference "C15")
+					(reference "C16")
 					(unit 1)
 				)
@@
 		(on_board yes)
 		(dnp no)
-		(property "Reference" "C14"
+		(property "Reference" "C15"
 			(at 151.9174 74.676 0)
 			(effects
@@
 			(project "echo"
 				(path "/8c0b3d8b-46d3-4173-ab1e-a61765f77d61/e606b562-b239-4a02-9f90-df2cbefa5295"
-					(reference "C14")
+					(reference "C15")
 					(unit 1)
 				)
@@
 		(on_board yes)
 		(dnp no)
-		(property "Reference" "R30"
+		(property "Reference" "R39"
 			(at 164.084 90.17 0)
 			(effects
@@
 			(project "echo"
 				(path "/8c0b3d8b-46d3-4173-ab1e-a61765f77d61/e606b562-b239-4a02-9f90-df2cbefa5295"
-					(reference "R30")
+					(reference "R39")
 					(unit 1)
 				)
@@
 		(on_board yes)
 		(dnp no)
-		(property "Reference" "R31"
+		(property "Reference" "R40"
 			(at 166.37 100.584 0)
 			(effects
@@
 			(project "echo"
 				(path "/8c0b3d8b-46d3-4173-ab1e-a61765f77d61/e606b562-b239-4a02-9f90-df2cbefa5295"
-					(reference "R31")
+					(reference "R40")
 					(unit 1)
 				)
@@
 		(dnp no)
 		(fields_autoplaced yes)
-		(property "Reference" "#PWR056"
+		(property "Reference" "#PWR068"
 			(at 182.88 90.17 0)
 			(effects
@@
 			(project "echo"
 				(path "/8c0b3d8b-46d3-4173-ab1e-a61765f77d61/e606b562-b239-4a02-9f90-df2cbefa5295"
-					(reference "#PWR056")
+					(reference "#PWR068")
 					(unit 1)
 				)

Commit message: Rev 1.05 WIP
Parts:
- removed C15, C16, C17: 100n, FRANK:Capacitor (0805), symbol Device:C
- removed D1: Zener 3V3, FRANK:Diode (0805), symbol PCM_Nuova-Elettronica-Diodes:Zener
- removed J9: PJ-320D, FRANK:Jack (3.5mm, PJ-320D), symbol FRANK:AudioJack_3.5mm
- removed R39, R40: 10K, FRANK:Resistor (0805), symbol Device:R
- added AJ1: PJ-320D, FRANK:Jack (3.5mm, PJ-320D), symbol FRANK:AudioJack_3.5mm
- added C41, C42: 100n, FRANK:Capacitor (0603), symbol Device:C
- added D2: 1N4148, FRANK:Diode (SOD-323), symbol Device:D
- added Q5, Q6: BC850, FRANK:SOT-23, symbol Transistor_BJT:BC850
- added R47, R49, R50: 10K, FRANK:Resistor (0603), symbol Device:R
- added R48: 1K, FRANK:Resistor (0603), symbol Device:R
- added R51: 100R, FRANK:Resistor (0603), symbol Device:R
Connections:
- net GND: now also AJ1.S, C41.2, Q5.2 (E), Q6.2 (E), R51.2
- net LOAD_IN: now also Q5.3 (C), R48.2
- new net: D2.2 (A), Q6.3 (C), R47.2, R49.1
- new net: D2.1 (K), Q6.1 (B), R50.2
- new net: AJ1.T, C42.1, R51.1
- new net: C42.2, R50.1
- new net: Q5.1 (B), R49.2
- new net +3V3: C41.1, R47.1, R48.1
- no-connect marks 0 -> 1

Commit message: HW 1.06 WIP
Parts:
- renumbered C42 to C55, C41 to C56, Q6 to Q5, Q5 to Q6, R51 to R54, R50 to R55, R47 to R56, R49 to R57, R48 to R58
Changed lines of the file:
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@@
 		(dnp no)
 		(fields_autoplaced yes)
-		(property "Reference" "R47"
+		(property "Reference" "R56"
 			(at 160.02 85.0899 0)
 			(effects
@@
 			(project "echo"
 				(path "/8c0b3d8b-46d3-4173-ab1e-a61765f77d61/e606b562-b239-4a02-9f90-df2cbefa5295"
-					(reference "R47")
+					(reference "R56")
 					(unit 1)
 				)
@@
 		(dnp no)
 		(fields_autoplaced yes)
-		(property "Reference" "#PWR0102"
+		(property "Reference" "#PWR0121"
 			(at 157.48 127 0)
 			(effects
@@
 			(project "echo"
 				(path "/8c0b3d8b-46d3-4173-ab1e-a61765f77d61/e606b562-b239-4a02-9f90-df2cbefa5295"
-					(reference "#PWR0102")
+					(reference "#PWR0121")
 					(unit 1)
 				)
@@
 		(dnp no)
 		(fields_autoplaced yes)
-		(property "Reference" "#PWR0101"
+		(property "Reference" "#PWR0120"
 			(at 124.46 127 0)
 			(effects
@@
 			(project "echo"
 				(path "/8c0b3d8b-46d3-4173-ab1e-a61765f77d61/e606b562-b239-4a02-9f90-df2cbefa5295"
-					(reference "#PWR0101")
+					(reference "#PWR0120")
 					(unit 1)
 				)
@@
 		(dnp no)
 		(fields_autoplaced yes)
-		(property "Reference" "#PWR099"
+		(property "Reference" "#PWR0124"
 			(at 196.85 91.44 0)
 			(effects
@@
 			(project "echo"
 				(path "/8c0b3d8b-46d3-4173-ab1e-a61765f77d61/e606b562-b239-4a02-9f90-df2cbefa5295"
-					(reference "#PWR099")
+					(reference "#PWR0124")
 					(unit 1)
 				)
@@
 		(dnp no)
 		(fields_autoplaced yes)
-		(property "Reference" "#PWR0100"
+		(property "Reference" "#PWR0119"
 			(at 114.3 113.03 0)
 			(effects
@@
 			(project "echo"
 				(path "/8c0b3d8b-46d3-4173-ab1e-a61765f77d61/e606b562-b239-4a02-9f90-df2cbefa5295"
-					(reference "#PWR0100")
+					(reference "#PWR0119")
 					(unit 1)
 				)
@@
 		(on_board yes)
 		(dnp no)
-		(property "Reference" "C41"
+		(property "Reference" "C56"
 			(at 193.421 82.6516 0)
 			(effects
@@
 			(project "echo"
 				(path "/8c0b3d8b-46d3-4173-ab1e-a61765f77d61/e606b562-b239-4a02-9f90-df2cbefa5295"
-					(reference "C41")
+					(reference "C56")
 					(unit 1)
 				)
@@
 		(dnp no)
 		(fields_autoplaced yes)
-		(property "Reference" "#PWR0103"
+		(property "Reference" "#PWR0122"
 			(at 175.26 127 0)
 			(effects
@@
 			(project "echo"
 				(path "/8c0b3d8b-46d3-4173-ab1e-a61765f77d61/e606b562-b239-4a02-9f90-df2cbefa5295"
-					(reference "#PWR0103")
+					(reference "#PWR0122")
 					(unit 1)
 				)
@@
 		(dnp no)
 		(fields_autoplaced yes)
-		(property "Reference" "Q6"
+		(property "Reference" "Q5"
 			(at 159.7914 104.5753 0)
 			(effects
@@
 			(project "echo"
 				(path "/8c0b3d8b-46d3-4173-ab1e-a61765f77d61/e606b562-b239-4a02-9f90-df2cbefa5295"
-					(reference "Q6")
+					(reference "Q5")
 					(unit 1)
 				)
@@
 		(on_board yes)
 		(dnp no)
-		(property "Reference" "C42"
+		(property "Reference" "C55"
 			(at 129.54 101.6 90)
 			(effects
@@
 			(project "echo"
 				(path "/8c0b3d8b-46d3-4173-ab1e-a61765f77d61/e606b562-b239-4a02-9f90-df2cbefa5295"
-					(reference "C42")
+					(reference "C55")
 					(unit 1)
 				)
@@
 		(dnp no)
 		(fields_autoplaced yes)
-		(property "Reference" "R50"
+		(property "Reference" "R55"
 			(at 139.7 99.06 90)
 			(effects
@@
 			(project "echo"
 				(path "/8c0b3d8b-46d3-4173-ab1e-a61765f77d61/e606b562-b239-4a02-9f90-df2cbefa5295"
-					(reference "R50")
+					(reference "R55")
 					(unit 1)
 				)
@@
 		(dnp no)
 		(fields_autoplaced yes)
-		(property "Reference" "#PWR098"
+		(property "Reference" "#PWR0123"
 			(at 180.34 76.2 0)
 			(effects
@@
 			(project "echo"
 				(path "/8c0b3d8b-46d3-4173-ab1e-a61765f77d61/e606b562-b239-4a02-9f90-df2cbefa5295"
-					(reference "#PWR098")
+					(reference "#PWR0123")
 					(unit 1)
 				)
@@
 		(dnp no)
 		(fields_autoplaced yes)
-		(property "Reference" "R49"
+		(property "Reference" "R57"
 			(at 163.83 91.44 90)
 			(effects
@@
 			(project "echo"
 				(path "/8c0b3d8b-46d3-4173-ab1e-a61765f77d61/e606b562-b239-4a02-9f90-df2cbefa5295"
-					(reference "R49")
+					(reference "R57")
 					(unit 1)
 				)
@@
 		(dnp no)
 		(fields_autoplaced yes)
-		(property "Reference" "R48"
+		(property "Reference" "R58"
 			(at 177.8 85.0899 0)
 			(effects
@@
 			(project "echo"
 				(path "/8c0b3d8b-46d3-4173-ab1e-a61765f77d61/e606b562-b239-4a02-9f90-df2cbefa5295"
-					(reference "R48")
+					(reference "R58")
 					(unit 1)
 				)
@@
 		(dnp no)
 		(fields_autoplaced yes)
-		(property "Reference" "Q5"
+		(property "Reference" "Q6"
 			(at 177.5714 96.9553 0)
 			(effects
@@
 			(project "echo"
 				(path "/8c0b3d8b-46d3-4173-ab1e-a61765f77d61/e606b562-b239-4a02-9f90-df2cbefa5295"
-					(reference "Q5")
+					(reference "Q6")
 					(unit 1)
 				)
@@
 		(dnp no)
 		(fields_autoplaced yes)
-		(property "Reference" "R51"
+		(property "Reference" "R54"
 			(at 126.238 115.6278 0)
 			(effects
@@
 			(project "echo"
 				(path "/8c0b3d8b-46d3-4173-ab1e-a61765f77d61/e606b562-b239-4a02-9f90-df2cbefa5295"
-					(reference "R51")
+					(reference "R54")
 					(unit 1)
 				)

Commit message: Echo HW 1.06 Release
Parts:
- renumbered AJ1 to J7
Changed lines of the file:
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@@
 		(on_board yes)
 		(dnp no)
-		(property "Reference" "AJ1"
+		(property "Reference" "J7"
 			(at 95.7581 106.4803 0)
 			(effects
@@
 			(project "echo"
 				(path "/8c0b3d8b-46d3-4173-ab1e-a61765f77d61/e606b562-b239-4a02-9f90-df2cbefa5295"
-					(reference "AJ1")
+					(reference "J7")
 					(unit 1)
 				)
