File: usb_hub.kicad_sch (KiCad schematic)
At the start: 2 parts, among them J2 D-SUB 9 Male

Commit message: Minor fixes
Parts:
- removed C10: 100n, FRANK:Capacitor (0805), symbol Device:C_Small
- removed J2: D-SUB 9 Male, FRANK:D-SUB (9 pin, male, top mount), symbol FRANK:DB9_Male_Small
- added C35: 4.7u, FRANK:Capacitor (0805), symbol Device:C_Small
- added U9: MW7211A, FRANK:SOP-16, symbol FRANK:MW7211A
Connections:
- net GND: now also C35.2, U9.15 (GND), U9.16 (GND)
- net VBUS: now also C35.1, U9.13 (VDD5)
- new net: U9.12 (VD33), U9.14 (VD3)
- new net DM1: U9.7 (DM3)
- new net DM2: U9.5 (DM2)
- new net DM3: U9.3 (DM1)
- new net DM4: U9.1 (DM0)
- new net DM_IN: U9.10 (DMU)
- new net DP1: U9.8 (DP3)
- new net DP2: U9.6 (DP2)
- new net DP3: U9.4 (DP1)
- new net DP4: U9.2 (DP0)
- new net DP_IN: U9.11 (DPU)
- no-connect marks 0 -> 1

Commit message: HW Rev 1.03
Parts:
- renumbered C35 to C34
Changed lines of the file:
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@@
 	(title_block
 		(title "${NAME}")
-		(date "2025-06-23")
+		(date "2025-07-20")
 		(rev "${VERSION}")
 		(company "Mikhail Matveev")
@@
 		(on_board yes)
 		(dnp no)
-		(property "Reference" "C35"
+		(property "Reference" "C34"
 			(at 183.388 108.204 90)
 			(effects
@@
 			(project "echo"
 				(path "/8c0b3d8b-46d3-4173-ab1e-a61765f77d61/c703e3e8-9da2-4a1d-9cec-42d7256180fc"
-					(reference "C35")
+					(reference "C34")
 					(unit 1)
 				)

Commit message: WIP
Parts:
- added C34, C35: 10u, FRANK:Capacitor (0805), symbol Device:C
- added J11: SS-52100-004, FRANK:USB Type A (stacked), symbol Connector:USB_A_Stacked
- added R52, R53, R54, R55: 22R, FRANK:Resistor (0805), symbol Device:R
- renumbered C34 to C36
Connections:
- net GND: now also C34.2, C35.2, J11.4 (GND1), J11.8 (GND2), J11.9 (Shield)
- net VBUS: now also C34.1, C35.1, J11.1 (VBUS1), J11.5 (VBUS2)
- net DM1: no longer names the net of U9.7 (DM3)
- net DM2: no longer names the net of U9.5 (DM2)
- net DM3 renamed D2-
- net D2-: now also R55.1
- net DM4 renamed D1-
- net D1-: now also R54.1
- net DP1: no longer names the net of U9.8 (DP3)
- net DP2: no longer names the net of U9.6 (DP2)
- net DP3 renamed D2+
- net D2+: now also R53.1
- net DP4 renamed D1+
- net D1+: now also R52.1
- new net: J11.2 (D1-), R54.2
- new net: J11.3 (D1+), R52.2
- new net: J11.6 (D2-), R55.2
- new net: J11.7 (D2+), R53.2
- no-connect marks 1 -> 5
Other:
- moved on the sheet: C36, U9

Commit message: Rev 1.05 WIP
Parts:
- C59: renamed from C34; footprint FRANK:Capacitor (0805) -> FRANK:Capacitor (0603)
- C60: renamed from C35; footprint FRANK:Capacitor (0805) -> FRANK:Capacitor (0603)
- C61: renamed from C36; footprint FRANK:Capacitor (0805) -> FRANK:Capacitor (0603)
- R63: renamed from R52; footprint FRANK:Resistor (0805) -> FRANK:Resistor (0603)
- R64: renamed from R53; footprint FRANK:Resistor (0805) -> FRANK:Resistor (0603)
- R65: renamed from R54; footprint FRANK:Resistor (0805) -> FRANK:Resistor (0603)
- R66: renamed from R55; footprint FRANK:Resistor (0805) -> FRANK:Resistor (0603)
- renumbered J11 to J8, U9 to U12
Changed lines of the file:
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@@
 		(dnp no)
 		(fields_autoplaced yes)
-		(property "Reference" "#PWR099"
+		(property "Reference" "#PWR0133"
 			(at 222.25 118.11 0)
 			(effects
@@
 			(project "echo"
 				(path "/8c0b3d8b-46d3-4173-ab1e-a61765f77d61/c703e3e8-9da2-4a1d-9cec-42d7256180fc"
-					(reference "#PWR099")
+					(reference "#PWR0133")
 					(unit 1)
 				)
@@
 		(dnp no)
 		(fields_autoplaced yes)
-		(property "Reference" "J11"
+		(property "Reference" "J8"
 			(at 72.39 71.12 0)
 			(effects
@@
 			(project "echo"
 				(path "/8c0b3d8b-46d3-4173-ab1e-a61765f77d61/c703e3e8-9da2-4a1d-9cec-42d7256180fc"
-					(reference "J11")
+					(reference "J8")
 					(unit 1)
 				)
@@
 		(on_board yes)
 		(dnp no)
-		(property "Reference" "C34"
+		(property "Reference" "C59"
 			(at 118.491 85.1916 0)
 			(effects
@@
 			)
 		)
-		(property "Footprint" "FRANK:Capacitor (0805)"
+		(property "Footprint" "FRANK:Capacitor (0603)"
 			(at 116.5352 90.17 0)
 			(effects
@@
 			(project "echo"
 				(path "/8c0b3d8b-46d3-4173-ab1e-a61765f77d61/c703e3e8-9da2-4a1d-9cec-42d7256180fc"
-					(reference "C34")
+					(reference "C59")
 					(unit 1)
 				)
@@
 		(dnp no)
 		(fields_autoplaced yes)
-		(property "Reference" "#PWR097"
+		(property "Reference" "#PWR0131"
 			(at 220.98 93.98 0)
 			(effects
@@
 			(project "echo"
 				(path "/8c0b3d8b-46d3-4173-ab1e-a61765f77d61/c703e3e8-9da2-4a1d-9cec-42d7256180fc"
-					(reference "#PWR097")
+					(reference "#PWR0131")
 					(unit 1)
 				)
@@
 		(on_board yes)
 		(dnp no)
-		(property "Reference" "R54"
+		(property "Reference" "R65"
 			(at 96.012 106.68 90)
 			(effects
@@
 			)
 		)
-		(property "Footprint" "FRANK:Resistor (0805)"
+		(property "Footprint" "FRANK:Resistor (0603)"
 			(at 92.202 106.68 90)
 			(effects
@@
 			(project "echo"
 				(path "/8c0b3d8b-46d3-4173-ab1e-a61765f77d61/c703e3e8-9da2-4a1d-9cec-42d7256180fc"
-					(reference "R54")
+					(reference "R65")
 					(unit 1)
 				)
@@
 		(on_board yes)
 		(dnp no)
-		(property "Reference" "C35"
+		(property "Reference" "C60"
 			(at 129.921 85.1916 0)
 			(effects
@@
 			)
 		)
-		(property "Footprint" "FRANK:Capacitor (0805)"
+		(property "Footprint" "FRANK:Capacitor (0603)"
 			(at 127.9652 90.17 0)
 			(effects
@@
 			(project "echo"
 				(path "/8c0b3d8b-46d3-4173-ab1e-a61765f77d61/c703e3e8-9da2-4a1d-9cec-42d7256180fc"
-					(reference "C35")
+					(reference "C60")
 					(unit 1)
 				)
@@
 		(dnp no)
 		(fields_autoplaced yes)
-		(property "Reference" "#PWR094"
+		(property "Reference" "#PWR0128"
 			(at 215.9 86.36 0)
 			(effects
@@
 			(project "echo"
 				(path "/8c0b3d8b-46d3-4173-ab1e-a61765f77d61/c703e3e8-9da2-4a1d-9cec-42d7256180fc"
-					(reference "#PWR094")
+					(reference "#PWR0128")
 					(unit 1)
 				)
@@
 		(on_board yes)
 		(dnp no)
-		(property "Reference" "#PWR092"
+		(property "Reference" "#PWR0126"
 			(at 86.36 81.28 0)
 			(effects
@@
 			(project "echo"
 				(path "/8c0b3d8b-46d3-4173-ab1e-a61765f77d61/c703e3e8-9da2-4a1d-9cec-42d7256180fc"
-					(reference "#PWR092")
+					(reference "#PWR0126")
 					(unit 1)
 				)
@@
 		(on_board yes)
 		(dnp no)
-		(property "Reference" "#PWR095"
+		(property "Reference" "#PWR0129"
 			(at 115.57 97.79 0)
 			(effects
@@
 			(project "echo"
 				(path "/8c0b3d8b-46d3-4173-ab1e-a61765f77d61/c703e3e8-9da2-4a1d-9cec-42d7256180fc"
-					(reference "#PWR095")
+					(reference "#PWR0129")
 					(unit 1)
 				)
@@
 		(on_board yes)
 		(dnp no)
-		(property "Reference" "R53"
+		(property "Reference" "R64"
 			(at 104.902 105.41 90)
 			(effects
@@
 			)
 		)
-		(property "Footprint" "FRANK:Resistor (0805)"
+		(property "Footprint" "FRANK:Resistor (0603)"
 			(at 101.092 105.41 90)
 			(effects
@@
 			(project "echo"
 				(path "/8c0b3d8b-46d3-4173-ab1e-a61765f77d61/c703e3e8-9da2-4a1d-9cec-42d7256180fc"
-					(reference "R53")
+					(reference "R64")
 					(unit 1)
 				)
@@
 		(on_board yes)
 		(dnp no)
-		(property "Reference" "#PWR096"
+		(property "Reference" "#PWR0130"
 			(at 127 97.79 0)
 			(effects
@@
 			(project "echo"
 				(path "/8c0b3d8b-46d3-4173-ab1e-a61765f77d61/c703e3e8-9da2-4a1d-9cec-42d7256180fc"
-					(reference "#PWR096")
+					(reference "#PWR0130")
 					(unit 1)
 				)
@@
 		(on_board yes)
 		(dnp no)
-		(property "Reference" "C36"
+		(property "Reference" "C61"
 			(at 225.298 108.204 90)
 			(effects
@@
 			)
 		)
-		(property "Footprint" "FRANK:Capacitor (0805)"
+		(property "Footprint" "FRANK:Capacitor (0603)"
 			(at 222.25 107.95 0)
 			(effects
@@
 			(project "echo"
 				(path "/8c0b3d8b-46d3-4173-ab1e-a61765f77d61/c703e3e8-9da2-4a1d-9cec-42d7256180fc"
-					(reference "C36")
+					(reference "C61")
 					(unit 1)
 				)
@@
 		(on_board yes)
 		(dnp no)
-		(property "Reference" "R52"
+		(property "Reference" "R63"
 			(at 92.202 100.33 90)
 			(effects
@@
 			)
 		)
-		(property "Footprint" "FRANK:Resistor (0805)"
+		(property "Footprint" "FRANK:Resistor (0603)"
 			(at 88.392 100.33 90)
 			(effects
@@
 			(project "echo"
 				(path "/8c0b3d8b-46d3-4173-ab1e-a61765f77d61/c703e3e8-9da2-4a1d-9cec-42d7256180fc"
-					(reference "R52")
+					(reference "R63")
 					(unit 1)
 				)
@@
 		(on_board yes)
 		(dnp no)
-		(property "Reference" "#PWR093"
+		(property "Reference" "#PWR0127"
 			(at 92.71 81.28 0)
 			(effects
@@
 			(project "echo"
 				(path "/8c0b3d8b-46d3-4173-ab1e-a61765f77d61/c703e3e8-9da2-4a1d-9cec-42d7256180fc"
-					(reference "#PWR093")
+					(reference "#PWR0127")
 					(unit 1)
 				)
@@
 		(dnp no)
 		(fields_autoplaced yes)
-		(property "Reference" "#PWR098"
+		(property "Reference" "#PWR0132"
 			(at 72.39 114.3 0)
 			(effects
@@
 			(project "echo"
 				(path "/8c0b3d8b-46d3-4173-ab1e-a61765f77d61/c703e3e8-9da2-4a1d-9cec-42d7256180fc"
-					(reference "#PWR098")
+					(reference "#PWR0132")
 					(unit 1)
 				)
@@
 		(dnp no)
 		(fields_autoplaced yes)
-		(property "Reference" "U9"
+		(property "Reference" "U12"
 			(at 180.34 76.2 0)
 			(effects
@@
 			(project "echo"
 				(path "/8c0b3d8b-46d3-4173-ab1e-a61765f77d61/c703e3e8-9da2-4a1d-9cec-42d7256180fc"
-					(reference "U9")
+					(reference "U12")
 					(unit 1)
 				)
@@
 		(on_board yes)
 		(dnp no)
-		(property "Reference" "R55"
+		(property "Reference" "R66"
 			(at 108.712 111.76 90)
 			(effects
@@
 			)
 		)
-		(property "Footprint" "FRANK:Resistor (0805)"
+		(property "Footprint" "FRANK:Resistor (0603)"
 			(at 104.902 111.76 90)
 			(effects
@@
 			(project "echo"
 				(path "/8c0b3d8b-46d3-4173-ab1e-a61765f77d61/c703e3e8-9da2-4a1d-9cec-42d7256180fc"
-					(reference "R55")
-					(unit 1)
-				)
+					(reference "R66")
+					(unit 1)
+				)

Commit message: HW 1.06 WIP
Parts:
- renumbered C59 to C73, C60 to C74, C61 to C75, R63 to R70, R65 to R71, R64 to R72, R66 to R73, U12 to U14
Changed lines of the file:
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@@
 		(dnp no)
 		(fields_autoplaced yes)
-		(property "Reference" "#PWR0133"
+		(property "Reference" "#PWR0153"
 			(at 222.25 118.11 0)
 			(effects
@@
 			(project "echo"
 				(path "/8c0b3d8b-46d3-4173-ab1e-a61765f77d61/c703e3e8-9da2-4a1d-9cec-42d7256180fc"
-					(reference "#PWR0133")
+					(reference "#PWR0153")
 					(unit 1)
 				)
@@
 		(on_board yes)
 		(dnp no)
-		(property "Reference" "C59"
+		(property "Reference" "C73"
 			(at 118.491 85.1916 0)
 			(effects
@@
 			(project "echo"
 				(path "/8c0b3d8b-46d3-4173-ab1e-a61765f77d61/c703e3e8-9da2-4a1d-9cec-42d7256180fc"
-					(reference "C59")
+					(reference "C73")
 					(unit 1)
 				)
@@
 		(dnp no)
 		(fields_autoplaced yes)
-		(property "Reference" "#PWR0131"
+		(property "Reference" "#PWR0154"
 			(at 220.98 93.98 0)
 			(effects
@@
 			(project "echo"
 				(path "/8c0b3d8b-46d3-4173-ab1e-a61765f77d61/c703e3e8-9da2-4a1d-9cec-42d7256180fc"
-					(reference "#PWR0131")
+					(reference "#PWR0154")
 					(unit 1)
 				)
@@
 		(on_board yes)
 		(dnp no)
-		(property "Reference" "R65"
+		(property "Reference" "R71"
 			(at 96.012 106.68 90)
 			(effects
@@
 			(project "echo"
 				(path "/8c0b3d8b-46d3-4173-ab1e-a61765f77d61/c703e3e8-9da2-4a1d-9cec-42d7256180fc"
-					(reference "R65")
+					(reference "R71")
 					(unit 1)
 				)
@@
 		(on_board yes)
 		(dnp no)
-		(property "Reference" "C60"
+		(property "Reference" "C74"
 			(at 129.921 85.1916 0)
 			(effects
@@
 			(project "echo"
 				(path "/8c0b3d8b-46d3-4173-ab1e-a61765f77d61/c703e3e8-9da2-4a1d-9cec-42d7256180fc"
-					(reference "C60")
+					(reference "C74")
 					(unit 1)
 				)
@@
 		(dnp no)
 		(fields_autoplaced yes)
-		(property "Reference" "#PWR0128"
+		(property "Reference" "#PWR0152"
 			(at 215.9 86.36 0)
 			(effects
@@
 			(project "echo"
 				(path "/8c0b3d8b-46d3-4173-ab1e-a61765f77d61/c703e3e8-9da2-4a1d-9cec-42d7256180fc"
-					(reference "#PWR0128")
+					(reference "#PWR0152")
 					(unit 1)
 				)
@@
 		(on_board yes)
 		(dnp no)
-		(property "Reference" "#PWR0126"
+		(property "Reference" "#PWR0148"
 			(at 86.36 81.28 0)
 			(effects
@@
 			(project "echo"
 				(path "/8c0b3d8b-46d3-4173-ab1e-a61765f77d61/c703e3e8-9da2-4a1d-9cec-42d7256180fc"
-					(reference "#PWR0126")
+					(reference "#PWR0148")
 					(unit 1)
 				)
@@
 		(on_board yes)
 		(dnp no)
-		(property "Reference" "#PWR0129"
+		(property "Reference" "#PWR0150"
 			(at 115.57 97.79 0)
 			(effects
@@
 			(project "echo"
 				(path "/8c0b3d8b-46d3-4173-ab1e-a61765f77d61/c703e3e8-9da2-4a1d-9cec-42d7256180fc"
-					(reference "#PWR0129")
+					(reference "#PWR0150")
 					(unit 1)
 				)
@@
 		(on_board yes)
 		(dnp no)
-		(property "Reference" "R64"
+		(property "Reference" "R72"
 			(at 104.902 105.41 90)
 			(effects
@@
 			(project "echo"
 				(path "/8c0b3d8b-46d3-4173-ab1e-a61765f77d61/c703e3e8-9da2-4a1d-9cec-42d7256180fc"
-					(reference "R64")
+					(reference "R72")
 					(unit 1)
 				)
@@
 		(on_board yes)
 		(dnp no)
-		(property "Reference" "#PWR0130"
+		(property "Reference" "#PWR0151"
 			(at 127 97.79 0)
 			(effects
@@
 			(project "echo"
 				(path "/8c0b3d8b-46d3-4173-ab1e-a61765f77d61/c703e3e8-9da2-4a1d-9cec-42d7256180fc"
-					(reference "#PWR0130")
+					(reference "#PWR0151")
 					(unit 1)
 				)
@@
 		(on_board yes)
 		(dnp no)
-		(property "Reference" "C61"
+		(property "Reference" "C75"
 			(at 225.298 108.204 90)
 			(effects
@@
 			(project "echo"
 				(path "/8c0b3d8b-46d3-4173-ab1e-a61765f77d61/c703e3e8-9da2-4a1d-9cec-42d7256180fc"
-					(reference "C61")
+					(reference "C75")
 					(unit 1)
 				)
@@
 		(on_board yes)
 		(dnp no)
-		(property "Reference" "R63"
+		(property "Reference" "R70"
 			(at 92.202 100.33 90)
 			(effects
@@
 			(project "echo"
 				(path "/8c0b3d8b-46d3-4173-ab1e-a61765f77d61/c703e3e8-9da2-4a1d-9cec-42d7256180fc"
-					(reference "R63")
+					(reference "R70")
 					(unit 1)
 				)
@@
 		(on_board yes)
 		(dnp no)
-		(property "Reference" "#PWR0127"
+		(property "Reference" "#PWR0149"
 			(at 92.71 81.28 0)
 			(effects
@@
 			(project "echo"
 				(path "/8c0b3d8b-46d3-4173-ab1e-a61765f77d61/c703e3e8-9da2-4a1d-9cec-42d7256180fc"
-					(reference "#PWR0127")
+					(reference "#PWR0149")
 					(unit 1)
 				)
@@
 		(dnp no)
 		(fields_autoplaced yes)
-		(property "Reference" "#PWR0132"
+		(property "Reference" "#PWR0147"
 			(at 72.39 114.3 0)
 			(effects
@@
 			(project "echo"
 				(path "/8c0b3d8b-46d3-4173-ab1e-a61765f77d61/c703e3e8-9da2-4a1d-9cec-42d7256180fc"
-					(reference "#PWR0132")
+					(reference "#PWR0147")
 					(unit 1)
 				)
@@
 		(dnp no)
 		(fields_autoplaced yes)
-		(property "Reference" "U12"
+		(property "Reference" "U14"
 			(at 180.34 76.2 0)
 			(effects
@@
 			(project "echo"
 				(path "/8c0b3d8b-46d3-4173-ab1e-a61765f77d61/c703e3e8-9da2-4a1d-9cec-42d7256180fc"
-					(reference "U12")
+					(reference "U14")
 					(unit 1)
 				)
@@
 		(on_board yes)
 		(dnp no)
-		(property "Reference" "R66"
+		(property "Reference" "R73"
 			(at 108.712 111.76 90)
 			(effects
@@
 			(project "echo"
 				(path "/8c0b3d8b-46d3-4173-ab1e-a61765f77d61/c703e3e8-9da2-4a1d-9cec-42d7256180fc"
-					(reference "R66")
-					(unit 1)
-				)
+					(reference "R73")
+					(unit 1)
+				)

Commit message: Echo HW 1.06 Release
Parts:
- renumbered J8 to J9
Changed lines of the file:
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@@
 		(dnp no)
 		(fields_autoplaced yes)
-		(property "Reference" "J8"
+		(property "Reference" "J9"
 			(at 72.39 71.12 0)
 			(effects
@@
 			(project "echo"
 				(path "/8c0b3d8b-46d3-4173-ab1e-a61765f77d61/c703e3e8-9da2-4a1d-9cec-42d7256180fc"
-					(reference "J8")
+					(reference "J9")
 					(unit 1)
 				)
